File: GPS-USB_Front_End_Board/kicad_board_design/usb_gps.kicad_pcb (KiCad board)
At the start: 4 copper layers, 99.1 x 53.3 mm, 90 parts, among them J1 Micro-USB Connector, J3 SMA, P1 CONN_02X12, U1 93LCxxB, U2 FT2232HL-REEL, U3 L4931 LDO, U4 MAX8510, U5 MAX8510, U6 MAX2769CETI+, U7 SAWTEK-855969, U8 LT1719S6 -- Not Populated, X1 13.368MHz TCXO, Y1 12MHz Crystal

Commit message: Minor cleanup.
Routing:
- net GND: track 108.3 -> 132.7 mm
- net /MAX_2769/D2: track 52.2 -> 37.1 mm
Changed lines of the file:
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@@
     (links 220)
     (no_connects 0)
-    (area 78.693 60.884999 181.685001 115.135)
+    (area 73.444143 60.395 190.588858 115.135)
     (thickness 1.6)
     (drawings 6)
-    (tracks 960)
+    (tracks 954)
     (zones 0)
     (modules 90)
@@
     (tags "resistor 0805")
     (attr smd)
-    (fp_text reference R14 (at 0 -2.1 180) (layer F.SilkS)
+    (fp_text reference R14 (at -4.064 0.381 180) (layer F.SilkS)
       (effects (font (size 1 1) (thickness 0.15)))
     )
@@
   (via (at 90.17 74.93) (size 0.4572) (layers F.Cu B.Cu) (net 0))
   (segment (start 90.14 74.96) (end 90.17 74.93) (width 0.254) (layer F.Cu) (net 0))
+  (segment (start 121.285 71.374) (end 122.174 71.374) (width 0.2032) (layer F.Cu) (net 1))
+  (segment (start 122.489 70.424) (end 123.571 70.424) (width 0.2032) (layer F.Cu) (net 1))
+  (segment (start 122.301 70.612) (end 122.489 70.424) (width 0.2032) (layer F.Cu) (net 1))
+  (segment (start 122.301 71.247) (end 122.301 70.612) (width 0.2032) (layer F.Cu) (net 1))
+  (segment (start 122.174 71.374) (end 122.301 71.247) (width 0.2032) (layer F.Cu) (net 1))
+  (segment (start 86.868 74.706) (end 88.295 74.706) (width 0.399999) (layer F.Cu) (net 1))
+  (segment (start 88.295 74.706) (end 89.408 75.819) (width 0.399999) (layer F.Cu) (net 1))
+  (segment (start 89.408 75.819) (end 97.79 75.819) (width 0.399999) (layer F.Cu) (net 1))
+  (segment (start 97.536 73.66) (end 96.64 73.66) (width 0.254) (layer F.Cu) (net 1))
+  (segment (start 97.536 73.66) (end 97.79 73.914) (width 0.254) (layer F.Cu) (net 1))
+  (segment (start 97.79 73.914) (end 97.79 75.819) (width 0.254) (layer F.Cu) (net 1))
+  (via (at 97.79 75.819) (size 0.4572) (layers F.Cu B.Cu) (net 1))
+  (segment (start 89.408 75.819) (end 97.79 75.819) (width 0.2032) (layer F.Cu) (net 1))
+  (segment (start 88.295 74.706) (end 89.408 75.819) (width 0.2032) (layer F.Cu) (net 1))
   (segment (start 166.262 69.5008) (end 166.262 68.599) (width 0.399999) (layer F.Cu) (net 1))
   (segment (start 162.433 68.834) (end 162.433 69.535) (width 0.399999) (layer F.Cu) (net 1))
@@
   (via (at 107.061 69.723) (size 0.4572) (layers F.Cu B.Cu) (net 1))
   (via (at 93.091 71.12) (size 0.4572) (layers F.Cu B.Cu) (net 1))
-  (via (at 97.79 75.819) (size 0.4572) (layers F.Cu B.Cu) (net 1))
   (via (at 92.71 65.786) (size 0.4572) (layers F.Cu B.Cu) (net 1))
   (segment (start 161.604 86.699) (end 161.608 86.7029) (width 0.254) (layer F.Cu) (net 1))
@@
   (segment (start 105.41 67.86) (end 105.41 68.072) (width 0.254) (layer F.Cu) (net 1))
   (segment (start 91.99 71.12) (end 93.091 71.12) (width 0.254) (layer F.Cu) (net 1))
-  (segment (start 97.79 73.914) (end 97.79 75.819) (width 0.254) (layer F.Cu) (net 1))
-  (segment (start 97.536 73.66) (end 97.79 73.914) (width 0.254) (layer F.Cu) (net 1))
-  (segment (start 96.64 73.66) (end 97.536 73.66) (width 0.254) (layer F.Cu) (net 1))
   (segment (start 92.668 65.744) (end 92.71 65.786) (width 0.254) (layer F.Cu) (net 1))
   (segment (start 91.567 65.744) (end 92.668 65.744) (width 0.254) (layer F.Cu) (net 1) (status 10))
@@
   (segment (start 143.9986 87.5933) (end 143.0641 86.6588) (width 0.2032) (layer F.Cu) (net 15))
   (segment (start 144.0173 87.5933) (end 143.9986 87.5933) (width 0.2032) (layer F.Cu) (net 15))
+  (segment (start 150.622 93.218) (end 151.765 93.218) (width 0.4) (layer F.Cu) (net 16))
   (segment (start 151.773 93.21) (end 152.56 93.21) (width 0.254) (layer F.Cu) (net 16))
   (segment (start 151.765 93.218) (end 151.773 93.21) (width 0.254) (layer F.Cu) (net 16))
   (segment (start 140.763 87.583) (end 140.549 87.797) (width 0.4) (layer F.Cu) (net 16))
   (segment (start 141.777 87.583) (end 140.763 87.583) (width 0.4) (layer F.Cu) (net 16))
-  (segment (start 150.622 93.218) (end 151.765 93.218) (width 0.4) (layer F.Cu) (net 16))
   (segment (start 147.955 90.551) (end 150.622 93.218) (width 0.4) (layer F.Cu) (net 16))
   (segment (start 141.478 90.551) (end 147.955 90.551) (width 0.4) (layer F.Cu) (net 16))
@@
   (segment (start 149.606 94.869) (end 154.4066 94.869) (width 0.2032) (layer In2.Cu) (net 30))
   (segment (start 154.4066 94.869) (end 154.432 94.8944) (width 0.2032) (layer In2.Cu) (net 30))
-  (segment (start 149.606 94.869) (end 149.606 96.5962) (width 0.2032) (layer In2.Cu) (net 30))
-  (segment (start 149.606 96.5962) (end 149.6568 96.647) (width 0.2032) (layer In2.Cu) (net 30))
-  (segment (start 151.4602 93.091) (end 151.4602 96.6724) (width 0.2032) (layer In2.Cu) (net 30))
-  (segment (start 150.2156 93.1926) (end 150.2156 94.2848) (width 0.2032) (layer In2.Cu) (net 30))
   (segment (start 143.51 94.869) (end 134.0615 94.869) (width 0.2032) (layer In2.Cu) (net 30))
   (segment (start 146.1262 94.869) (end 143.51 94.869) (width 0.2032) (layer In2.Cu) (net 30))
@@
   (segment (start 149.6314 94.869) (end 149.606 94.869) (width 0.2032) (layer In2.Cu) (net 30))
   (segment (start 149.606 94.869) (end 146.1262 94.869) (width 0.2032) (layer In2.Cu) (net 30))
-  (segment (start 150.2156 94.2848) (end 149.6314 94.869) (width 0.2032) (layer In2.Cu) (net 30))
   (segment (start 155.0924 94.8944) (end 154.432 94.8944) (width 0.2032) (layer In2.Cu) (net 30))
-  (segment (start 150.5204 91.821) (end 150.5204 91.7194) (width 0.2032) (layer In2.Cu) (net 30))
-  (segment (start 150.5712 91.821) (end 150.5204 91.821) (width 0.2032) (layer In2.Cu) (net 30))
-  (segment (start 150.2156 92.1766) (end 150.5712 91.821) (width 0.2032) (layer In2.Cu) (net 30))
-  (segment (start 150.2156 93.1926) (end 150.2156 92.1766) (width 0.2032) (layer In2.Cu) (net 30))
-  (segment (start 150.1902 93.218) (end 150.2156 93.1926) (width 0.2032) (layer In2.Cu) (net 30))
-  (segment (start 151.3332 93.218) (end 150.1902 93.218) (width 0.2032) (layer In2.Cu) (net 30))
-  (segment (start 151.4602 93.091) (end 151.3332 93.218) (width 0.2032) (layer In2.Cu) (net 30))
-  (segment (start 151.4602 92.4052) (end 151.4602 93.091) (width 0.2032) (layer In2.Cu) (net 30))
-  (segment (start 154.432 94.8944) (end 151.8412 92.3036) (width 0.2032) (layer In2.Cu) (net 30))
-  (segment (start 151.8412 92.3036) (end 151.5618 92.3036) (width 0.2032) (layer In2.Cu) (net 30))
-  (segment (start 151.5618 92.3036) (end 151.4602 92.4052) (width 0.2032) (layer In2.Cu) (net 30))
   (segment (start 155.8798 95.6818) (end 155.0924 94.8944) (width 0.2032) (layer In2.Cu) (net 30))
   (segment (start 155.0924 94.8944) (end 155.067 94.869) (width 0.2032) (layer In2.Cu) (net 30))

Commit message: Intermediate routing.
Parts:
- removed R11: NC, Resistors_SMD:R_0805_HandSoldering
- removed R12: 0, Resistors_SMD:R_0805_HandSoldering
- removed REF** (x4): MountingHole_2.2mm_M2_Pad_Via, Mounting_Holes:MountingHole_2.2mm_M2_Pad_Via
- added C39: .47nF, Capacitors_SMD:C_0402, F.Cu at (154.9, 85.3)
- added L1: 5.6nH, Capacitors_SMD:C_0402, F.Cu at (159.5, 92.2)
- added P2: CONN_01X03, Connectors_Molex:Molex_KK-6410-03_03x2.54mm_Straight, F.Cu at (177.2, 75.6)
- added W7: -BB, Measurement_Points:Measurement_Point_Round-TH_Small, F.Cu at (162.3, 98.0)
- added W8: +BB, Measurement_Points:Measurement_Point_Round-TH_Small, F.Cu at (160.0, 98.0)
- C19, C31, C32: footprint Capacitors_SMD:C_0805_HandSoldering -> Capacitors_SMD:C_0402
- C23, C36: value .1uF -> 2.2uF; footprint Capacitors_SMD:C_0402 -> Capacitors_SMD:C_0805
- C29: value NC -> 1.7pF; footprint Capacitors_SMD:C_0805_HandSoldering -> Capacitors_SMD:C_0402
- U6: value MAX2769CETI+ -> MAX2771
- moved C27 38.4 mm to (135.6, 84.5)
- moved C25 36.2 mm to (137.4, 79.4), turned to 180 degrees
- moved R13 36.2 mm to (137.4, 81.9), turned to 0 degrees
- moved R16 30.9 mm to (135.1, 92.7), turned to 0 degrees
- moved R15 27.1 mm to (135.1, 95.2), turned to 180 degrees
- moved C23 26.6 mm to (160.3, 69.1), turned to 0 degrees
- moved C29 26.4 mm to (161.2, 94.1)
- moved C26 19.4 mm to (142.0, 74.3)
- moved C30 15.2 mm to (178.1, 85.0)
- moved U7 14.7 mm to (156.1, 80.9), turned to 180 degrees
- moved C17 14.4 mm to (152.9, 68.2), turned to 270 degrees
- moved C19 13.6 mm to (158.5, 90.3), turned to 0 degrees
- moved C28 11.6 mm to (154.8, 77.9), turned to 270 degrees
- moved C11 11.5 mm to (146.6, 108.1), turned to 90 degrees
- moved C13 11.4 mm to (151.5, 89.3)
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Connections:
- C29 pad 1: Net-(C28-Pad2) -> Net-(C29-Pad1)
- C29 pad 2: /MAX_2769/MIXIN -> GND
- C30 pad 1: /MAX_2769/ANTBIAS -> Net-(C30-Pad1)
- C31 pad 1: /MAX_2769/ANTBIAS -> Net-(C30-Pad1)
- C32 pad 2: /MAX_2769/LNA2 -> Net-(C29-Pad1)
- L4 pad 1: /MAX_2769/ANTBIAS -> Net-(C30-Pad1)
- R7 pad 1: /USB_FT2232/GPIO2 -> /USB_FT2232/GPIO0
- U2 pad 26: /MAX_2769/ANTFLAG -> /USB_FT2232/GPIO0
- U2 pad 28: /USB_FT2232/GPIO2 -> Net-(U2-Pad28)
- U2 pad 29: /USB_FT2232/GPIO3 -> Net-(U2-Pad29)
- U6 pad 1: /MAX_2769/ANTFLAG -> Net-(C25-Pad1)
- U6 pad 10: /MAX_2769/CS# -> /MAX_2769/Q1
- U6 pad 11: /MAX_2769/VCCA -> /MAX_2769/Q0
- U6 pad 12: Net-(C25-Pad1) -> /MAX_2769/I0
- U6 pad 13: /MAX_2769/VCCA -> /MAX_2769/I1
- U6 pad 14: /MAX_2769/VCCA -> /MAX_2769/VCCD
- U6 pad 15: Net-(C20-Pad2) -> Net-(U6-Pad15)
- U6 pad 16: Net-(C26-Pad1) -> Net-(U6-Pad16)
- U6 pad 17: /MAX_2769/Q1 -> /USB_FT2232/GPIO1
- U6 pad 18: /MAX_2769/Q0 -> /USB_FT2232/GPIO0
- U6 pad 19: /MAX_2769/VCCD -> Net-(L1-Pad2)
- U6 pad 2: Net-(C28-Pad1) -> /MAX_2769/VCCA
- U6 pad 20: /MAX_2769/I0 -> Net-(U6-Pad20)
- U6 pad 21: /MAX_2769/I1 -> Net-(U6-Pad21)
- U6 pad 22: Net-(U6-Pad22) -> /MAX_2769/VCCA
- U6 pad 23: /MAX_2769/VCCA -> Net-(U6-Pad23)
- U6 pad 24: /USB_FT2232/GPIO3 -> Net-(C28-Pad1)
- U6 pad 25: /MAX_2769/LNA2 -> Net-(C39-Pad2)
- U6 pad 27: Net-(U6-Pad27) -> /MAX_2769/VCCA
- U6 pad 28: Net-(U6-Pad28) -> /MAX_2769/VCCA
- U6 pad 3: /MAX_2769/ANTBIAS -> Net-(C20-Pad2)
- U6 pad 4: /MAX_2769/VCCA -> Net-(C26-Pad1)
- U6 pad 5: /MAX_2769/MIXIN -> Net-(U6-Pad5)
- U6 pad 6: /USB_FT2232/GPIO1 -> /MAX_2769/VCCA
- U6 pad 7: /USB_FT2232/GPIO2 -> /MAX_2769/SDATA
- U6 pad 8: /MAX_2769/SDATA -> /MAX_2769/SCLKL
- U6 pad 9: /MAX_2769/SCLKL -> /MAX_2769/CS#
Routing:
- net /MAX_2769/VCCA: track 41.9 -> 171.8 mm, vias 18 -> 0
- net /USB_FT2232/GPIO3: track 110.5 -> 0.00 mm, vias 4 -> 0
- net /MAX_2769/VCC3V3: track 35.9 -> 98.3 mm, vias 21 -> 22
- net /USB_FT2232/GPIO2: track 57.2 -> 0.00 mm, vias 2 -> 0
- net /MAX_2769/VCCD: track 61.9 -> 6.86 mm, vias 2 -> 0
- net /MAX_2769/ANTFLAG: track 49.9 -> 0.00 mm, vias 2 -> 0
- net GND: track 132.7 -> 88.9 mm, vias 25 -> 31
- net Net-(C26-Pad2): track 48.7 -> 10.0 mm
- net /MAX_2769/D2: track 37.1 -> 1.09 mm, vias 1 -> 0
- net /MAX_2769/D3: track 33.7 -> 1.09 mm, vias 1 -> 0
- net Net-(U2-Pad29): track 0.00 -> 31.1 mm, vias 0 -> 2
- net /MAX_2769/SCLKL: track 30.1 -> 0.00 mm
- net /MAX_2769/ANTBIAS: track 25.9 -> 0.00 mm, vias 2 -> 0
- net /MAX_2769/I1: track 25.6 -> 0.00 mm, vias 2 -> 0
- net /MAX_2769/I0: track 24.6 -> 0.00 mm, vias 2 -> 0
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