File: MicroSemi_FPGA_Dev_Board/kicad_board_design/A3P250_Dev_Board/UnitA.sch (KiCad schematic (older format))
At the start: 4 parts, among them J1 Conn_01x20, U1 A3P250

Commit message: Routed, fixed labels, added test points.
Connections:
- net GND: no longer U1.100 (VMV0)
- net at C22.1, C23.1, J1.9 (Pin_9)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: now also U1.100 (VMV0)
Other:
- moved on the sheet: C22, C23
Changed lines of the file:
@@
 L power:PWR_FLAG #FLG0101
 U 1 1 5DCBCE58
-P 4250 3050
-F 0 "#FLG0101" H 4250 3125 50  0001 C CNN
-F 1 "PWR_FLAG" H 4250 3224 50  0000 C CNN
-F 2 "" H 4250 3050 50  0001 C CNN
-F 3 "~" H 4250 3050 50  0001 C CNN
-	1    4250 3050
+P 4100 3050
+F 0 "#FLG0101" H 4100 3125 50  0001 C CNN
+F 1 "PWR_FLAG" H 4100 3224 50  0000 C CNN
+F 2 "" H 4100 3050 50  0001 C CNN
+F 3 "~" H 4100 3050 50  0001 C CNN
+	1    4100 3050
 	1    0    0    -1
 $EndComp
@@
 	1    0    0    -1
 $EndComp
-Text GLabel 4300 3450 0    50   Input ~ 0
+Text GLabel 4150 3450 0    50   Input ~ 0
 GND
 Text GLabel 4650 2650 0    50   Input ~ 0
@@
 	5200 2650 5200 3550
 Wire Wire Line
-	4300 3450 4450 3450
-Wire Wire Line
-	5100 3450 5100 3550
+	4150 3450 4300 3450
 $Comp
 L Device:C_Small C?
 U 1 1 5DD0839D
-P 4750 3250
+P 4600 3250
 AR Path="/5DC7725E/5DD0839D" Ref="C?"  Part="1"
 AR Path="/5DC77250/5DD0839D" Ref="C23"  Part="1"
-F 0 "C23" H 4842 3296 50  0000 L CNN
-F 1 "0.01uF" H 4842 3205 50  0000 L CNN
-F 2 "Capacitor_SMD:C_0402_1005Metric" H 4750 3250 50  0001 C CNN
-F 3 "~" H 4750 3250 50  0001 C CNN
-F 4 "Murata" H 4750 3250 50  0001 C CNN "MFR"
-F 5 "GRM155R71C103KA01D" H 4750 3250 50  0001 C CNN "MPN"
-F 6 "Digikey" H 4750 3250 50  0001 C CNN "SPR"
-F 7 "490-1313-1-ND" H 4750 3250 50  0001 C CNN "SPN"
-F 8 "-" H -1850 -700 50  0001 C CNN "SPURL"
-	1    4750 3250
+F 0 "C23" H 4692 3296 50  0000 L CNN
+F 1 "0.01uF" H 4692 3205 50  0000 L CNN
+F 2 "Capacitor_SMD:C_0402_1005Metric" H 4600 3250 50  0001 C CNN
+F 3 "~" H 4600 3250 50  0001 C CNN
+F 4 "Murata" H 4600 3250 50  0001 C CNN "MFR"
+F 5 "GRM155R71C103KA01D" H 4600 3250 50  0001 C CNN "MPN"
+F 6 "Digikey" H 4600 3250 50  0001 C CNN "SPR"
+F 7 "490-1313-1-ND" H 4600 3250 50  0001 C CNN "SPN"
+F 8 "-" H -2000 -700 50  0001 C CNN "SPURL"
+	1    4600 3250
 	1    0    0    -1
 $EndComp
@@
 L Device:C_Small C?
 U 1 1 5DD083AA
-P 4450 3250
+P 4300 3250
 AR Path="/5DC7725E/5DD083AA" Ref="C?"  Part="1"
 AR Path="/5DC77250/5DD083AA" Ref="C22"  Part="1"
-F 0 "C22" H 4542 3296 50  0000 L CNN
-F 1 ".1uF" H 4500 3200 50  0000 L CNN
-F 2 "Capacitor_SMD:C_0402_1005Metric" H 4450 3250 50  0001 C CNN
-F 3 "~" H 4450 3250 50  0001 C CNN
-F 4 "Yageo" H 4450 3250 50  0001 C CNN "TDK"
-F 5 "CGA2B1X7R1C104K050BC" H 4450 3250 50  0001 C CNN "MPN"
-F 6 "Digikey" H 4450 3250 50  0001 C CNN "SPR"
-F 7 "445-5613-1-ND" H 4450 3250 50  0001 C CNN "SPN"
-F 8 "-" H -1850 -700 50  0001 C CNN "MFR"
-F 9 "-" H -1850 -700 50  0001 C CNN "SPURL"
-	1    4450 3250
+F 0 "C22" H 4392 3296 50  0000 L CNN
+F 1 ".1uF" H 4350 3200 50  0000 L CNN
+F 2 "Capacitor_SMD:C_0402_1005Metric" H 4300 3250 50  0001 C CNN
+F 3 "~" H 4300 3250 50  0001 C CNN
+F 4 "Yageo" H 4300 3250 50  0001 C CNN "TDK"
+F 5 "CGA2B1X7R1C104K050BC" H 4300 3250 50  0001 C CNN "MPN"
+F 6 "Digikey" H 4300 3250 50  0001 C CNN "SPR"
+F 7 "445-5613-1-ND" H 4300 3250 50  0001 C CNN "SPN"
+F 8 "-" H -2000 -700 50  0001 C CNN "MFR"
+F 9 "-" H -2000 -700 50  0001 C CNN "SPURL"
+	1    4300 3250
 	1    0    0    -1
 $EndComp
@@
 	6100 2450 6100 3050
 Wire Wire Line
-	4250 3050 4450 3050
+	4100 3050 4300 3050
 Connection ~ 6100 3050
 Wire Wire Line
 	6100 3050 6100 3550
 Wire Wire Line
-	4750 3050 4750 3150
-Connection ~ 4750 3050
+	4600 3050 4600 3150
+Connection ~ 4600 3050
 Wire Wire Line
-	4750 3050 6100 3050
+	4600 3050 5100 3050
 Wire Wire Line
-	4750 3350 4750 3450
-Connection ~ 4750 3450
+	4600 3350 4600 3450
 Wire Wire Line
-	4750 3450 5100 3450
+	4300 3350 4300 3450
+Connection ~ 4300 3450
 Wire Wire Line
-	4450 3350 4450 3450
-Connection ~ 4450 3450
+	4300 3450 4600 3450
 Wire Wire Line
-	4450 3450 4750 3450
+	4300 3050 4300 3150
+Connection ~ 4300 3050
 Wire Wire Line
-	4450 3050 4450 3150
-Connection ~ 4450 3050
+	4300 3050 4600 3050
 Wire Wire Line
-	4450 3050 4750 3050
+	5100 3050 5100 3550
+Connection ~ 5100 3050
+Wire Wire Line
+	5100 3050 6100 3050
 $EndSCHEMATC
