File: MicroSemi_FPGA_Dev_Board/kicad_board_design/A3P250_Dev_Board/UnitB.sch (KiCad schematic (older format))
At the start: 4 parts, among them J2 Conn_01x20, U1 A3P250

Commit message: Routed, fixed labels, added test points.
Connections:
- net GND: no longer U1.74 (VMV1)
- net at C24.1, C25.1, J2.6 (Pin_6)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: now also U1.74 (VMV1)
Changed lines of the file:
@@
 	7500 3150 6950 3150
-Wire Wire Line
-	5950 3150 5950 3300
-Wire Wire Line
-	5700 3300 5950 3300
 Wire Wire Line
 	7500 2750 6950 2750
 Wire Wire Line
-	6050 2750 6050 3900
+	6050 2750 6050 3300
 Connection ~ 6050 3900
 Wire Wire Line
@@
 Wire Wire Line
 	6650 3050 6650 3150
-Connection ~ 6650 3150
-Wire Wire Line
-	6650 3150 5950 3150
 Wire Wire Line
 	6950 3050 6950 3150
@@
 Wire Wire Line
 	6950 3150 6650 3150
+Wire Wire Line
+	5700 3300 6050 3300
+Connection ~ 6050 3300
+Wire Wire Line
+	6050 3300 6050 3900
 $EndSCHEMATC
