File: MicroSemi_FPGA_Dev_Board/kicad_board_design/A3P250_Dev_Board/UnitC.sch (KiCad schematic (older format))
At the start: 4 parts, among them J3 Conn_01x20, U1 A3P250

Commit message: Routed, fixed labels, added test points.
Connections:
- net GND: no longer U1.50 (VMV2)
- net at C26.1, C27.1, J3.9 (Pin_9)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: now also U1.50 (VMV2)
Changed lines of the file:
@@
 	5100 3750 5100 4850
-Wire Wire Line
-	6900 3750 6900 4400
-Wire Wire Line
-	6900 4400 7250 4400
 Wire Wire Line
 	6900 4850 6900 4550
@@
 Wire Wire Line
 	7250 4300 7250 4400
-Connection ~ 7250 4400
 Wire Wire Line
 	7250 4400 7550 4400
@@
 Connection ~ 7250 4000
 Wire Wire Line
-	7250 4000 6200 4000
+	7250 4000 6900 4000
+Wire Wire Line
+	6900 3750 6900 4000
+Connection ~ 6900 4000
+Wire Wire Line
+	6900 4000 6200 4000
 $EndSCHEMATC
