File: MicroSemi_FPGA_Dev_Board/kicad_board_design/A3P250_Dev_Board/UnitE.sch (KiCad schematic (older format))
At the start: 31 parts, among them U1 A3P250, U2 LTC3561A, U3 LT1962-3.3

Commit message: Routed, fixed labels, added test points.
Parts:
- added TP3: +5V, TestPoint:TestPoint_THTPad_1.5x1.5mm_Drill0.7mm, symbol Connector:TestPoint
- added TP4: GND, TestPoint:TestPoint_THTPad_1.5x1.5mm_Drill0.7mm, symbol Connector:TestPoint
- added TP5: 1.5V Core, TestPoint:TestPoint_THTPad_1.5x1.5mm_Drill0.7mm, symbol Connector:TestPoint
- added TP6: 1.5V PLL, TestPoint:TestPoint_THTPad_1.5x1.5mm_Drill0.7mm, symbol Connector:TestPoint
Connections:
- net +5V: now also TP3.1
- net GND: now also TP4.1
- net at C10.1, C14.1, C15.1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: now also TP5.1
- net at C11.1, C12.1, C13.1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: now also TP6.1
Other:
- note removed: "1.5V"
Changed lines of the file:
@@
 L power:+5V #PWR04
 U 1 1 5DC9E8F1
-P 1500 1150
-F 0 "#PWR04" H 1500 1000 50  0001 C CNN
-F 1 "+5V" H 1515 1323 50  0000 C CNN
-F 2 "" H 1500 1150 50  0001 C CNN
-F 3 "" H 1500 1150 50  0001 C CNN
-	1    1500 1150
+P 1700 1150
+F 0 "#PWR04" H 1700 1000 50  0001 C CNN
+F 1 "+5V" H 1715 1323 50  0000 C CNN
+F 2 "" H 1700 1150 50  0001 C CNN
+F 3 "" H 1700 1150 50  0001 C CNN
+	1    1700 1150
 	1    0    0    -1
 $EndComp
@@
 L power:GND #PWR03
 U 1 1 5DC9E91D
-P 1150 1700
-F 0 "#PWR03" H 1150 1450 50  0001 C CNN
-F 1 "GND" H 1155 1527 50  0000 C CNN
-F 2 "" H 1150 1700 50  0001 C CNN
-F 3 "" H 1150 1700 50  0001 C CNN
-	1    1150 1700
+P 1350 1700
+F 0 "#PWR03" H 1350 1450 50  0001 C CNN
+F 1 "GND" H 1355 1527 50  0000 C CNN
+F 2 "" H 1350 1700 50  0001 C CNN
+F 3 "" H 1350 1700 50  0001 C CNN
+	1    1350 1700
 	1    0    0    -1
 $EndComp
@@
 L power:PWR_FLAG #FLG0105
 U 1 1 5DCE6D49
-P 1200 1250
-F 0 "#FLG0105" H 1200 1325 50  0001 C CNN
-F 1 "PWR_FLAG" H 1200 1424 50  0000 C CNN
-F 2 "" H 1200 1250 50  0001 C CNN
-F 3 "~" H 1200 1250 50  0001 C CNN
-	1    1200 1250
+P 1150 1250
+F 0 "#FLG0105" H 1150 1325 50  0001 C CNN
+F 1 "PWR_FLAG" H 1150 1424 50  0001 C CNN
+F 2 "" H 1150 1250 50  0001 C CNN
+F 3 "~" H 1150 1250 50  0001 C CNN
+	1    1150 1250
 	1    0    0    -1
 $EndComp
@@
 L power:PWR_FLAG #FLG0104
 U 1 1 5DCE9C10
-P 6300 2800
-F 0 "#FLG0104" H 6300 2875 50  0001 C CNN
-F 1 "PWR_FLAG" H 6300 2974 50  0000 C CNN
-F 2 "" H 6300 2800 50  0001 C CNN
-F 3 "~" H 6300 2800 50  0001 C CNN
-	1    6300 2800
+P 5750 2800
+F 0 "#FLG0104" H 5750 2875 50  0001 C CNN
+F 1 "PWR_FLAG" H 5750 2974 50  0001 C CNN
+F 2 "" H 5750 2800 50  0001 C CNN
+F 3 "~" H 5750 2800 50  0001 C CNN
+	1    5750 2800
 	1    0    0    -1
 $EndComp
@@
 L power:PWR_FLAG #FLG0106
 U 1 1 5DD01F1E
-P 5000 2300
-F 0 "#FLG0106" H 5000 2375 50  0001 C CNN
-F 1 "PWR_FLAG" H 5000 2474 50  0000 C CNN
-F 2 "" H 5000 2300 50  0001 C CNN
-F 3 "~" H 5000 2300 50  0001 C CNN
-	1    5000 2300
+P 5600 2300
+F 0 "#FLG0106" H 5600 2375 50  0001 C CNN
+F 1 "PWR_FLAG" H 5600 2474 50  0001 C CNN
+F 2 "" H 5600 2300 50  0001 C CNN
+F 3 "~" H 5600 2300 50  0001 C CNN
+	1    5600 2300
 	1    0    0    -1
 $EndComp
@@
 P 1150 1550
 F 0 "#FLG0107" H 1150 1625 50  0001 C CNN
-F 1 "PWR_FLAG" H 1150 1724 50  0000 C CNN
+F 1 "PWR_FLAG" H 1150 1724 50  0001 C CNN
 F 2 "" H 1150 1550 50  0001 C CNN
 F 3 "~" H 1150 1550 50  0001 C CNN
@@
 Text GLabel 950  1550 0    50   Input ~ 0
 GND
-Text Notes 5150 2250 0    50   ~ 0
-1.5V
 Text GLabel 5000 5100 2    50   Input ~ 0
 VCCIB3
@@
 VJTAG
 Wire Wire Line
-	950  1250 1200 1250
+	950  1250 1150 1250
 Wire Wire Line
 	3700 1250 3700 1500
@@
 	4100 2450 3800 2450
 Wire Wire Line
-	1500 1150 1500 1250
-Wire Wire Line
-	1500 1250 3700 1250
+	1700 1150 1700 1250
+Wire Wire Line
+	1700 1250 1350 1250
 Wire Wire Line
 	3800 2800 3950 2800
@@
 	950  1550 1150 1550
 Wire Wire Line
-	1150 1550 1150 1700
+	1350 1550 1350 1700
 Wire Wire Line
 	5000 2800 5300 2800
@@
 	9100 2700 9100 2800
 Wire Wire Line
-	5000 2300 7150 2300
+	5000 2300 5600 2300
 Wire Wire Line
 	5000 2300 5000 2800
@@
 	4350 5100 4900 5100
 Wire Wire Line
-	1500 1250 1500 5100
-Wire Wire Line
-	1500 5100 2400 5100
+	1700 1250 1700 5100
+Wire Wire Line
+	1700 5100 2400 5100
 Wire Wire Line
 	5000 4900 4900 4900
@@
 Wire Wire Line
 	3250 5600 3250 5650
-Wire Wire Line
-	1200 1250 1500 1250
 Wire Wire Line
 	6300 4050 6300 4100
@@
 Connection ~ 3700 1250
 Connection ~ 4100 2300
-Connection ~ 1500 1250
+Connection ~ 1700 1250
 Connection ~ 4750 2800
 Connection ~ 4750 3100
@@
 Connection ~ 4350 5100
 Connection ~ 4900 5100
-Connection ~ 1200 1250
 Connection ~ 6300 2800
-Connection ~ 5000 2300
 Connection ~ 6300 4100
 Connection ~ 1500 6550
 Connection ~ 3250 5600
 Connection ~ 3200 3150
-Connection ~ 1150 1550
+Connection ~ 1350 1550
 Connection ~ 10350 3600
 Connection ~ 10350 4000
@@
 	1    0    0    -1
 $EndComp
+$Comp
+L Connector:TestPoint TP3
+U 1 1 5DD255AD
+P 1350 1250
+F 0 "TP3" H 1408 1370 50  0000 L CNN
+F 1 "+5V" H 1400 1450 50  0000 L CNN
+F 2 "TestPoint:TestPoint_THTPad_1.5x1.5mm_Drill0.7mm" H 1550 1250 50  0001 C CNN
+F 3 "~" H 1550 1250 50  0001 C CNN
+	1    1350 1250
+	1    0    0    -1
+$EndComp
+$Comp
+L Connector:TestPoint TP4
+U 1 1 5DD257FC
+P 1350 1550
+F 0 "TP4" H 1408 1670 50  0000 L CNN
+F 1 "GND" H 1400 1600 50  0000 L CNN
+F 2 "TestPoint:TestPoint_THTPad_1.5x1.5mm_Drill0.7mm" H 1550 1550 50  0001 C CNN
+F 3 "~" H 1550 1550 50  0001 C CNN
+	1    1350 1550
+	1    0    0    -1
+$EndComp
+Connection ~ 1350 1250
+Wire Wire Line
+	1700 1250 3700 1250
+Connection ~ 1150 1250
+Wire Wire Line
+	1150 1250 1350 1250
+Connection ~ 1150 1550
+Wire Wire Line
+	1150 1550 1350 1550
+$Comp
+L Connector:TestPoint TP5
+U 1 1 5DD3E74F
+P 5000 2300
+F 0 "TP5" H 5058 2420 50  0000 L CNN
+F 1 "1.5V Core" H 5050 2500 50  0000 L CNN
+F 2 "TestPoint:TestPoint_THTPad_1.5x1.5mm_Drill0.7mm" H 5200 2300 50  0001 C CNN
+F 3 "~" H 5200 2300 50  0001 C CNN
+	1    5000 2300
+	1    0    0    -1
+$EndComp
+Connection ~ 5600 2300
+Wire Wire Line
+	5600 2300 7150 2300
+Connection ~ 5000 2300
+$Comp
+L Connector:TestPoint TP6
+U 1 1 5DD451A3
+P 6300 2800
+F 0 "TP6" H 6358 2920 50  0000 L CNN
+F 1 "1.5V PLL" H 6350 3000 50  0000 L CNN
+F 2 "TestPoint:TestPoint_THTPad_1.5x1.5mm_Drill0.7mm" H 6500 2800 50  0001 C CNN
+F 3 "~" H 6500 2800 50  0001 C CNN
+	1    6300 2800
+	1    0    0    -1
+$EndComp
