File: MicroSemi_FPGA_Dev_Board/kicad_board_design/A3P250_Dev_Board/UnitD.sch (KiCad schematic (older format))
At the start: 10 parts, among them J4 Conn_01x20, U1 A3P250, X1 ASE-25MHz

Commit message: Routed, fixed labels, added test points.
Parts:
- added TP1, TP2: VCCIO, TestPoint:TestPoint_THTPad_1.5x1.5mm_Drill0.7mm, symbol Connector:TestPoint
Connections:
- net GND: no longer U1.24 (VMV3)
- net VCCIB3: now also U1.24 (VMV3), TP1.1
- net at J4.11 (Pin_11), U1.10 (GFB1/IO109PDB3), X1.3 (OUT): now also TP2.1
Changed lines of the file:
@@
 	5850 1950 8350 1950
 Wire Wire Line
-	6100 4650 5900 4650
-Wire Wire Line
-	5900 4650 5900 5250
-Wire Wire Line
-	5900 5250 6050 5250
-Wire Wire Line
 	5000 4050 5300 4050
 Wire Wire Line
@@
 	6000 3450 6100 3450
 Wire Wire Line
-	5300 4050 6100 4050
+	5300 4050 5850 4050
 Wire Wire Line
 	5000 3950 6100 3950
@@
 Wire Wire Line
 	5650 5150 5650 5250
-Wire Wire Line
-	5650 5250 5900 5250
-Connection ~ 5900 5250
 Text Notes 4550 4700 0    50   ~ 0
 FPGA\nReset out
@@
 Wire Wire Line
 	3350 5000 3650 5000
+Wire Wire Line
+	5650 5250 6050 5250
+Wire Wire Line
+	5850 4650 5850 4050
+Wire Wire Line
+	5850 4650 6100 4650
+Connection ~ 5850 4050
+Wire Wire Line
+	5850 4050 6100 4050
+$Comp
+L Connector:TestPoint TP1
+U 1 1 5DD218F3
+P 3350 5000
+F 0 "TP1" H 3408 5120 50  0000 L CNN
+F 1 "VCCIO" H 3400 5200 50  0000 L CNN
+F 2 "TestPoint:TestPoint_THTPad_1.5x1.5mm_Drill0.7mm" H 3550 5000 50  0001 C CNN
+F 3 "~" H 3550 5000 50  0001 C CNN
+	1    3350 5000
+	1    0    0    -1
+$EndComp
+$Comp
+L Connector:TestPoint TP2
+U 1 1 5DD21AC8
+P 6500 5400
+F 0 "TP2" H 6558 5520 50  0000 L CNN
+F 1 "VCCIO" H 6550 5600 50  0000 L CNN
+F 2 "TestPoint:TestPoint_THTPad_1.5x1.5mm_Drill0.7mm" H 6700 5400 50  0001 C CNN
+F 3 "~" H 6700 5400 50  0001 C CNN
+	1    6500 5400
+	1    0    0    -1
+$EndComp
+Wire Wire Line
+	5500 5400 6500 5400
+Connection ~ 5500 5400
 $EndSCHEMATC

Commit message: Add solder paste layer.
Parts:
- TP1, TP2: footprint TestPoint:TestPoint_THTPad_1.5x1.5mm_Drill0.7mm -> TestPoint:TestPoint_THTPad_D1.0mm_Drill0.5mm
Changed lines of the file:
@@
 F 0 "TP1" H 3408 5120 50  0000 L CNN
 F 1 "VCCIO" H 3400 5200 50  0000 L CNN
-F 2 "TestPoint:TestPoint_THTPad_1.5x1.5mm_Drill0.7mm" H 3550 5000 50  0001 C CNN
+F 2 "TestPoint:TestPoint_THTPad_D1.0mm_Drill0.5mm" H 3550 5000 50  0001 C CNN
 F 3 "~" H 3550 5000 50  0001 C CNN
 	1    3350 5000
@@
 F 0 "TP2" H 6558 5520 50  0000 L CNN
 F 1 "VCCIO" H 6550 5600 50  0000 L CNN
-F 2 "TestPoint:TestPoint_THTPad_1.5x1.5mm_Drill0.7mm" H 6700 5400 50  0001 C CNN
+F 2 "TestPoint:TestPoint_THTPad_D1.0mm_Drill0.5mm" H 6700 5400 50  0001 C CNN
 F 3 "~" H 6700 5400 50  0001 C CNN
 	1    6500 5400
