File: MicroSemi_FPGA_Dev_Board/kicad_base_board_design/BaseBoard/UnitE.sch (KiCad schematic (older format))
At the start: 35 parts, among them U1 A3P250, U2 LTC3561A, U3 LT1962-3.3

Commit message: Add solder paste layer.
Parts:
- renumbered C6 to C?, C10 to C?, C9 to C?, C4 to C?, C2 to C?, C13 to C?, C12 to C?, C15 to C?, C17 to C?, C21 to C?, C19 to C?, C14 to C?, C16 to C?, C20 to C?, C18 to C?, C3 to C?, C11 to C?, C8 to C?, C7 to C?, C5 to C?, L1 to L?, L2 to L?, R5 to R?, R4 to R?, R3 to R?, R2 to R?, TP3 to TP?, TP4 to TP?, TP5 to TP?, TP6 to TP?, U2 to U?, U1 to U?, U3 to U?
