File: oresat-gps-card/oresat-gps-card-sch-max2771.kicad_sch (KiCad schematic)
At the start: 35 parts, among them U13 MAX2769, U24 D32G-016.368M, U28 LT1719IS6

Commit message: BOM Update
Parts:
- C100, C102, C115, C117, C119, C121, C123, C125, C53, C79: DIS (none) -> DigiKey; DPN (none) -> 399-6856-1-ND; MFR (none) -> KEMET; MPN (none) -> C0603C104K5RACAUTO
- C86: DIS (none) -> DigiKey; DPN (none) -> 490-GRM1885C1H1R7BA01DCT-ND; MFR (none) -> Murata Electronics; MPN (none) -> GRM1885C1H1R7BA01D
- C88: DIS (none) -> DigiKey; DPN (none) -> 399-12983-1-ND; MFR (none) -> KEMET; MPN (none) -> C0603C103J5RACAUTO
- C92: DIS (none) -> DigiKey; DPN (none) -> 490-17767-1-ND; MFR (none) -> Murata Electronics; MPN (none) -> GCM1885C2A270JA16D
- R81: DIS (none) -> DigiKey; DPN (none) -> 738-RAVF164DJT20K0CT-ND; MFR (none) -> Stackpole Electronics; MPN (none) -> RAVF164DJT20K0

Commit message: Large BOM changes for v1.2, no changes to PCB
Parts:
- FL2: DIS (none) -> DigiKey; DPN (none) -> 478-SF14-1575F5UUR1CT-ND; MFR (none) -> KYOCERA AVX; MPN (none) -> SF14-1575F5UUR1
- R52: value 1k -> 4.7k; DPN RMCF0603FT2K70CT-ND -> RMCF0603FT4K70CT-ND; MPN RMCF0603FT1K00 -> RMCF0603FT4K70
Changed lines of the file:
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@@
 			)
 		)
-		(property "Value" "1k"
+		(property "Value" "4.7k"
 			(at 167.386 173.736 0)
 			(show_name no)
@@
 			)
 		)
-		(property "Description" "1 kOhms ±1% 0.1W, 1/10W Chip Resistor 0603 (1608 Metric) Automotive AEC-Q200 Thick Film"
+		(property "Description" "4.7 kOhms ±1% 0.1W, 1/10W Chip Resistor 0603 (1608 Metric) Automotive AEC-Q200 Thick Film"
 			(at 171.45 172.72 0)
 			(hide yes)
@@
 			)
 		)
-		(property "DPN" "RMCF0603FT2K70CT-ND"
+		(property "DPN" "RMCF0603FT4K70CT-ND"
 			(at 171.45 172.72 0)
 			(hide yes)
@@
 			)
 		)
-		(property "MPN" "RMCF0603FT1K00"
+		(property "MPN" "RMCF0603FT4K70"
 			(at 171.45 172.72 0)
 			(hide yes)
@@
 			)
 		)
-		(property "Datasheet" "https://global.kyocera.com/prdct/electro/product/pdf/sf14_gnss.pdf"
+		(property "Datasheet" "https://ele.kyocera.com/assets/products/saw-device/specification/SF14-1575F5UUR1_DS.pdf"
 			(at 144.78 160.02 0)
 			(hide yes)
@@
 			)
 		)
-		(property "Description" ""
+		(property "Description" "1.57542GHz Frequency GPS RF SAW Filter (Surface Acoustic Wave) 0.45dB 2MHz Bandwidth 5-SMD, No Lead"
+			(at 144.78 160.02 0)
+			(hide yes)
+			(show_name no)
+			(do_not_autoplace no)
+			(effects
+				(font
+					(size 1.27 1.27)
+				)
+			)
+		)
+		(property "DIS" "DigiKey"
+			(at 144.78 160.02 0)
+			(hide yes)
+			(show_name no)
+			(do_not_autoplace no)
+			(effects
+				(font
+					(size 1.27 1.27)
+				)
+			)
+		)
+		(property "DPN" "478-SF14-1575F5UUR1CT-ND"
+			(at 144.78 160.02 0)
+			(hide yes)
+			(show_name no)
+			(do_not_autoplace no)
+			(effects
+				(font
+					(size 1.27 1.27)
+				)
+			)
+		)
+		(property "MFR" "KYOCERA AVX"
+			(at 144.78 160.02 0)
+			(hide yes)
+			(show_name no)
+			(do_not_autoplace no)
+			(effects
+				(font
+					(size 1.27 1.27)
+				)
+			)
+		)
+		(property "MPN" "SF14-1575F5UUR1"
 			(at 144.78 160.02 0)
 			(hide yes)
@@
 		)
 		(property "Value" "GND"
-			(at 166.37 179.07 0)
+			(at 169.672 180.086 0)
 			(show_name no)
 			(do_not_autoplace no)
@@
 		)
 		(property "Value" "GND"
-			(at 194.31 177.8 0)
+			(at 197.358 179.07 0)
 			(show_name no)
 			(do_not_autoplace no)
@@
 		(in_pos_files yes)
 		(dnp no)
-		(fields_autoplaced yes)
 		(property "Reference" "#GND0248"
 			(at 308.61 149.86 0)
@@
 		)
 		(property "Value" "GND"
-			(at 311.15 144.7799 0)
+			(at 307.086 147.32 0)
 			(show_name no)
 			(do_not_autoplace no)
@@
 		(in_pos_files yes)
 		(dnp no)
-		(fields_autoplaced yes)
 		(property "Reference" "#GND0251"
 			(at 254 156.21 0)
@@
 		)
 		(property "Value" "GND"
-			(at 256.54 151.1299 0)
+			(at 252.222 153.416 0)
 			(show_name no)
 			(do_not_autoplace no)

Commit message: Updated Layout
Changes to BOM. Changes to footprint assignments.
Parts:
- R81: DPN 738-RAVF164DJT20K0CT-ND -> RMCF0603FT20K0CT-ND; MPN RAVF164DJT20K0 -> RMCF0603FT20K0
Changed lines of the file:
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@@
 			)
 		)
-		(property "Datasheet" "https://www.seielect.com/catalog/SEI-RAVF.pdf"
+		(property "Datasheet" "https://www.seielect.com/catalog/SEI-RMCF_RMCP.pdf"
 			(at 210.82 184.15 0)
 			(hide yes)
@@
 			)
 		)
-		(property "Description" "20k Ohm ±5% 100mW Power Per Element Isolated 4 Resistor Network/Array ±200ppm/°C 1206 (3216 Metric), Convex, Long Side Terminals"
+		(property "Description" "20 kOhms ±1% 0.1W, 1/10W Chip Resistor 0603 (1608 Metric) Automotive AEC-Q200 Thick Film"
 			(at 210.82 184.15 0)
 			(hide yes)
@@
 			)
 		)
-		(property "DPN" "738-RAVF164DJT20K0CT-ND"
+		(property "DPN" "RMCF0603FT20K0CT-ND"
 			(at 210.82 184.15 90)
 			(hide yes)
@@
 			)
 		)
-		(property "MPN" "RAVF164DJT20K0"
+		(property "MPN" "RMCF0603FT20K0"
 			(at 210.82 184.15 90)
 			(hide yes)

Commit message: Upped to v1.3.
Fixed backward EEPROM programming pin, fixed potential boot error with missing PMIC connections, fixed some power domain issues.
Parts:
- FL2: value SF14-1575F5UUA1 -> SF14-1575F5UUR1
- L4: MPN FIXED IND 5.6NH 800MA 200 MOHM -> LQG18HN5N6S00D
Connections:
- net 2.85VD: now also R51.1, R88.2
- net GND: no longer R51.1, R88.2
Other:
- note added: "PULL LOW WHEN NOT POWERING GPS DOMAIN."
- moved on the sheet: R88

Commit message: routine push
Parts:
- U24: footprint oresat-ics:U-Connor-Winfield-D32G-016368M -> oresat-footprints:U-Connor-Winfield-D32G-016368M
Other:
- moved on the sheet: R86, R88

Commit message: Schematic and layout changes
Updated OPD schematic and layout. Updated schematic and layout to include uart.
Parts:
- U24: DIS DigiKey -> (none); DPN CW660CT-ND -> (none); MFR Connor Winfield -> (none); MPN D32G-016.368M -> (none)
- U28: DIS DigiKey -> (none); DPN 505-LT1719IS6#TRMPBFCT-ND -> (none); MFR Analog Devices Inc. -> (none); MPN LT1719IS6#TRMPBF -> (none)
Changed lines of the file:
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@@
 	)
 	(symbol
-		(lib_name "LT1719IS6_1")
 		(lib_id "oresat-ics:LT1719IS6")
 		(at 274.32 137.16 0)
@@
 		(dnp no)
 		(property "Reference" "U28"
-			(at 275.844 133.858 0)
+			(at 274.32 137.16 0)
+			(hide yes)
 			(show_name no)
 			(do_not_autoplace no)
@@
 		)
 		(property "Value" "LT1719IS6"
-			(at 273.05 141.986 0)
+			(at 274.32 142.24 0)
+			(hide yes)
 			(show_name no)
 			(do_not_autoplace no)
 			(effects
 				(font
-					(size 1.27 1.27)
+					(size 1.778 1.5113)
 				)
 				(justify left bottom)
@@
 			)
 		)
-		(property "DIS" "DigiKey"
-			(at 274.32 137.16 0)
-			(hide yes)
-			(show_name no)
-			(do_not_autoplace no)
-			(effects
-				(font
-					(size 1.27 1.27)
-				)
-			)
-		)
-		(property "DPN" "505-LT1719IS6#TRMPBFCT-ND"
-			(at 274.32 137.16 0)
-			(hide yes)
-			(show_name no)
-			(do_not_autoplace no)
-			(effects
-				(font
-					(size 1.27 1.27)
-				)
-			)
-		)
-		(property "MFR" "Analog Devices Inc."
-			(at 274.32 137.16 0)
-			(hide yes)
-			(show_name no)
-			(do_not_autoplace no)
-			(effects
-				(font
-					(size 1.27 1.27)
-				)
-			)
-		)
-		(property "MPN" "LT1719IS6#TRMPBF"
-			(at 274.32 137.16 0)
-			(hide yes)
-			(show_name no)
-			(do_not_autoplace no)
-			(effects
-				(font
-					(size 1.27 1.27)
-				)
-			)
-		)
 		(pin "1"
 		)
@@
 		(fields_autoplaced yes)
 		(property "Reference" "U24"
-			(at 276.86 151.13 0)
+			(at 276.86 149.86 0)
 			(show_name no)
 			(do_not_autoplace no)
 			(effects
 				(font
-					(size 1.27 1.27)
+					(size 1.27 1.0795)
 				)
 			)
 		)
 		(property "Value" "D32G-016.368M"
-			(at 276.86 153.67 0)
+			(at 276.86 152.4 0)
 			(show_name no)
 			(do_not_autoplace no)
 			(effects
 				(font
-					(size 1.27 1.27)
+					(size 1.27 1.0795)
 				)
 			)
 		)
 		(property "Footprint" "oresat-footprints:U-Connor-Winfield-D32G-016368M"
-			(at 276.86 148.082 0)
+			(at 274.828 144.272 0)
 			(hide yes)
 			(show_name no)
@@
 		)
 		(property "Datasheet" "http://www.conwin.com/datasheets/tx/tx240.pdf"
-			(at 276.86 146.304 0)
+			(at 275.59 146.558 0)
 			(hide yes)
 			(show_name no)
@@
 		)
 		(property "Description" "16.368 MHz TCXO, 4-pin 3.2x2.5mm"
-			(at 276.86 160.02 0)
-			(hide yes)
-			(show_name no)
-			(do_not_autoplace no)
-			(effects
-				(font
-					(size 1.27 1.27)
-				)
-			)
-		)
-		(property "DIS" "DigiKey"
-			(at 276.86 160.02 0)
-			(hide yes)
-			(show_name no)
-			(do_not_autoplace no)
-			(effects
-				(font
-					(size 1.27 1.27)
-				)
-			)
-		)
-		(property "DPN" "CW660CT-ND"
-			(at 276.86 160.02 0)
-			(hide yes)
-			(show_name no)
-			(do_not_autoplace no)
-			(effects
-				(font
-					(size 1.27 1.27)
-				)
-			)
-		)
-		(property "MFR" "Connor Winfield"
-			(at 276.86 160.02 0)
-			(hide yes)
-			(show_name no)
-			(do_not_autoplace no)
-			(effects
-				(font
-					(size 1.27 1.27)
-				)
-			)
-		)
-		(property "MPN" "D32G-016.368M"
-			(at 276.86 160.02 0)
+			(at 276.86 141.478 0)
 			(hide yes)
 			(show_name no)
@@
 			)
 		)
-		(property "Description" "Comparator Standard (General Purpose) CMOS, Rail-to-Rail, TTL TSOT-23-6"
+		(property "Description" "General Purpose Comparator, SOT-23-6"
 			(at 306.07 137.16 0)
 			(hide yes)
