File: oresat-gps-card/oresat-gps-card-sch-power.kicad_sch (KiCad schematic)
At the start: 102 parts, among them Q1 DMP2240UDM, Q10 DMP3050LVT-7, Q11 DMP3050LVT-7, Q12 PMV45EN, Q8 PMV45EN, U2 MAX7310ATE, U20 TS5A21366DCUR, U21 MAX4211FETE, U3 MIC842LYC5, U4 MIC842LYC5, U6 LTC3624

Commit message: Routine Push
Lots of footprint changes
Parts:
- removed D10: MBR0520L, Diode_SMD:D_SOD-123, symbol Device:D_Small
- removed Q1: DMP2240UDM, Package_TO_SOT_SMD:SOT-23-6, symbol Device:Q_Dual_PMOS_G1S2G2D2S1D1
- removed Q10, Q11: DMP3050LVT-7, Package_TO_SOT_SMD:TSOT-23-6, symbol oresat-transistors:DMP3050LVT-7
- removed Q12: PMV45EN, Package_TO_SOT_SMD:SOT-23, symbol Transistor_FET:Q_NMOS_GSD
- removed TP6, TP7: 1x01, oresat-misc:TestPoint-0.75mm-th, symbol oresat-misc:Test-Point-0.75mm-th
- added Q1: DMP2110UVTQ-7, Package_TO_SOT_SMD:SOT-23-6, symbol Transistor_FET:Q_Dual_PMOS_G1S2G2D2S1D1
- added Q2, Q7: DMPH2040UVTQ-7, Package_TO_SOT_SMD:TSOT-23-6, symbol oresat-transistors:DMP3050LVT-7
- added Q9: DMN2050LQ-7, Package_TO_SOT_SMD:SOT-23, symbol Transistor_FET:Q_NMOS_GSD
- C1, C15, C2, C3, C4, C5, C7: footprint Capacitor_SMD:C_0603_1608Metric -> oresat-passives:0603-C-NOSILK
- C10: value 2u2 -> 2.2u; footprint Capacitor_SMD:C_0603_1608Metric -> oresat-passives:0603-C-NOSILK
- Q8: value PMV45EN -> DMN2050LQ-7; DPN 1727-2307-1-ND -> 31-DMN2050LQ-7CT-ND; MFR Nexperia -> Diodes Incorporated; MPN PMV45EN2R -> DMN2050LQ-7
- R1, R10, R13, R14, R15, R17, R18, R19, R2, R22, R28, R29, R33, R59, R6, R9: footprint Resistor_SMD:R_0603_1608Metric -> oresat-passives:0603-C-NOSILK
- R11: value 100 -> 10; footprint Resistor_SMD:R_0603_1608Metric -> oresat-passives:0603-C-NOSILK
- R12, R16, R20, R21, R3, R4, R5, R7, R8: value NP -> 100
- R99: footprint Resistor_SMD:R_1206_3216Metric -> oresat-passives:1206-C
Connections:
- net VPD is gone; now on net 3.3V: C3.2, C4.2, C5.1, D9.1 (K), R108.2, R17.2, R18.2, R19.2, R22.1, R4.2, R8.2, TP3.1, U2.14 (V+), U3.5 (VDD), U4.5 (VDD)
- net CB_CTRL: now also Q9.1 (G)
- net GND: now also Q9.2 (S)
- net PEN-SCL-FILT: now also Q1.4 (D)
- net PEN-SDA-FILT: now also Q1.6 (D)
- net VBUS: now also Q7.4 (S)
- net VBUSP: now also Q2.1 (D), Q2.2 (D), Q2.5 (D), Q2.6 (D)
- net ~{FAULT}: now also Q9.3 (D)
- net at C63.1, R105.1, R106.2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: now also Q2.3 (G)
- net at C63.2, R105.2, R99.2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: now also Q2.4 (S)
- net at C59.1, R99.1, U21.16 (RS+): now also Q7.1 (D), Q7.2 (D), Q7.5 (D), Q7.6 (D)
- net at Q8.3 (D), R64.1: now also Q7.3 (G)
- net at R10.2: now also Q1.1 (G)
- net at R1.2: now also Q1.2 (S)
- net at R9.2: now also Q1.3 (G)
- net at R2.2: now also Q1.5 (S)

Commit message: Routine Push
Parts:
- removed TP33, TP36, TP38: Test-Point, oresat-misc:TestPoint-0.75mm-th, symbol oresat-misc:Test-Point-0.75mm-th
- renumbered D13 to D1, D9 to D10, D5 to D2, D2 to D3
