File: oresat-gps-card/oresat-gps-card-sch-power.kicad_sch (KiCad schematic)
At the start: 96 parts, among them Q1 DMP2110UVTQ-7, Q2 DMPH2040UVTQ-7, Q7 DMPH2040UVTQ-7, Q8 DMN2050LQ-7, Q9 DMN2050LQ-7, U2 MAX7310ATE, U20 TS5A21366DCUR, U21 MAX4211FETE, U3 MIC842LYC5, U4 MIC842LYC5, U6 LTC3624

Commit message: Review Push
Still several line items to fix
Parts:
- removed TP34, TP41: Test-Point, oresat-misc:TestPoint-0.75mm-th, symbol oresat-misc:Test-Point-0.75mm-th
Changed lines of the file:
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@@
 	)
 	(junction
-		(at 189.23 54.61)
-		(diameter 0)
-		(color 0 0 0 0)
-	)
-	(junction
 		(at 200.66 215.9)
 		(diameter 0)
@@
 	)
 	(junction
-		(at 354.33 91.44)
-		(diameter 0)
-		(color 0 0 0 0)
-	)
-	(junction
 		(at 284.48 59.69)
 		(diameter 0)
@@
 	)
 	(symbol
-		(lib_id "oresat-misc:Test-Point-0.75mm-th")
-		(at 189.23 54.61 0)
-		(unit 1)
-		(body_style 1)
-		(exclude_from_sim no)
-		(in_bom no)
-		(on_board yes)
-		(in_pos_files yes)
-		(dnp no)
-		(property "Reference" "TP34"
-			(at 183.388 55.118 0)
-			(show_name no)
-			(do_not_autoplace no)
-			(effects
-				(font
-					(size 1.27 1.0795)
-				)
-				(justify left bottom)
-			)
-		)
-		(property "Value" "Test-Point"
-			(at 189.23 46.99 0)
-			(hide yes)
-			(show_name no)
-			(do_not_autoplace no)
-			(effects
-				(font
-					(size 1.27 1.27)
-				)
-			)
-		)
-		(property "Footprint" "oresat-misc:TestPoint-0.75mm-th"
-			(at 189.23 44.45 0)
-			(hide yes)
-			(show_name no)
-			(do_not_autoplace no)
-			(effects
-				(font
-					(size 1.27 1.27)
-				)
-			)
-		)
-		(property "Datasheet" ""
-			(at 189.23 54.61 0)
-			(hide yes)
-			(show_name no)
-			(do_not_autoplace no)
-			(effects
-				(font
-					(size 1.27 1.27)
-				)
-			)
-		)
-		(property "Description" "0.75 mm TH test point; good for scope probes and jumpers"
-			(at 189.23 54.61 0)
-			(hide yes)
-			(show_name no)
-			(do_not_autoplace no)
-			(effects
-				(font
-					(size 1.27 1.27)
-				)
-			)
-		)
-		(pin "1"
-		)
-		(instances
-			(project "oresat-gps-card"
-				(path "/65d12cdd-c326-4033-9053-c59fa4e0b25e/2134bb9a-062c-4e32-a41e-d15ce3545372"
-					(reference "TP34")
-					(unit 1)
-				)
-			)
-		)
-	)
-	(symbol
 		(lib_id "power:PWR_FLAG")
 		(at 250.19 215.9 270)
@@
 					(unit 1)
 				)
-			)
-		)
-	)
-	(symbol
-		(lib_id "oresat-misc:Test-Point-0.75mm-th")
-		(at 354.33 91.44 0)
-		(unit 1)
-		(body_style 1)
-		(exclude_from_sim no)
-		(in_bom no)
-		(on_board yes)
-		(in_pos_files yes)
-		(dnp no)
-		(property "Reference" "TP41"
-			(at 355.854 92.202 0)
-			(show_name no)
-			(do_not_autoplace no)
-			(effects
-				(font
-					(size 1.27 1.0795)
-				)
-				(justify left bottom)
-			)
-		)
-		(property "Value" "Test-Point"
-			(at 354.33 83.82 0)
-			(hide yes)
-			(show_name no)
-			(do_not_autoplace no)
-			(effects
-				(font
-					(size 1.27 1.27)
-				)
-			)
-		)
-		(property "Footprint" "oresat-misc:TestPoint-0.75mm-th"
-			(at 354.33 81.28 0)
-			(hide yes)
-			(show_name no)
-			(do_not_autoplace no)
-			(effects
-				(font
-					(size 1.27 1.27)
-				)
-			)
-		)
-		(property "Datasheet" ""
-			(at 354.33 91.44 0)
-			(hide yes)
-			(show_name no)
-			(do_not_autoplace no)
-			(effects
-				(font
-					(size 1.27 1.27)
-				)
-			)
-		)
-		(property "Description" "0.75 mm TH test point; good for scope probes and jumpers"
-			(at 354.33 91.44 0)
-			(hide yes)
-			(show_name no)
-			(do_not_autoplace no)
-			(effects
-				(font
-					(size 1.27 1.27)
-				)
-			)
-		)
-		(pin "1"
-		)
-		(instances
-			(project "oresat-gps-card"
-				(path "/65d12cdd-c326-4033-9053-c59fa4e0b25e/2134bb9a-062c-4e32-a41e-d15ce3545372"
-					(reference "TP41")
-					(unit 1)
-				)

Commit message: Routine Push
Parts:
- C1, C2: DIS (none) -> DigiKey; DPN (none) -> 490-GRT188R71E105KE13DCT-ND; MFR (none) -> Murata Electronics; MPN (none) -> GRT188R71E105KE13D
- C10: DIS (none) -> DigiKey; DPN (none) -> 490-GRT188C71E225KE13DCT-ND; MFR (none) -> Murata Electronics; MPN (none) -> GRT188C71E225KE13D
- C7: DIS (none) -> DigiKey; DPN (none) -> 490-GRT21BC71E106KE13KCT-ND; MFR (none) -> Murata Electronics; MPN (none) -> GRT21BC71E106KE13K
- D3: DIS (none) -> DigiKey; DPN (none) -> 732-4971-1-ND; MFR (none) -> Wurth; MPN (none) -> 150060GS75000
- L1: value 3u3 -> 3.3u
- R1, R13, R17, R2, R6: DIS (none) -> DigiKey; DPN (none) -> RMCF0603FT100RCT-ND; MFR (none) -> Stackpole Electronics; MPN (none) -> RMCF0603FT100R
- R10, R9: DIS (none) -> DigiKey; DPN (none) -> RMCF0603FT665KCT-ND; MFR (none) -> Stackpole Electronics; MPN (none) -> RMCF0603FT665K
- R100, R101, R102, R105, R106, R107, R108, R109, R64, R93, R96, R97, R98, R99: MFR Stackpole Electronics Inc -> Stackpole Electronics
- R11: DIS (none) -> DigiKey; DPN (none) -> RMCF0603FT10R0CT-ND; MFR (none) -> Stackpole Electronics; MPN (none) -> RMCF0603FT10R0
- R14, R15: DIS (none) -> DigiKey; DPN (none) -> RMCF0603FT330KCT-ND; MFR (none) -> Stackpole Electronics; MPN (none) -> RMCF0603FT330K
- R18, R19: DIS (none) -> DigiKey; DPN (none) -> RMCF0603FT1M00CT-ND; MFR (none) -> Stackpole Electronics; MPN (none) -> RMCF0603FT1M00
- R22, R33, R59: DIS (none) -> DigiKey; DPN (none) -> RMCF0603FT10K0CT-ND; MFR (none) -> Stackpole Electronics; MPN (none) -> RMCF0603FT10K0
- R28, R29: DIS (none) -> DigiKey; DPN (none) -> RMCF0603FT100KCT-ND; MFR (none) -> Stackpole Electronics; MPN (none) -> RMCF0603FT100K
- R92, R94, R95: DPN RMCF0603FT1K00CT-ND -> RMCF0603FT2K70CT-ND; MFR Stackpole Electronics Inc -> Stackpole Electronics
- U2: DIS (none) -> DigiKey; DPN (none) -> MAX7310ATE+-ND; MFR (none) -> Analog Devices; MPN (none) -> MAX7310ATE+
- U3, U4: DIS (none) -> DigiKey; DPN (none) -> 576-2927-1-ND; MFR (none) -> Microchip; MPN (none) -> MIC842LYC5-TR
- U6: DIS (none) -> DigiKey; DPN (none) -> 1676-1002-ND

Commit message: Routine Push
Parts:
- L1: footprint oresat-passives:L_ECS-MPI4040 -> oresat-passives:L_ECS_MPIP0420; DIS (none) -> DigiKey; DPN (none) -> 50-ECS-MPIP0420-3R3MCCT-ND; MPN ECS-MPI4040R3-3R3-R -> ECS-MPIP0420-3R3MC
Changed lines of the file:
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@@
 			)
 		)
-		(property "Footprint" "oresat-passives:L_ECS-MPI4040"
+		(property "Footprint" "oresat-passives:L_ECS_MPIP0420"
 			(at 231.14 215.9 0)
 			(hide yes)
@@
 			)
 		)
-		(property "Datasheet" "https://ecsxtal.com/store/pdf/ECS-MPI4040.pdf"
+		(property "Datasheet" "https://ecsxtal.com/store/pdf/ECS-MPIP0420.pdf"
 			(at 231.14 215.9 0)
 			(hide yes)
@@
 			)
 		)
-		(property "Description" "FIXED IND 3.3UH 3A 60 MOHM SMD"
+		(property "Description" "3.3 µH Shielded Molded Inductor 3 A 87mOhm Max Nonstandard"
 			(at 231.14 215.9 90)
 			(hide yes)
@@
 			)
 		)
-		(property "MPN" "ECS-MPI4040R3-3R3-R"
+		(property "MPN" "ECS-MPIP0420-3R3MC"
 			(at 231.14 215.9 90)
 			(hide yes)
+			(show_name no)
+			(do_not_autoplace no)
+			(effects
+				(font
+					(size 1.27 1.27)
+				)
+			)
+		)
+		(property "DIS" "DigiKey"
+			(at 231.14 215.9 90)
+			(hide yes)
+			(show_name no)
+			(do_not_autoplace no)
+			(effects
+				(font
+					(size 1.27 1.27)
+				)
+			)
+		)
+		(property "DPN" "50-ECS-MPIP0420-3R3MCCT-ND"
+			(at 231.14 215.9 90)
+			(hide yes)

Commit message: ERC and DRC cleaneup
Fixed symbols, fixed footprints, changed DRC rules to reduce errors,
updated footprints, mostly done.
Parts:
- removed D10: MBR0520L, Diode_SMD:D_SOD-123, symbol Device:D_Small
- D1: value AMBER -> AMB
- L1: footprint oresat-passives:L_ECS_MPIP0420 -> oresat-passives:L_ECS-MPI4040
- R101, R102: value 0 -> 100
- R109: value 2.7k -> 10k; DPN RMCF0603FT2K70CT-ND -> (none); MPN RMCF0603FT2K70 -> (none)
- R11: value 10 -> 100; DPN RMCF0603FT10R0CT-ND -> (none); MPN RMCF0603FT10R0 -> (none)
- R92: value 1k -> 4.7k; DPN RMCF0603FT2K70CT-ND -> (none); MPN RMCF0603FT1K00 -> (none)
- R94, R95: value 1k -> 100; DPN RMCF0603FT2K70CT-ND -> (none); MPN RMCF0603FT1K00 -> (none)
- R99: value 100m -> 30m; DPN CSR1206FKR100CT-ND -> (none); MPN CSR1206FKR100 -> (none)
Connections:
- net 3.3V is gone; now on net VPD: C3.2, C4.2, C5.1, R108.2, R17.2, R18.2, R19.2, R22.1, R4.2, R8.2, TP3.1, U2.14 (V+), U3.5 (VDD), U4.5 (VDD)
- net VPD: now reaches R11.2
- net BOOTCFG: now reaches TP13.1, U2.10 (IO5)
- net 411-IOUT: no longer names the net of R102.2, U21.14 (IOUT)
- net MCU-UART-RX renamed UART0_RX
- net MCU-UART-TX renamed UART0_TX
Other:
- note added: "Feedback settings trips at 985m mA"
- note removed: "Feedback settings trips at 295m mA"
- note removed: "OreSat Power Enable (PEN)"
- company: (none) -> Portland State Aerospace Society

Commit message: Review commit
Parts:
- R12, R16, R20, R21, R3, R4, R5, R7, R8: footprint Resistor_SMD:R_0603_1608Metric -> oresat-passives:0603-C-NOSILK
Changed lines of the file:
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@@
 			)
 		)
-		(property "Footprint" "Resistor_SMD:R_0603_1608Metric"
+		(property "Footprint" "oresat-passives:0603-C-NOSILK"
 			(at 46.736 76.454 90)
 			(hide yes)
@@
 			)
 		)
-		(property "Footprint" "Resistor_SMD:R_0603_1608Metric"
+		(property "Footprint" "oresat-passives:0603-C-NOSILK"
 			(at 51.816 76.454 90)
 			(hide yes)
@@
 			)
 		)
-		(property "Footprint" "Resistor_SMD:R_0603_1608Metric"
+		(property "Footprint" "oresat-passives:0603-C-NOSILK"
 			(at 77.216 76.454 90)
 			(hide yes)
@@
 			)
 		)
-		(property "Footprint" "Resistor_SMD:R_0603_1608Metric"
+		(property "Footprint" "oresat-passives:0603-C-NOSILK"
 			(at 67.056 76.454 90)
 			(hide yes)
@@
 			)
 		)
-		(property "Footprint" "Resistor_SMD:R_0603_1608Metric"
+		(property "Footprint" "oresat-passives:0603-C-NOSILK"
 			(at 46.736 86.614 90)
 			(hide yes)
@@
 			)
 		)
-		(property "Footprint" "Resistor_SMD:R_0603_1608Metric"
+		(property "Footprint" "oresat-passives:0603-C-NOSILK"
 			(at 82.296 86.614 90)
 			(hide yes)
@@
 			)
 		)
-		(property "Footprint" "Resistor_SMD:R_0603_1608Metric"
+		(property "Footprint" "oresat-passives:0603-C-NOSILK"
 			(at 61.976 86.614 90)
 			(hide yes)
@@
 			)
 		)
-		(property "Footprint" "Resistor_SMD:R_0603_1608Metric"
+		(property "Footprint" "oresat-passives:0603-C-NOSILK"
 			(at 61.976 76.454 90)
 			(hide yes)
@@
 			)
 		)
-		(property "Footprint" "Resistor_SMD:R_0603_1608Metric"
+		(property "Footprint" "oresat-passives:0603-C-NOSILK"
 			(at 82.296 76.454 90)
 			(hide yes)

Commit message: Last of the GPS card cleanup
    Better plains in the RF section, lots of shortening and straitening, cleaned up all ERC and DRCs.
Parts:
- added C52: 22u, Capacitor_SMD:C_1206_3216Metric, symbol Device:C
Connections:
- net 5V: now also C52.1
- net GND: now also C52.2
Other:
- note added: "GPS Card address is 0x19"
- note added: "OreSat Power Domain (OPD) Power Supply (3.3V)"
- note removed: "Address selection for Card (See MAX7310 datasheet)"
- note removed: "OreSat Power Domain (OPD) Power Supply (3.3V) Address 0011001 or 19"
- moved on the sheet: D3, R33

Commit message: BOM Update
Parts:
- C15, C3, C4, C5: DIS (none) -> DigiKey; DPN (none) -> 399-6856-1-ND; MFR (none) -> KEMET; MPN (none) -> C0603C104K5RACAUTO
- C63: DPN 399-6851-1-ND -> 399-12983-1-ND; MPN C0603C103K5RACAUTO -> C0603C103J5RACAUTO
- R92: DPN (none) -> RMCF0603FT4K70CT-ND; MPN (none) -> RMCF0603FT4K70
- R99: DPN (none) -> CSR1206FK30L0CT-ND; MPN (none) -> CSR1206FK30L0
Changed lines of the file:
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@@
 			)
 		)
-		(property "Description" "10000 pF ±10% 50V Ceramic Capacitor X7R 0603 (1608 Metric)"
+		(property "Description" "10000 pF ±5% 50V Ceramic Capacitor X7R 0603 (1608 Metric)"
 			(at 326.39 44.45 0)
 			(hide yes)
@@
 			)
 		)
-		(property "DPN" "399-6851-1-ND"
+		(property "DPN" "399-12983-1-ND"
 			(at 326.39 44.45 0)
 			(hide yes)
@@
 			)
 		)
-		(property "MPN" "C0603C103K5RACAUTO"
+		(property "MPN" "C0603C103J5RACAUTO"
 			(at 326.39 44.45 0)
 			(hide yes)
@@
 			)
 		)
-		(property "Datasheet" ""
+		(property "Datasheet" "https://search.kemet.com/download/specsheet/C0603C104K5RACAUTO"
 			(at 119.38 99.06 0)
 			(hide yes)
@@
 			)
 		)
-		(property "Description" "Unpolarized capacitor"
+		(property "Description" "0.1 µF ±10% 50V Ceramic Capacitor X7R 0603 (1608 Metric)"
 			(at 119.38 99.06 0)
 			(hide yes)
@@
 			)
 		)
+		(property "DIS" "DigiKey"
+			(at 119.38 99.06 90)
+			(hide yes)
+			(show_name no)
+			(do_not_autoplace no)
+			(effects
+				(font
+					(size 1.27 1.27)
+				)
+			)
+		)
+		(property "DPN" "399-6856-1-ND"
+			(at 119.38 99.06 90)
+			(hide yes)
+			(show_name no)
+			(do_not_autoplace no)
+			(effects
+				(font
+					(size 1.27 1.27)
+				)
+			)
+		)
+		(property "MFR" "KEMET"
+			(at 119.38 99.06 90)
+			(hide yes)
+			(show_name no)
+			(do_not_autoplace no)
+			(effects
+				(font
+					(size 1.27 1.27)
+				)
+			)
+		)
+		(property "MPN" "C0603C104K5RACAUTO"
+			(at 119.38 99.06 90)
+			(hide yes)
+			(show_name no)
+			(do_not_autoplace no)
+			(effects
+				(font
+					(size 1.27 1.27)
+				)
+			)
+		)
 		(pin "1"
 		)
@@
 			)
 		)
-		(property "Datasheet" ""
+		(property "Datasheet" "https://search.kemet.com/download/specsheet/C0603C104K5RACAUTO"
 			(at 247.65 222.25 0)
 			(hide yes)
@@
 			)
 		)
-		(property "Description" "Unpolarized capacitor"
+		(property "Description" "0.1 µF ±10% 50V Ceramic Capacitor X7R 0603 (1608 Metric)"
 			(at 247.65 222.25 0)
 			(hide yes)
@@
 			)
 		)
-		(property "MPN" ""
+		(property "MPN" "C0603C104K5RACAUTO"
+			(at 247.65 222.25 0)
+			(hide yes)
+			(show_name no)
+			(do_not_autoplace no)
+			(effects
+				(font
+					(size 1.27 1.27)
+				)
+			)
+		)
+		(property "MFR" "KEMET"
 			(at 247.65 222.25 0)
 			(hide yes)
@@
 			)
 		)
-		(property "MFR" ""
+		(property "DIS" "DigiKey"
+			(at 247.65 222.25 0)
+			(hide yes)
+			(show_name no)
+			(do_not_autoplace no)
+			(effects
+				(font
+					(size 1.27 1.27)
+				)
+			)
+		)
+		(property "DPN" "399-6856-1-ND"
 			(at 247.65 222.25 0)
 			(hide yes)
@@
 			)
 		)
-		(property "Datasheet" ""
+		(property "Datasheet" "https://search.kemet.com/download/specsheet/C0603C104K5RACAUTO"
 			(at 99.06 166.37 0)
 			(hide yes)
@@
 			)
 		)
-		(property "Description" "Unpolarized capacitor"
+		(property "Description" "0.1 µF ±10% 50V Ceramic Capacitor X7R 0603 (1608 Metric)"
+			(at 99.06 166.37 0)
+			(hide yes)
+			(show_name no)
+			(do_not_autoplace no)
+			(effects
+				(font
+					(size 1.27 1.27)
+				)
+			)
+		)
+		(property "DIS" "DigiKey"
+			(at 99.06 166.37 0)
+			(hide yes)
+			(show_name no)
+			(do_not_autoplace no)
+			(effects
+				(font
+					(size 1.27 1.27)
+				)
+			)
+		)
+		(property "DPN" "399-6856-1-ND"
+			(at 99.06 166.37 0)
+			(hide yes)
+			(show_name no)
+			(do_not_autoplace no)
+			(effects
+				(font
+					(size 1.27 1.27)
+				)
+			)
+		)
+		(property "MFR" "KEMET"
+			(at 99.06 166.37 0)
+			(hide yes)
+			(show_name no)
+			(do_not_autoplace no)
+			(effects
+				(font
+					(size 1.27 1.27)
+				)
+			)
+		)
+		(property "MPN" "C0603C104K5RACAUTO"
 			(at 99.06 166.37 0)
 			(hide yes)
@@
 			)
 		)
-		(property "Description" ""
+		(property "Description" "30 mOhms ±1% 0.5W, 1/2W Chip Resistor 1206 (3216 Metric) Current Sense Thick Film"
 			(at 264.16 38.1 0)
 			(hide yes)
@@
 			)
 		)
-		(property "DPN" ""
+		(property "DPN" "CSR1206FK30L0CT-ND"
 			(at 264.16 38.1 0)
 			(hide yes)
@@
 			)
 		)
-		(property "MPN" ""
+		(property "MPN" "CSR1206FK30L0"
 			(at 264.16 38.1 0)
 			(hide yes)
@@
 			)
 		)
-		(property "Datasheet" ""
+		(property "Datasheet" "https://search.kemet.com/download/specsheet/C0603C104K5RACAUTO"
 			(at 99.06 214.63 0)
 			(hide yes)
@@
 			)
 		)
-		(property "Description" "Unpolarized capacitor"
+		(property "Description" "0.1 µF ±10% 50V Ceramic Capacitor X7R 0603 (1608 Metric)"
+			(at 99.06 214.63 0)
+			(hide yes)
+			(show_name no)
+			(do_not_autoplace no)
+			(effects
+				(font
+					(size 1.27 1.27)
+				)
+			)
+		)
+		(property "DIS" "DigiKey"
+			(at 99.06 214.63 0)
+			(hide yes)
+			(show_name no)
+			(do_not_autoplace no)
+			(effects
+				(font
+					(size 1.27 1.27)
+				)
+			)
+		)
+		(property "DPN" "399-6856-1-ND"
+			(at 99.06 214.63 0)
+			(hide yes)
+			(show_name no)
+			(do_not_autoplace no)
+			(effects
+				(font
+					(size 1.27 1.27)
+				)
+			)
+		)
+		(property "MFR" "KEMET"
+			(at 99.06 214.63 0)
+			(hide yes)
+			(show_name no)
+			(do_not_autoplace no)
+			(effects
+				(font
+					(size 1.27 1.27)
+				)
+			)
+		)
+		(property "MPN" "C0603C104K5RACAUTO"
 			(at 99.06 214.63 0)
 			(hide yes)
@@
 			)
 		)
-		(property "Description" ""
+		(property "Description" "4.7 kOhms ±1% 0.1W, 1/10W Chip Resistor 0603 (1608 Metric) Automotive AEC-Q200 Thick Film"
 			(at 189.23 127 0)
 			(hide yes)
@@
 			)
 		)
-		(property "DPN" ""
+		(property "DPN" "RMCF0603FT4K70CT-ND"
 			(at 189.23 127 0)
 			(hide yes)
@@
 			)
 		)
-		(property "MPN" ""
+		(property "MPN" "RMCF0603FT4K70"
 			(at 189.23 127 0)
 			(hide yes)

Commit message: Large BOM changes for v1.2, no changes to PCB
Parts:
- R101, R102: DPN RMCF0603ZT0R00CT-ND -> RMCF0603FT100RCT-ND; MPN RMCF0603ZT0R00 -> RMCF0603FT100R
- R109: DPN (none) -> RMCF0603FT10K0CT-ND; MPN (none) -> RMCF0603FT10K0
- R11, R94, R95: DPN (none) -> RMCF0603FT100RCT-ND; MPN (none) -> RMCF0603FT100R
- TP1, TP10, TP11, TP110, TP12, TP13, TP14, TP15, TP2, TP3, TP4, TP5, TP8, TP9: value 1x01 -> Test-Point; now left out of the parts list
- U6: DPN 1676-1002-ND -> LTC3624EDD-5#PBF-ND
