File: oresat-gps-card/oresat-gps-card-sch-osd3358-usb-xtal.kicad_sch (KiCad schematic)
At the start: 15 parts, among them U1 OSD3358-512M-BSM, U11 RCLAMP0504FB, Y1 24MHz, Y2 Crystal

Commit message: Routine Push
Lots of footprint changes
Parts:
- C26, C27, C28, C29, C30: footprint Capacitor_SMD:C_0603_1608Metric -> oresat-passives:0603-C-NOSILK
- R46: value NP -> 1M
- R47, R75, R76, R77: footprint Resistor_SMD:R_0603_1608Metric -> oresat-passives:0603-C-NOSILK
Changed lines of the file:
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@@
 			)
 		)
-		(property "Footprint" "Capacitor_SMD:C_0603_1608Metric"
+		(property "Footprint" "oresat-passives:0603-C-NOSILK"
 			(at 123.19 77.7748 0)
 			(hide yes)
@@
 			)
 		)
-		(property "Footprint" "Resistor_SMD:R_0603_1608Metric"
+		(property "Footprint" "oresat-passives:0603-C-NOSILK"
 			(at 125.984 128.524 90)
 			(hide yes)
@@
 			)
 		)
-		(property "Value" "NP"
+		(property "Value" "1M"
 			(at 139.954 102.616 0)
 			(show_name no)
@@
 			)
 		)
-		(property "Footprint" "Capacitor_SMD:C_0603_1608Metric"
+		(property "Footprint" "oresat-passives:0603-C-NOSILK"
 			(at 174.2948 189.23 0)
 			(hide yes)
@@
 			)
 		)
-		(property "Footprint" "Capacitor_SMD:C_0603_1608Metric"
+		(property "Footprint" "oresat-passives:0603-C-NOSILK"
 			(at 124.46 108.2548 0)
 			(hide yes)
@@
 			)
 		)
-		(property "Footprint" "Capacitor_SMD:C_0603_1608Metric"
+		(property "Footprint" "oresat-passives:0603-C-NOSILK"
 			(at 123.19 93.0148 0)
 			(hide yes)
@@
 			)
 		)
-		(property "Footprint" "Resistor_SMD:R_0603_1608Metric"
+		(property "Footprint" "oresat-passives:0603-C-NOSILK"
 			(at 133.096 128.524 90)
 			(hide yes)
@@
 			)
 		)
-		(property "Footprint" "Capacitor_SMD:C_0603_1608Metric"
+		(property "Footprint" "oresat-passives:0603-C-NOSILK"
 			(at 123.19 62.5348 0)
 			(hide yes)
@@
 			)
 		)
-		(property "Footprint" "Resistor_SMD:R_0603_1608Metric"
+		(property "Footprint" "oresat-passives:0603-C-NOSILK"
 			(at 140.716 71.374 90)
 			(hide yes)
@@
 			)
 		)
-		(property "Footprint" "Resistor_SMD:R_0603_1608Metric"
+		(property "Footprint" "oresat-passives:0603-C-NOSILK"
 			(at 120.396 142.494 90)
 			(hide yes)

Commit message: Routine Push
Parts:
- R47: DIS (none) -> DigiKey; DPN (none) -> RMCF0603FT1M00CT-ND; MFR (none) -> Stackpole Electronics; MPN (none) -> RMCF0603FT1M00
- R75, R76, R77: DIS (none) -> DigiKey; DPN (none) -> RMCF0603FT10K0CT-ND; MFR (none) -> Stackpole Electronics; MPN (none) -> RMCF0603FT10K0
- U1: DIS (none) -> DigiKey; MFR (none) -> Octavo Systems LLC
- U11: DIS (none) -> DigiKey; DPN (none) -> RCLAMP0504FBTCTCT-ND; MFR (none) -> Semtech Corporation; MPN (none) -> RCLAMP0504FBTCT

Commit message: ERC and DRC cleaneup
Fixed symbols, fixed footprints, changed DRC rules to reduce errors,
updated footprints, mostly done.
Other:
- company: (none) -> Portland State Aerospace Society
Changed lines of the file:
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@@
 	(title_block
 		(title "OreSat GPS Card")
-		(date "2026-06-28")
+		(date "2026-07-06")
 		(rev "1.2")
+		(company "Portland State Aerospace Society")
 	)
 	(text "To monitor TPS65217 PMIC voltages"
@@
 	(wire
 		(pts
-			(xy 134.62 71.12) (xy 134.62 86.36)
-		)
-		(stroke
-			(width 0)
-			(type default)
-		)
-	)
-	(wire
-		(pts
 			(xy 127 139.7) (xy 154.94 139.7)
 		)
@@
 	(wire
 		(pts
-			(xy 130.81 71.12) (xy 134.62 71.12)
-		)
-		(stroke
-			(width 0)
-			(type default)
-		)
-	)
-	(wire
-		(pts
 			(xy 215.9 71.12) (xy 218.44 71.12)
 		)
@@
 					(unit 1)
 				)
-			)
-		)
-	)
-	(symbol
-		(lib_id "power:GND")
-		(at 134.62 86.36 0)
-		(unit 1)
-		(body_style 1)
-		(exclude_from_sim no)
-		(in_bom yes)
-		(on_board yes)
-		(in_pos_files yes)
-		(dnp no)
-		(property "Reference" "#GND0154"
-			(at 134.62 92.71 0)
-			(hide yes)
-			(show_name no)
-			(do_not_autoplace no)
-			(effects
-				(font
-					(size 1.27 1.27)
-				)
-			)
-		)
-		(property "Value" "GND"
-			(at 132.588 90.17 0)
-			(show_name no)
-			(do_not_autoplace no)
-			(effects
-				(font
-					(size 1.27 1.27)
-				)
-				(justify left)
-			)
-		)
-		(property "Footprint" ""
-			(at 134.62 86.36 0)
-			(hide yes)
-			(show_name no)
-			(do_not_autoplace no)
-			(effects
-				(font
-					(size 1.27 1.27)
-				)
-			)
-		)
-		(property "Datasheet" ""
-			(at 134.62 86.36 0)
-			(hide yes)
-			(show_name no)
-			(do_not_autoplace no)
-			(effects
-				(font
-					(size 1.27 1.27)
-				)
-			)
-		)
-		(property "Description" "Power symbol creates a global label with name \"GND\" , ground"
-			(at 134.62 86.36 0)
-			(hide yes)
-			(show_name no)
-			(do_not_autoplace no)
-			(effects
-				(font
-					(size 1.27 1.27)
-				)
-			)
-		)
-		(pin "1"
-		)
-		(instances
-			(project "oresat-gps-card"
-				(path "/65d12cdd-c326-4033-9053-c59fa4e0b25e/0d3a1fa4-c9ee-4335-9068-a81ae0178f3f"
-					(reference "#GND0154")
-					(unit 1)
-				)
