File: oresat-gps-card/oresat-gps-card-sch-osd3358-usb-xtal.kicad_sch (KiCad schematic)
At the start: 15 parts, among them U1 OSD3358-512M-BSM, U11 RCLAMP0504FB, Y1 24MHz, Y2 Crystal

Commit message: Last of the GPS card cleanup
    Better plains in the RF section, lots of shortening and straitening, cleaned up all ERC and DRCs.
Parts:
- added C51: 100n, oresat-passives:0603-C-NOSILK, symbol Device:C
Connections:
- net GND: no longer Y1.2 (G), Y1.4 (G)
- net OSC0_GND: now also Y1.2 (G), Y1.4 (G)
- net at U1.A7 (SYS_ADC_1P8V): now also U1.B7 (VREFP), C51.2
- net at U1.A9 (AGND_ADC), U1.B9 (VREFN): now also C51.1; no longer U1.B7 (VREFP)
- no-connect marks 23 -> 22
Other:
- note added: "32 KHz"
- note added: "HH"
- note added: "L0"
- note added: "LL"
- note added: "ZZ"
- note removed: "1M if populated"

Commit message: BOM Update
Parts:
- C26, C27, C28, C29: DIS (none) -> DigiKey; DPN (none) -> 490-1405-1-ND; MFR (none) -> Murata Electronics; MPN (none) -> GRM1885C1H120JA01D
- C30, C51: DIS (none) -> DigiKey; DPN (none) -> 399-6856-1-ND; MFR (none) -> KEMET; MPN (none) -> C0603C104K5RACAUTO

Commit message: Large BOM changes for v1.2, no changes to PCB
Parts:
- FB1: DIS (none) -> DigiKey; DPN (none) -> 490-14027-1-ND; MFR (none) -> Murata; MPN (none) -> BLM18KG300JH1D
- U1: DPN (none) -> 1676-OSD3358-1G-ISM-ND; MFR Octavo Systems LLC -> Octavo Systems; MPN OSD3358-512M-BSM -> OSD3358-1G-ISM
- Y1: DIS (none) -> DigiKey; DPN (none) -> XC2580CT-ND; MFR (none) -> ECS Inc; MPN (none) -> ECS-240-12-30BQ-AEN-TR
- Y2: DIS (none) -> DigiKey; DPN (none) -> 535-9542-1-ND; MFR (none) -> Abracon LLC; MPN (none) -> ABS07-32.768KHZ-T
Changed lines of the file:
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@@
 			)
 		)
-		(property "Datasheet" ""
+		(property "Datasheet" "https://ecsxtal.com/store/pdf/ECX-53BQ.pdf"
 			(at 125.73 71.12 0)
 			(hide yes)
@@
 			)
 		)
-		(property "Description" ""
+		(property "Description" "CRYSTAL 24.0000MHZ 12PF SMD"
 			(at 125.73 71.12 0)
+			(hide yes)
+			(show_name no)
+			(do_not_autoplace no)
+			(effects
+				(font
+					(size 1.27 1.27)
+				)
+			)
+		)
+		(property "DIS" "DigiKey"
+			(at 125.73 71.12 90)
+			(hide yes)
+			(show_name no)
+			(do_not_autoplace no)
+			(effects
+				(font
+					(size 1.27 1.27)
+				)
+			)
+		)
+		(property "DPN" "XC2580CT-ND"
+			(at 125.73 71.12 90)
+			(hide yes)
+			(show_name no)
+			(do_not_autoplace no)
+			(effects
+				(font
+					(size 1.27 1.27)
+				)
+			)
+		)
+		(property "MFR" "ECS Inc"
+			(at 125.73 71.12 90)
+			(hide yes)
+			(show_name no)
+			(do_not_autoplace no)
+			(effects
+				(font
+					(size 1.27 1.27)
+				)
+			)
+		)
+		(property "MPN" "ECS-240-12-30BQ-AEN-TR"
+			(at 125.73 71.12 90)
 			(hide yes)
 			(show_name no)
@@
 			)
 		)
-		(property "Datasheet" ""
+		(property "Datasheet" "https://abracon.com/Resonators/ABS07.pdf"
 			(at 127 101.6 0)
 			(hide yes)
@@
 			)
 		)
-		(property "Description" ""
+		(property "Description" "32.768 kHz ±20ppm Crystal 12.5pF 70 kOhms 2-SMD, No Lead"
 			(at 127 101.6 0)
+			(hide yes)
+			(show_name no)
+			(do_not_autoplace no)
+			(effects
+				(font
+					(size 1.27 1.27)
+				)
+			)
+		)
+		(property "DIS" "DigiKey"
+			(at 127 101.6 90)
+			(hide yes)
+			(show_name no)
+			(do_not_autoplace no)
+			(effects
+				(font
+					(size 1.27 1.27)
+				)
+			)
+		)
+		(property "DPN" "535-9542-1-ND"
+			(at 127 101.6 90)
+			(hide yes)
+			(show_name no)
+			(do_not_autoplace no)
+			(effects
+				(font
+					(size 1.27 1.27)
+				)
+			)
+		)
+		(property "MFR" "Abracon LLC"
+			(at 127 101.6 90)
+			(hide yes)
+			(show_name no)
+			(do_not_autoplace no)
+			(effects
+				(font
+					(size 1.27 1.27)
+				)
+			)
+		)
+		(property "MPN" "ABS07-32.768KHZ-T"
+			(at 127 101.6 90)
 			(hide yes)
 			(show_name no)
@@
 			)
 		)
-		(property "Datasheet" ""
+		(property "Datasheet" "https://pim.murata.com/asset/pim4/ferriteBeadInductortypefilter/QNFA9129_PDF_FERRITEBEADINDUCTORTYPEFILTER?lastModifiedDatetime=20250918112959"
 			(at 129.54 193.04 0)
 			(hide yes)
@@
 			)
 		)
-		(property "Description" ""
+		(property "Description" "30 Ohms @ 100 MHz 1 Power Line Ferrite Bead 0603 (1608 Metric) 3.3A 10mOhm"
 			(at 129.54 193.04 0)
+			(hide yes)
+			(show_name no)
+			(do_not_autoplace no)
+			(effects
+				(font
+					(size 1.27 1.27)
+				)
+			)
+		)
+		(property "DIS" "DigiKey"
+			(at 129.54 193.04 90)
+			(hide yes)
+			(show_name no)
+			(do_not_autoplace no)
+			(effects
+				(font
+					(size 1.27 1.27)
+				)
+			)
+		)
+		(property "DPN" "490-14027-1-ND"
+			(at 129.54 193.04 90)
+			(hide yes)
+			(show_name no)
+			(do_not_autoplace no)
+			(effects
+				(font
+					(size 1.27 1.27)
+				)
+			)
+		)
+		(property "MFR" "Murata"
+			(at 129.54 193.04 90)
+			(hide yes)
+			(show_name no)
+			(do_not_autoplace no)
+			(effects
+				(font
+					(size 1.27 1.27)
+				)
+			)
+		)
+		(property "MPN" "BLM18KG300JH1D"
+			(at 129.54 193.04 90)
 			(hide yes)
 			(show_name no)
@@
 			)
 		)
-		(property "Description" "OSD335x Embedded Module 1GHz 512MB"
+		(property "Description" "Embedded Module ARM® Cortex®-A8, AM3358 1GHz 1GB"
 			(at 185.42 2.54 0)
 			(hide yes)
@@
 			)
 		)
-		(property "MPN" "OSD3358-512M-BSM"
+		(property "MPN" "OSD3358-1G-ISM"
 			(at 185.42 7.62 0)
 			(hide yes)
@@
 			)
 		)
-		(property "MFR" "Octavo Systems LLC"
+		(property "MFR" "Octavo Systems"
 			(at 185.42 106.68 0)
 			(hide yes)
+			(show_name no)
+			(do_not_autoplace no)
+			(effects
+				(font
+					(size 1.27 1.27)
+				)
+			)
+		)
+		(property "DPN" "1676-OSD3358-1G-ISM-ND"
+			(at 185.42 106.68 0)
+			(hide yes)

Commit message: Upped to v1.3.
Fixed backward EEPROM programming pin, fixed potential boot error with missing PMIC connections, fixed some power domain issues.
Parts:
- U1: value OSD3358-512M-BSM -> OSD3358-1G-ISM
Connections:
- net nRESET: no longer names the net of U11.4 (I3)
- no-connect marks 22 -> 23
Other:
- note removed: "24 MHz RTC XO"
Changed lines of the file:
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@@
 	(title_block
 		(title "OreSat GPS Card")
-		(date "2026-07-06")
-		(rev "1.2")
+		(date "2026-09-17")
+		(rev "1.3")
 		(company "Portland State Aerospace Society")
 	)
@@
 			)
 			(justify right bottom)
-		)
-	)
-	(text "24 MHz RTC XO"
-		(exclude_from_sim no)
-		(at 90.17 72.39 0)
-		(effects
-			(font
-				(size 1.27 1.27)
-			)
-			(justify left bottom)
 		)
 	)
@@
 	)
 	(no_connect
+		(at 151.13 200.66)
+	)
+	(no_connect
 		(at 215.9 149.86)
 	)
@@
 	(wire
 		(pts
-			(xy 147.32 200.66) (xy 151.13 200.66)
-		)
-		(stroke
-			(width 0)
-			(type default)
-		)
-	)
-	(wire
-		(pts
 			(xy 113.03 83.82) (xy 154.94 83.82)
 		)
@@
 		)
 	)
+	(wire
+		(pts
+			(xy 115.57 63.5) (xy 113.03 63.5)
+		)
+		(stroke
+			(width 0)
+			(type default)
+		)
+	)
+	(wire
+		(pts
+			(xy 138.43 109.22) (xy 127 109.22)
+		)
+		(stroke
+			(width 0)
+			(type default)
+		)
+	)
+	(wire
+		(pts
+			(xy 113.03 78.74) (xy 113.03 83.82)
+		)
+		(stroke
+			(width 0)
+			(type default)
+		)
+	)
+	(wire
+		(pts
+			(xy 139.7 63.5) (xy 139.7 67.31)
+		)
+		(stroke
+			(width 0)
+			(type default)
+		)
+	)
+	(wire
+		(pts
+			(xy 139.7 195.58) (xy 151.13 195.58)
+		)
+		(stroke
+			(width 0)
+			(type default)
+		)
+	)
+	(wire
+		(pts
+			(xy 127 105.41) (xy 127 109.22)
+		)
+		(stroke
+			(width 0)
+			(type default)
+		)
+	)
+	(wire
+		(pts
+			(xy 218.44 60.96) (xy 218.44 71.12)
+		)
+		(stroke
+			(width 0)
+			(type default)
+		)
+	)
+	(wire
+		(pts
+			(xy 138.43 93.98) (xy 154.94 93.98)
+		)
+		(stroke
+			(width 0)
+			(type default)
+		)
+	)
 	(polyline
 		(pts
-			(xy 88.9 73.66) (xy 106.68 73.66)
-		)
-		(stroke
-			(width 0)
-			(type default)
-		)
-	)
-	(wire
-		(pts
-			(xy 115.57 63.5) (xy 113.03 63.5)
-		)
-		(stroke
-			(width 0)
-			(type default)
-		)
-	)
-	(wire
-		(pts
-			(xy 138.43 109.22) (xy 127 109.22)
-		)
-		(stroke
-			(width 0)
-			(type default)
-		)
-	)
-	(wire
-		(pts
-			(xy 113.03 78.74) (xy 113.03 83.82)
-		)
-		(stroke
-			(width 0)
-			(type default)
-		)
-	)
-	(polyline
-		(pts
-			(xy 106.68 73.66) (xy 106.68 68.58)
-		)
-		(stroke
-			(width 0)
-			(type default)
-		)
-	)
-	(wire
-		(pts
-			(xy 139.7 63.5) (xy 139.7 67.31)
-		)
-		(stroke
-			(width 0)
-			(type default)
-		)
-	)
-	(wire
-		(pts
-			(xy 139.7 195.58) (xy 151.13 195.58)
-		)
-		(stroke
-			(width 0)
-			(type default)
-		)
-	)
-	(wire
-		(pts
-			(xy 127 105.41) (xy 127 109.22)
-		)
-		(stroke
-			(width 0)
-			(type default)
-		)
-	)
-	(wire
-		(pts
-			(xy 218.44 60.96) (xy 218.44 71.12)
-		)
-		(stroke
-			(width 0)
-			(type default)
-		)
-	)
-	(wire
-		(pts
-			(xy 138.43 93.98) (xy 154.94 93.98)
-		)
-		(stroke
-			(width 0)
-			(type default)
-		)
-	)
-	(polyline
-		(pts
 			(xy 227.33 128.27) (xy 227.33 135.89)
 		)
@@
 		)
 	)
-	(polyline
-		(pts
-			(xy 88.9 68.58) (xy 88.9 73.66)
-		)
-		(stroke
-			(width 0)
-			(type default)
-		)
-	)
 	(wire
 		(pts
@@
 		(pts
 			(xy 132.08 121.92) (xy 129.54 121.92)
-		)
-		(stroke
-			(width 0)
-			(type default)
-		)
-	)
-	(polyline
-		(pts
-			(xy 88.9 68.58) (xy 106.68 68.58)
 		)
 		(stroke
@@
 			(font
 				(size 1.27 1.27)
-			)
-			(justify right)
-		)
-	)
-	(hierarchical_label "nRESET"
-		(shape input)
-		(at 147.32 200.66 180)
-		(effects
-			(font
-				(size 1.27 1.27)
+				(thickness 0.254)
+				(bold yes)
 			)
 			(justify right)
@@
 			(font
 				(size 1.27 1.27)
+				(thickness 0.254)
+				(bold yes)
 			)
 			(justify right)
@@
 			(font
 				(size 1.27 1.27)
+				(thickness 0.254)
+				(bold yes)
 			)
 			(justify right)
@@
 			)
 		)
-		(property "Value" "OSD3358-512M-BSM"
+		(property "Value" "OSD3358-1G-ISM"
 			(at 185.42 45.72 0)
 			(show_name no)
