File: oresat-gps-card/oresat-gps-card-sch-osd3358-sysboot.kicad_sch (KiCad schematic)
At the start: 6 parts, among them J2 Conn_01x02, J5 Conn_01x06, U1 OSD3358-512M-BSM

Commit message: Routine Push
Parts:
- U1: DIS (none) -> DigiKey; MFR (none) -> Octavo Systems LLC
Changed lines of the file:
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@@
+			)
+		)
+		(property "DIS" "DigiKey"
+			(at 184.15 143.51 0)
+			(hide yes)
+			(show_name no)
+			(do_not_autoplace no)
+			(effects
+				(font
+					(size 1.27 1.27)
+				)
+			)
+		)
+		(property "MFR" "Octavo Systems LLC"
+			(at 184.15 143.51 0)
+			(hide yes)
+			(show_name no)
+			(do_not_autoplace no)
+			(effects
+				(font
+					(size 1.27 1.27)
+				)
 			)
 		)

Commit message: ERC and DRC cleaneup
Fixed symbols, fixed footprints, changed DRC rules to reduce errors,
updated footprints, mostly done.
Connections:
- net SYSBOOT2 renamed BOOTCFG
Other:
- company: (none) -> Portland State Aerospace Society
Changed lines of the file:
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@@
 	(title_block
 		(title "OreSat GPS Card")
-		(date "2026-06-28")
+		(date "2026-07-06")
 		(rev "1.2")
+		(company "Portland State Aerospace Society")
 	)
 	(text "0"
@@
 		)
 	)
-	(hierarchical_label "SYSBOOT2"
+	(hierarchical_label "BOOTCFG"
 		(shape input)
 		(at 313.69 138.43 0)

Commit message: Last of the GPS card cleanup
    Better plains in the RF section, lots of shortening and straitening, cleaned up all ERC and DRCs.
Parts:
- removed J5: Conn_01x06, Connector_PinHeader_2.54mm:PinHeader_1x06_P2.54mm_Vertical, symbol Connector_Generic:Conn_01x06
Other:
- note added: "HH"
- note added: "LL"
- note added: "ZL"
- note added: "ZZ"
