File: oresat-gps-card/oresat-gps-card-sch-osd3358-sysboot.kicad_sch (KiCad schematic)
At the start: 5 parts, among them J2 Conn_01x02, U1 OSD3358-512M-BSM

Commit message: Clean up Orion UART names
Connections:
- net STQ_UART2_RX renamed UART2_RX
- net STQ_UART2_TX renamed UART2_TX
Changed lines of the file:
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@@
 		)
 	)
-	(hierarchical_label "STQ_UART2_TX"
+	(hierarchical_label "UART2_TX"
 		(shape input)
 		(at 128.27 118.11 180)
@@
 		)
 	)
-	(hierarchical_label "STQ_UART2_RX"
+	(hierarchical_label "UART2_RX"
 		(shape input)
 		(at 128.27 115.57 180)

Commit message: BOM Update
Parts:
- R72, R73, R74: DIS (none) -> DigiKey; DPN (none) -> 738-RAVF164DJT47K0CT-ND; MFR (none) -> Stackpole Electronics Inc; MPN (none) -> RAVF164DJT47K0
Changed lines of the file:
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@@
 			)
 		)
-		(property "Datasheet" "http://www.vishay.com/docs/31509/csc.pdf"
+		(property "Datasheet" "https://www.seielect.com/catalog/SEI-RAVF.pdf"
 			(at 283.21 171.45 0)
 			(hide yes)
@@
 			)
 		)
-		(property "Description" ""
+		(property "Description" "47k Ohm ±5% 100mW Power Per Element Isolated 4 Resistor Network/Array ±200ppm/°C 1206 (3216 Metric), Convex, Long Side Terminals"
 			(at 283.21 171.45 0)
+			(hide yes)
+			(show_name no)
+			(do_not_autoplace no)
+			(effects
+				(font
+					(size 1.27 1.27)
+				)
+			)
+		)
+		(property "DIS" "DigiKey"
+			(at 283.21 171.45 90)
+			(hide yes)
+			(show_name no)
+			(do_not_autoplace no)
+			(effects
+				(font
+					(size 1.27 1.27)
+				)
+			)
+		)
+		(property "DPN" "738-RAVF164DJT47K0CT-ND"
+			(at 283.21 171.45 90)
+			(hide yes)
+			(show_name no)
+			(do_not_autoplace no)
+			(effects
+				(font
+					(size 1.27 1.27)
+				)
+			)
+		)
+		(property "MFR" "Stackpole Electronics Inc"
+			(at 283.21 171.45 90)
+			(hide yes)
+			(show_name no)
+			(do_not_autoplace no)
+			(effects
+				(font
+					(size 1.27 1.27)
+				)
+			)
+		)
+		(property "MPN" "RAVF164DJT47K0"
+			(at 283.21 171.45 90)
 			(hide yes)
 			(show_name no)
@@
 			)
 		)
-		(property "Datasheet" "http://www.vishay.com/docs/31509/csc.pdf"
+		(property "Datasheet" "https://www.seielect.com/catalog/SEI-RAVF.pdf"
 			(at 257.81 171.45 0)
 			(hide yes)
@@
 			)
 		)
-		(property "Description" ""
+		(property "Description" "47k Ohm ±5% 100mW Power Per Element Isolated 4 Resistor Network/Array ±200ppm/°C 1206 (3216 Metric), Convex, Long Side Terminals"
 			(at 257.81 171.45 0)
+			(hide yes)
+			(show_name no)
+			(do_not_autoplace no)
+			(effects
+				(font
+					(size 1.27 1.27)
+				)
+			)
+		)
+		(property "DIS" "DigiKey"
+			(at 257.81 171.45 90)
+			(hide yes)
+			(show_name no)
+			(do_not_autoplace no)
+			(effects
+				(font
+					(size 1.27 1.27)
+				)
+			)
+		)
+		(property "DPN" "738-RAVF164DJT47K0CT-ND"
+			(at 257.81 171.45 90)
+			(hide yes)
+			(show_name no)
+			(do_not_autoplace no)
+			(effects
+				(font
+					(size 1.27 1.27)
+				)
+			)
+		)
+		(property "MFR" "Stackpole Electronics Inc"
+			(at 257.81 171.45 90)
+			(hide yes)
+			(show_name no)
+			(do_not_autoplace no)
+			(effects
+				(font
+					(size 1.27 1.27)
+				)
+			)
+		)
+		(property "MPN" "RAVF164DJT47K0"
+			(at 257.81 171.45 90)
 			(hide yes)
 			(show_name no)
@@
 			)
 		)
-		(property "Datasheet" "http://www.vishay.com/docs/31509/csc.pdf"
+		(property "Datasheet" "https://www.seielect.com/catalog/SEI-RAVF.pdf"
 			(at 285.75 90.17 0)
 			(hide yes)
@@
 			)
 		)
-		(property "Description" ""
+		(property "Description" "47k Ohm ±5% 100mW Power Per Element Isolated 4 Resistor Network/Array ±200ppm/°C 1206 (3216 Metric), Convex, Long Side Terminals"
 			(at 285.75 90.17 0)
 			(hide yes)
 			(show_name no)
+			(do_not_autoplace no)
+			(effects
+				(font
+					(size 1.27 1.27)
+				)
+			)
+		)
+		(property "DIS" "DigiKey"
+			(at 285.75 90.17 90)
+			(hide yes)
+			(show_name no)
+			(do_not_autoplace no)
+			(effects
+				(font
+					(size 1.27 1.27)
+				)
+			)
+		)
+		(property "DPN" "738-RAVF164DJT47K0CT-ND"
+			(at 285.75 90.17 90)
+			(hide yes)
+			(show_name no)
+			(do_not_autoplace no)
+			(effects
+				(font
+					(size 1.27 1.27)
+				)
+			)
+		)
+		(property "MFR" "Stackpole Electronics Inc"
+			(at 285.75 90.17 90)
+			(hide yes)
+			(show_name no)
+			(do_not_autoplace no)
+			(effects
+				(font
+					(size 1.27 1.27)
+				)
+			)
+		)
+		(property "MPN" "RAVF164DJT47K0"
+			(at 285.75 90.17 90)
+			(hide yes)
+			(show_name no)

Commit message: Large BOM changes for v1.2, no changes to PCB
Parts:
- R72, R73, R74: DPN 738-RAVF164DJT47K0CT-ND -> U7473CT-ND; MFR Stackpole Electronics Inc -> Panasonic Electronic Components; MPN RAVF164DJT47K0 -> EXB-A10P473J
- U1: DPN (none) -> 1676-OSD3358-1G-ISM-ND; MFR Octavo Systems LLC -> Octavo Systems; MPN OSD3358-512M-BSM -> OSD3358-1G-ISM
Changed lines of the file:
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@@
 			)
 		)
-		(property "Datasheet" "https://www.seielect.com/catalog/SEI-RAVF.pdf"
+		(property "Datasheet" "https://industrial.panasonic.com/ww/products/pt/resistor-network-array/models/EXBA10P473J"
 			(at 283.21 171.45 0)
 			(hide yes)
@@
 			)
 		)
-		(property "Description" "47k Ohm ±5% 100mW Power Per Element Isolated 4 Resistor Network/Array ±200ppm/°C 1206 (3216 Metric), Convex, Long Side Terminals"
+		(property "Description" "47k Ohm ±5% 62.5mW Power Per Element Bussed 8 Resistor Network/Array ±200ppm/°C 2512 (6432 Metric), Concave, Long Side Terminals"
 			(at 283.21 171.45 0)
 			(hide yes)
@@
 			)
 		)
-		(property "DPN" "738-RAVF164DJT47K0CT-ND"
+		(property "DPN" "U7473CT-ND"
 			(at 283.21 171.45 90)
 			(hide yes)
@@
 			)
 		)
-		(property "MFR" "Stackpole Electronics Inc"
+		(property "MFR" "Panasonic Electronic Components"
 			(at 283.21 171.45 90)
 			(hide yes)
@@
 			)
 		)
-		(property "MPN" "RAVF164DJT47K0"
+		(property "MPN" "EXB-A10P473J"
 			(at 283.21 171.45 90)
 			(hide yes)
@@
 			)
 		)
-		(property "Description" "OSD335x Embedded Module 1GHz 512MB"
+		(property "Description" "Embedded Module ARM® Cortex®-A8, AM3358 1GHz 1GB"
 			(at 184.15 39.37 0)
 			(hide yes)
@@
 			)
 		)
-		(property "MPN" "OSD3358-512M-BSM"
+		(property "MPN" "OSD3358-1G-ISM"
 			(at 184.15 44.45 0)
 			(hide yes)
@@
 			)
 		)
-		(property "MFR" "Octavo Systems LLC"
+		(property "MFR" "Octavo Systems"
+			(at 184.15 143.51 0)
+			(hide yes)
+			(show_name no)
+			(do_not_autoplace no)
+			(effects
+				(font
+					(size 1.27 1.27)
+				)
+			)
+		)
+		(property "DPN" "1676-OSD3358-1G-ISM-ND"
 			(at 184.15 143.51 0)
 			(hide yes)
@@
 			)
 		)
-		(property "Datasheet" "https://www.seielect.com/catalog/SEI-RAVF.pdf"
+		(property "Datasheet" "https://industrial.panasonic.com/ww/products/pt/resistor-network-array/models/EXBA10P473J"
 			(at 257.81 171.45 0)
 			(hide yes)
@@
 			)
 		)
-		(property "Description" "47k Ohm ±5% 100mW Power Per Element Isolated 4 Resistor Network/Array ±200ppm/°C 1206 (3216 Metric), Convex, Long Side Terminals"
+		(property "Description" "47k Ohm ±5% 62.5mW Power Per Element Bussed 8 Resistor Network/Array ±200ppm/°C 2512 (6432 Metric), Concave, Long Side Terminals"
 			(at 257.81 171.45 0)
 			(hide yes)
@@
 			)
 		)
-		(property "DPN" "738-RAVF164DJT47K0CT-ND"
+		(property "DPN" "U7473CT-ND"
 			(at 257.81 171.45 90)
 			(hide yes)
@@
 			)
 		)
-		(property "MFR" "Stackpole Electronics Inc"
+		(property "MFR" "Panasonic Electronic Components"
 			(at 257.81 171.45 90)
 			(hide yes)
@@
 			)
 		)
-		(property "MPN" "RAVF164DJT47K0"
+		(property "MPN" "EXB-A10P473J"
 			(at 257.81 171.45 90)
 			(hide yes)
@@
 			)
 		)
-		(property "Datasheet" "https://www.seielect.com/catalog/SEI-RAVF.pdf"
+		(property "Datasheet" "https://industrial.panasonic.com/ww/products/pt/resistor-network-array/models/EXBA10P473J"
 			(at 285.75 90.17 0)
 			(hide yes)
@@
 			)
 		)
-		(property "Description" "47k Ohm ±5% 100mW Power Per Element Isolated 4 Resistor Network/Array ±200ppm/°C 1206 (3216 Metric), Convex, Long Side Terminals"
+		(property "Description" "47k Ohm ±5% 62.5mW Power Per Element Bussed 8 Resistor Network/Array ±200ppm/°C 2512 (6432 Metric), Concave, Long Side Terminals"
 			(at 285.75 90.17 0)
 			(hide yes)
@@
 			)
 		)
-		(property "DPN" "738-RAVF164DJT47K0CT-ND"
+		(property "DPN" "U7473CT-ND"
 			(at 285.75 90.17 90)
 			(hide yes)
@@
 			)
 		)
-		(property "MFR" "Stackpole Electronics Inc"
+		(property "MFR" "Panasonic Electronic Components"
 			(at 285.75 90.17 90)
 			(hide yes)
@@
 			)
 		)
-		(property "MPN" "RAVF164DJT47K0"
+		(property "MPN" "EXB-A10P473J"
 			(at 285.75 90.17 90)
 			(hide yes)

Commit message: Upped to v1.3.
Fixed backward EEPROM programming pin, fixed potential boot error with missing PMIC connections, fixed some power domain issues.
Parts:
- U1: value OSD3358-512M-BSM -> OSD3358-1G-ISM
Changed lines of the file:
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@@
 	(title_block
 		(title "OreSat GPS Card")
-		(date "2026-07-06")
-		(rev "1.2")
+		(date "2026-09-17")
+		(rev "1.3")
 		(company "Portland State Aerospace Society")
 	)
@@
 	)
 	(hierarchical_label "MAX_~{SHDN}"
-		(shape input)
+		(shape output)
 		(at 128.27 128.27 180)
 		(effects
 			(font
 				(size 1.27 1.27)
+				(thickness 0.254)
+				(bold yes)
 			)
 			(justify right)
@@
 	)
 	(hierarchical_label "MAX_SPI1_CS0"
-		(shape input)
+		(shape output)
 		(at 128.27 135.89 180)
 		(effects
 			(font
 				(size 1.27 1.27)
+				(thickness 0.254)
+				(bold yes)
 			)
 			(justify right)
@@
 	)
 	(hierarchical_label "GPS-EN"
-		(shape input)
+		(shape output)
 		(at 128.27 153.67 180)
 		(effects
 			(font
 				(size 1.27 1.27)
+				(thickness 0.254)
+				(bold yes)
 			)
 			(justify right)
@@
 	)
 	(hierarchical_label "MAX_SPI1_D0"
-		(shape input)
+		(shape output)
 		(at 128.27 130.81 180)
 		(effects
 			(font
 				(size 1.27 1.27)
+				(thickness 0.254)
+				(bold yes)
 			)
 			(justify right)
@@
 	)
 	(hierarchical_label "UART2_TX"
-		(shape input)
+		(shape output)
 		(at 128.27 118.11 180)
 		(effects
 			(font
 				(size 1.27 1.27)
+				(thickness 0.254)
+				(bold yes)
 			)
 			(justify right)
@@
 			(font
 				(size 1.27 1.27)
+				(thickness 0.254)
+				(bold yes)
 			)
 			(justify right)
@@
 			(font
 				(size 1.27 1.27)
+				(thickness 0.254)
+				(bold yes)
 			)
 			(justify left)
@@
 	)
 	(hierarchical_label "MAX_SPI1_SCLK"
-		(shape input)
+		(shape output)
 		(at 128.27 133.35 180)
 		(effects
 			(font
 				(size 1.27 1.27)
+				(thickness 0.254)
+				(bold yes)
 			)
 			(justify right)
@@
 			(font
 				(size 1.27 1.27)
+				(thickness 0.254)
+				(bold yes)
 			)
 			(justify right)
@@
 			(font
 				(size 1.27 1.27)
+				(thickness 0.254)
+				(bold yes)
 			)
 			(justify right)
@@
 			)
 		)
-		(property "Value" "OSD3358-512M-BSM"
+		(property "Value" "OSD3358-1G-ISM"
 			(at 184.15 107.95 0)
 			(show_name no)
