File: oresat-gps-card/oresat-gps-card-sch-rf-power.kicad_sch (KiCad schematic)
At the start: 26 parts, among them U15 SKY65723-81, U16 BP2G+, U17 MAX8510EXK29+T, U18 MAX8510EXK29+T, U19 MAX8510EXK33+T

Commit message: Routine Push
Lots of footprint changes
Parts:
- C31, C32: footprint Capacitor_SMD:C_0603_1608Metric -> oresat-passives:0805-C-NOSILK
- C37, C38, C39, C40, C41, C42, C43, C44, C45, C46, C47, C48, C49, C50: footprint Capacitor_SMD:C_0603_1608Metric -> oresat-passives:0603-C-NOSILK
- FB2: footprint Resistor_SMD:R_0805_2012Metric -> oresat-passives:0805-C-NOSILK
- R58: footprint Resistor_SMD:R_0402_1005Metric -> oresat-passives:0603-C-NOSILK
- R60: footprint Resistor_SMD:R_0603_1608Metric -> oresat-passives:0603-C-NOSILK
Other:
- note removed: "FIXME"
Changed lines of the file:
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@@
 		(rev "1.2")
 	)
-	(text "FIXME"
-		(exclude_from_sim no)
-		(at 260.35 80.518 0)
-		(effects
-			(font
-				(size 2 2)
-				(thickness 0.4)
-				(bold yes)
-				(color 255 0 0 1)
-			)
-		)
-	)
 	(text "3.3V supply for SkyTraq"
 		(exclude_from_sim no)
@@
 			)
 		)
-		(property "Footprint" "Capacitor_SMD:C_0603_1608Metric"
+		(property "Footprint" "oresat-passives:0603-C-NOSILK"
 			(at 315.9252 81.28 0)
 			(hide yes)
@@
 			)
 		)
-		(property "Footprint" "Resistor_SMD:R_0402_1005Metric"
+		(property "Footprint" "oresat-passives:0603-C-NOSILK"
 			(at 105.156 85.344 90)
 			(hide yes)
@@
 			)
 		)
-		(property "Footprint" "Capacitor_SMD:C_0603_1608Metric"
+		(property "Footprint" "oresat-passives:0603-C-NOSILK"
 			(at 336.2452 111.76 0)
 			(hide yes)
@@
 			)
 		)
-		(property "Footprint" "Capacitor_SMD:C_0603_1608Metric"
+		(property "Footprint" "oresat-passives:0603-C-NOSILK"
 			(at 82.8548 87.63 0)
 			(hide yes)
@@
 			)
 		)
-		(property "Footprint" "Capacitor_SMD:C_0603_1608Metric"
+		(property "Footprint" "oresat-passives:0603-C-NOSILK"
 			(at 280.3652 83.82 0)
 			(hide yes)
@@
 			)
 		)
-		(property "Footprint" "Capacitor_SMD:C_0603_1608Metric"
+		(property "Footprint" "oresat-passives:0603-C-NOSILK"
 			(at 280.3652 114.3 0)
 			(hide yes)
@@
 			)
 		)
-		(property "Footprint" "Resistor_SMD:R_0805_2012Metric"
+		(property "Footprint" "oresat-passives:0805-C-NOSILK"
 			(at 251.46 75.438 90)
 			(hide yes)
@@
 			)
 		)
-		(property "Footprint" "Capacitor_SMD:C_0603_1608Metric"
+		(property "Footprint" "oresat-passives:0603-C-NOSILK"
 			(at 326.0852 157.48 0)
 			(hide yes)
@@
 			)
 		)
-		(property "Footprint" "Capacitor_SMD:C_0603_1608Metric"
+		(property "Footprint" "oresat-passives:0603-C-NOSILK"
 			(at 336.2452 81.28 0)
 			(hide yes)
@@
 			)
 		)
-		(property "Footprint" "Capacitor_SMD:C_0603_1608Metric"
+		(property "Footprint" "oresat-passives:0603-C-NOSILK"
 			(at 94.9452 87.63 0)
 			(hide yes)
@@
 			)
 		)
-		(property "Footprint" "Capacitor_SMD:C_0603_1608Metric"
+		(property "Footprint" "oresat-passives:0603-C-NOSILK"
 			(at 326.0852 111.76 0)
 			(hide yes)
@@
 			)
 		)
-		(property "Footprint" "Capacitor_SMD:C_0603_1608Metric"
+		(property "Footprint" "oresat-passives:0603-C-NOSILK"
 			(at 315.9252 111.76 0)
 			(hide yes)
@@
 			)
 		)
-		(property "Footprint" "Capacitor_SMD:C_0603_1608Metric"
+		(property "Footprint" "oresat-passives:0805-C-NOSILK"
 			(at 258.1148 83.82 0)
 			(hide yes)
@@
 			)
 		)
-		(property "Footprint" "Capacitor_SMD:C_0603_1608Metric"
+		(property "Footprint" "oresat-passives:0603-C-NOSILK"
 			(at 326.0852 81.28 0)
 			(hide yes)
@@
 			)
 		)
-		(property "Footprint" "Capacitor_SMD:C_0603_1608Metric"
+		(property "Footprint" "oresat-passives:0603-C-NOSILK"
 			(at 280.3652 158.75 0)
 			(hide yes)
@@
 			)
 		)
-		(property "Footprint" "Capacitor_SMD:C_0603_1608Metric"
+		(property "Footprint" "oresat-passives:0603-C-NOSILK"
 			(at 336.2452 157.48 0)
 			(hide yes)
@@
 			)
 		)
-		(property "Footprint" "Capacitor_SMD:C_0603_1608Metric"
+		(property "Footprint" "oresat-passives:0603-C-NOSILK"
 			(at 315.9252 157.48 0)
 			(hide yes)
@@
 			)
 		)
-		(property "Footprint" "Resistor_SMD:R_0603_1608Metric"
+		(property "Footprint" "oresat-passives:0603-C-NOSILK"
 			(at 290.576 178.054 90)
 			(hide yes)
@@
 			)
 		)
-		(property "Footprint" "Capacitor_SMD:C_0603_1608Metric"
+		(property "Footprint" "oresat-passives:0805-C-NOSILK"
 			(at 268.2748 83.82 0)
 			(hide yes)

Commit message: Routine Push
Parts:
- C39, C40, C41, C48, C49, C50: DIS (none) -> DigiKey; DPN (none) -> 490-GRT188R71E105KE13DCT-ND; MFR (none) -> Murata Electronics; MPN (none) -> GRT188R71E105KE13D
- R58, R60: DIS (none) -> DigiKey; DPN (none) -> RMCF0603FT10K0CT-ND; MFR (none) -> Stackpole Electronics; MPN (none) -> RMCF0603FT10K0
- U15: DPN (none) -> 863-2063-1-ND; MFR (none) -> Skyworks Solutions Inc.; MPN (none) -> SKY65723-81
- U17, U18: DIS (none) -> DigiKey; DPN (none) -> MAX8510EXK29+TCT-ND; MFR (none) -> Analog Devices Inc./Maxim Integrated; MPN (none) -> MAX8510EXK29+T
- U19: DIS (none) -> DigiKey; DPN (none) -> MAX8510EXK33+TCT-ND; MFR (none) -> Analog Devices Inc./Maxim Integrated; MPN (none) -> MAX8510EXK33+T

Commit message: Routine Push
Parts:
- L3: footprint oresat-passives:L_ECS-MPI4040 -> oresat-passives:L_ECS_MPIP0420; DIS (none) -> DigiKey; DPN (none) -> 50-ECS-MPIP0420-6R8MCCT-ND; MFR (none) -> ECS Inc.; MPN (none) -> ECS-MPIP0420-6R8MC
Changed lines of the file:
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@@
 			)
 		)
-		(property "Footprint" "oresat-passives:L_ECS-MPI4040"
+		(property "Footprint" "oresat-passives:L_ECS_MPIP0420"
 			(at 264.16 73.66 0)
 			(hide yes)
@@
 			)
 		)
-		(property "Datasheet" ""
+		(property "Datasheet" "https://ecsxtal.com/store/pdf/ECS-MPIP0420.pdf"
 			(at 264.16 73.66 0)
 			(hide yes)
@@
 			)
 		)
-		(property "Description" ""
+		(property "Description" "6.8 µH Shielded Molded Inductor 2 A 175mOhm Max Nonstandard"
 			(at 264.16 73.66 0)
 			(hide yes)
 			(show_name no)
+			(do_not_autoplace no)
+			(effects
+				(font
+					(size 1.27 1.27)
+				)
+			)
+		)
+		(property "DIS" "DigiKey"
+			(at 264.16 73.66 90)
+			(hide yes)
+			(show_name no)
+			(do_not_autoplace no)
+			(effects
+				(font
+					(size 1.27 1.27)
+				)
+			)
+		)
+		(property "DPN" "50-ECS-MPIP0420-6R8MCCT-ND"
+			(at 264.16 73.66 90)
+			(hide yes)
+			(show_name no)
+			(do_not_autoplace no)
+			(effects
+				(font
+					(size 1.27 1.27)
+				)
+			)
+		)
+		(property "MFR" "ECS Inc."
+			(at 264.16 73.66 90)
+			(hide yes)
+			(show_name no)
+			(do_not_autoplace no)
+			(effects
+				(font
+					(size 1.27 1.27)
+				)
+			)
+		)
+		(property "MPN" "ECS-MPIP0420-6R8MC"
+			(at 264.16 73.66 90)
+			(hide yes)
+			(show_name no)

Commit message: ERC and DRC cleaneup
Fixed symbols, fixed footprints, changed DRC rules to reduce errors,
updated footprints, mostly done.
Other:
- company: (none) -> Portland State Aerospace Society
Changed lines of the file:
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@@
 	(title_block
 		(title "OreSat GPS Card")
-		(date "2026-06-28")
+		(date "2026-07-06")
 		(rev "1.2")
+		(company "Portland State Aerospace Society")
 	)
 	(text "3.3V supply for SkyTraq"
@@
 		(pin "7"
 		)
+		(pin "[4,5]"
+		)
 		(instances
 			(project "oresat-gps-card"
@@
 	)
 	(symbol
-		(lib_id "gps-power:2.85VA")
+		(lib_id "power:VDDF")
 		(at 93.98 76.2 0)
 		(unit 1)
 		(body_style 1)
 		(exclude_from_sim no)
-		(in_bom no)
-		(on_board no)
+		(in_bom yes)
+		(on_board yes)
 		(in_pos_files yes)
 		(dnp no)
@@
 		)
 		(property "Value" "2.85VA"
-			(at 93.98 71.12 0)
+			(at 96.52 74.9299 0)
 			(show_name no)
 			(do_not_autoplace no)
@@
 					(size 1.27 1.27)
 				)
+				(justify left)
 			)
 		)
 		(property "Footprint" ""
-			(at 93.98 71.12 0)
+			(at 93.98 76.2 0)
 			(hide yes)
 			(show_name no)
@@
 		)
 		(property "Datasheet" ""
-			(at 93.98 71.12 0)
+			(at 93.98 76.2 0)
 			(hide yes)
 			(show_name no)
@@
 			)
 		)
-		(property "Description" ""
+		(property "Description" "Power symbol creates a global label with name \"VDDF\""
 			(at 93.98 76.2 0)
 			(hide yes)
@@
 	)
 	(symbol
-		(lib_id "gps-power:2.85VA")
+		(lib_id "power:VDDF")
 		(at 104.14 76.2 0)
 		(unit 1)
 		(body_style 1)
 		(exclude_from_sim no)
-		(in_bom no)
-		(on_board no)
+		(in_bom yes)
+		(on_board yes)
 		(in_pos_files yes)
 		(dnp no)
@@
 		)
 		(property "Value" "2.85VA"
-			(at 104.14 71.12 0)
+			(at 106.68 74.9299 0)
 			(show_name no)
 			(do_not_autoplace no)
@@
 					(size 1.27 1.27)
 				)
+				(justify left)
 			)
 		)
 		(property "Footprint" ""
-			(at 104.14 71.12 0)
+			(at 104.14 76.2 0)
 			(hide yes)
 			(show_name no)
@@
 		)
 		(property "Datasheet" ""
-			(at 104.14 71.12 0)
+			(at 104.14 76.2 0)
 			(hide yes)
 			(show_name no)
@@
 			)
 		)
-		(property "Description" ""
+		(property "Description" "Power symbol creates a global label with name \"VDDF\""
 			(at 104.14 76.2 0)
 			(hide yes)
@@
 	)
 	(symbol
-		(lib_id "gps-power:2.85VA")
+		(lib_id "power:VDDF")
 		(at 350.52 101.6 0)
 		(unit 1)
 		(body_style 1)
 		(exclude_from_sim no)
-		(in_bom no)
-		(on_board no)
+		(in_bom yes)
+		(on_board yes)
 		(in_pos_files yes)
 		(dnp no)
@@
 		)
 		(property "Footprint" ""
-			(at 350.52 96.52 0)
+			(at 350.52 101.6 0)
 			(hide yes)
 			(show_name no)
@@
 		)
 		(property "Datasheet" ""
-			(at 350.52 96.52 0)
+			(at 350.52 101.6 0)
 			(hide yes)
 			(show_name no)
@@
 			)
 		)
-		(property "Description" ""
+		(property "Description" "Power symbol creates a global label with name \"VDDF\""
 			(at 350.52 101.6 0)
 			(hide yes)

Commit message: Last of the GPS card cleanup
    Better plains in the RF section, lots of shortening and straitening, cleaned up all ERC and DRCs.
Parts:
- added D5: GRN, LED_SMD:LED_0603_1608Metric, symbol Device:LED
- added R62: 10k, oresat-passives:0603-C-NOSILK, symbol Device:R_US
- added TP21: 1x01, oresat-misc:TestPoint-0.75mm-th, symbol oresat-misc:Test-Point-0.75mm-th
Connections:
- net 3.3V-S: now also R62.2
- net GND: now also D5.1 (K)
- net GPS-EN: now also TP21.1
- net 5V-FILT: now reaches C31.1, C39.1, C40.1, C41.1, L3.2, U17.1 (IN), U18.1 (IN), U19.1 (IN)
- net RF-IN renamed LNA-IN-RF
- net RF-OUT renamed LNA-OUT-RF
- new net: D5.2 (A), R62.1
