File: oresat-gps-card/oresat-gps-card-sch-rf-power.kicad_sch (KiCad schematic)
At the start: 29 parts, among them U15 SKY65723-81, U16 BP2G+, U17 MAX8510EXK29+T, U18 MAX8510EXK29+T, U19 MAX8510EXK33+T

Commit message: BOM Update
Parts:
- C31, C32: DIS (none) -> DigiKey; DPN (none) -> 490-GRT21BC71E106KE13KCT-ND; MFR (none) -> Murata Electronics; MPN (none) -> GRT21BC71E106KE13K
- C37: DIS (none) -> DigiKey; DPN (none) -> 490-1345-1-ND; MFR (none) -> Murata Electronics; MPN (none) -> GRM1885C2A560JA01D
- C38, C45, C46, C47: DIS (none) -> DigiKey; DPN (none) -> 399-6856-1-ND; MFR (none) -> KEMET; MPN (none) -> C0603C104K5RACAUTO
- C42, C43, C44: DIS (none) -> DigiKey; DPN (none) -> 399-12983-1-ND; MFR (none) -> KEMET; MPN (none) -> C0603C103J5RACAUTO

Commit message: Large BOM changes for v1.2, no changes to PCB
Parts:
- FB2: DIS (none) -> DigiKey; DPN (none) -> 490-5988-1-ND; MFR (none) -> Murata; MPN (none) -> BLM21PG331SN1D
- SH1: value BMI-S-202-C -> BMI-S-202-F; DIS (none) -> DigiKey; DPN (none) -> 903-1051-1-ND; MFR (none) -> Laird Technologies EMI; MPN (none) -> BMI-S-202-F; now not fitted
- TP21: value 1x01 -> Test-Point; now left out of the parts list
- U15: DIS (none) -> DigiKey
- U16: DIS (none) -> DigiKey; DPN (none) -> 3157-BP2G1+CT-ND; MFR (none) -> Mini-Circuits; MPN (none) -> BP2G1+
Other:
- note added: "Cover: Laird BMI-S-202-C"
Changed lines of the file:
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@@
 		)
 	)
+	(text "Cover: Laird BMI-S-202-C"
+		(exclude_from_sim no)
+		(at 114.046 127 0)
+		(effects
+			(font
+				(size 1.27 1.27)
+			)
+		)
+	)
 	(text "All resistors are 0603 1% AEC-Q200 unless marked.\nAll capacitors are 0603 AEC-Q200 Vw >= 16V X5R or better unless marked."
 		(exclude_from_sim no)
@@
 			)
 		)
-		(property "Description" ""
+		(property "Description" "RF Power Divider 1.2 GHz ~ 2 GHz Isolation (Min) 10dB, 1.3 VSWR (Typ), 3° Imbalance (Max) 8-SOIC (0.154\", 3.90mm Width)"
+			(at 142.24 104.14 0)
+			(hide yes)
+			(show_name no)
+			(do_not_autoplace no)
+			(effects
+				(font
+					(size 1.27 1.27)
+				)
+			)
+		)
+		(property "DIS" "DigiKey"
+			(at 142.24 104.14 0)
+			(hide yes)
+			(show_name no)
+			(do_not_autoplace no)
+			(effects
+				(font
+					(size 1.27 1.27)
+				)
+			)
+		)
+		(property "DPN" "3157-BP2G1+CT-ND"
+			(at 142.24 104.14 0)
+			(hide yes)
+			(show_name no)
+			(do_not_autoplace no)
+			(effects
+				(font
+					(size 1.27 1.27)
+				)
+			)
+		)
+		(property "MFR" "Mini-Circuits"
+			(at 142.24 104.14 0)
+			(hide yes)
+			(show_name no)
+			(do_not_autoplace no)
+			(effects
+				(font
+					(size 1.27 1.27)
+				)
+			)
+		)
+		(property "MPN" "BP2G1+"
 			(at 142.24 104.14 0)
 			(hide yes)
@@
 		(body_style 1)
 		(exclude_from_sim no)
-		(in_bom yes)
+		(in_bom no)
 		(on_board yes)
 		(in_pos_files yes)
@@
 			)
 		)
-		(property "Value" "1x01"
+		(property "Value" "Test-Point"
 			(at 276.86 170.18 0)
 			(hide yes)
@@
 		)
 		(property "Footprint" "oresat-misc:TestPoint-0.75mm-th"
-			(at 276.86 170.18 0)
+			(at 276.86 162.56 0)
 			(hide yes)
 			(show_name no)
@@
 		)
 		(property "Datasheet" ""
-			(at 276.86 170.18 0)
+			(at 276.86 172.72 0)
 			(hide yes)
 			(show_name no)
@@
 			)
 		)
-		(property "Description" ""
+		(property "Description" "0.75 mm TH test point; good for scope probes and jumpers"
 			(at 276.86 172.72 0)
 			(hide yes)
@@
 			)
 		)
+		(property "DIS" "DigiKey"
+			(at 99.06 101.6 0)
+			(hide yes)
+			(show_name no)
+			(do_not_autoplace no)
+			(effects
+				(font
+					(size 1.27 1.27)
+				)
+			)
+		)
 		(pin "1"
 		)
@@
 		(on_board yes)
 		(in_pos_files yes)
-		(dnp no)
-		(fields_autoplaced yes)
+		(dnp yes)
 		(property "Reference" "SH1"
-			(at 130.81 135.8899 0)
+			(at 113.284 131.318 0)
 			(show_name no)
 			(do_not_autoplace no)
@@
 			)
 		)
-		(property "Value" "BMI-S-202-C"
-			(at 130.81 138.4299 0)
+		(property "Value" "BMI-S-202-F"
+			(at 108.204 133.858 0)
 			(show_name no)
 			(do_not_autoplace no)
@@
 			)
 		)
-		(property "Datasheet" ""
+		(property "Datasheet" "https://www.laird.com/document/datasheet/bmi-s-202-sales"
 			(at 114.3 139.7 0)
 			(hide yes)
@@
 			)
 		)
-		(property "Description" ""
+		(property "Description" "RF Shield Frame 0.650\" (16.50mm) X 0.650\" (16.50mm) Surface Mount"
+			(at 114.3 137.16 0)
+			(hide yes)
+			(show_name no)
+			(do_not_autoplace no)
+			(effects
+				(font
+					(size 1.27 1.27)
+				)
+			)
+		)
+		(property "DIS" "DigiKey"
+			(at 114.3 137.16 0)
+			(hide yes)
+			(show_name no)
+			(do_not_autoplace no)
+			(effects
+				(font
+					(size 1.27 1.27)
+				)
+			)
+		)
+		(property "DPN" "903-1051-1-ND"
+			(at 114.3 137.16 0)
+			(hide yes)
+			(show_name no)
+			(do_not_autoplace no)
+			(effects
+				(font
+					(size 1.27 1.27)
+				)
+			)
+		)
+		(property "MFR" "Laird Technologies EMI"
+			(at 114.3 137.16 0)
+			(hide yes)
+			(show_name no)
+			(do_not_autoplace no)
+			(effects
+				(font
+					(size 1.27 1.27)
+				)
+			)
+		)
+		(property "MPN" "BMI-S-202-F"
 			(at 114.3 137.16 0)
 			(hide yes)
@@
 			)
 		)
-		(property "Datasheet" ""
+		(property "Datasheet" "https://pim.murata.com/asset/pim4/ferriteBeadInductortypefilter/ENFA0005_PDF_FERRITEBEADINDUCTORTYPEFILTER?lastModifiedDatetime=20260105172120"
 			(at 251.46 73.66 0)
 			(hide yes)
@@
 			)
 		)
-		(property "Description" ""
+		(property "Description" "330 Ohms @ 100 MHz 1 Power Line Ferrite Bead 0805 (2012 Metric) 1.5A 70mOhm"
 			(at 251.46 73.66 0)
 			(hide yes)
 			(show_name no)
+			(do_not_autoplace no)
+			(effects
+				(font
+					(size 1.27 1.27)
+				)
+			)
+		)
+		(property "DIS" "DigiKey"
+			(at 251.46 73.66 90)
+			(hide yes)
+			(show_name no)
+			(do_not_autoplace no)
+			(effects
+				(font
+					(size 1.27 1.27)
+				)
+			)
+		)
+		(property "DPN" "490-5988-1-ND"
+			(at 251.46 73.66 90)
+			(hide yes)
+			(show_name no)
+			(do_not_autoplace no)
+			(effects
+				(font
+					(size 1.27 1.27)
+				)
+			)
+		)
+		(property "MFR" "Murata"
+			(at 251.46 73.66 90)
+			(hide yes)
+			(show_name no)
+			(do_not_autoplace no)
+			(effects
+				(font
+					(size 1.27 1.27)
+				)
+			)
+		)
+		(property "MPN" "BLM21PG331SN1D"
+			(at 251.46 73.66 90)
+			(hide yes)
+			(show_name no)

Commit message: Updated Layout
Changes to BOM. Changes to footprint assignments.
Parts:
- L3: footprint oresat-passives:L_ECS_MPIP0420 -> oresat-passives:L_ECS-MPI4040
Changed lines of the file:
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@@
 			)
 		)
-		(property "Footprint" "oresat-passives:L_ECS_MPIP0420"
+		(property "Footprint" "oresat-passives:L_ECS-MPI4040"
 			(at 264.16 73.66 0)
 			(hide yes)

Commit message: Upped to v1.3.
Fixed backward EEPROM programming pin, fixed potential boot error with missing PMIC connections, fixed some power domain issues.
Changed lines of the file:
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@@
 	(title_block
 		(title "OreSat GPS Card")
-		(date "2026-07-06")
-		(rev "1.2")
+		(date "2026-09-17")
+		(rev "1.3")
 		(company "Portland State Aerospace Society")
 	)
@@
 			(font
 				(size 1.27 1.27)
+				(thickness 0.254)
+				(bold yes)
 			)
 			(justify right)
@@
 			(font
 				(size 1.27 1.27)
+				(thickness 0.254)
+				(bold yes)
 			)
 			(justify right)
@@
 	)
 	(hierarchical_label "STQ-RF"
-		(shape input)
+		(shape output)
 		(at 157.48 99.06 0)
 		(effects
 			(font
 				(size 1.27 1.27)
+				(thickness 0.254)
+				(bold yes)
 			)
 			(justify left)
@@
 	)
 	(hierarchical_label "MAX-RF"
-		(shape input)
+		(shape output)
 		(at 157.48 104.14 0)
 		(effects
 			(font
 				(size 1.27 1.27)
+				(thickness 0.254)
+				(bold yes)
 			)
 			(justify left)
@@
 			)
 		)
-		(property "Description" "Ultra-low-noise LDO 2.85 V, SC-70-5"
+		(property "Description" "Linear Voltage Regulator IC Positive Fixed 1 Output 120mA SC-70-5"
 			(at 302.26 106.68 0)
 			(hide yes)
@@
 			)
 		)
-		(property "Description" "Ultra-low-noise LDO 2.85 V, SC-70-5"
+		(property "Description" "Linear Voltage Regulator IC Positive Fixed 1 Output 120mA SC-70-5"
 			(at 302.26 76.2 0)
 			(hide yes)
@@
 			)
 		)
-		(property "Description" "Ultra-low-noise LDO 2.85 V, SC-70-5"
+		(property "Description" "Linear Voltage Regulator IC Positive Fixed 1 Output 120mA SC-70-5"
 			(at 302.26 152.4 0)
 			(hide yes)
