File: oresat-gps-card/oresat-gps-card.kicad_pcb (KiCad board)
At the start: 4 copper layers, 99.8 x 94.6 mm, 245 parts, among them J1 J-SAMTEC-TFM-120-01-L-D-RA, J2 Conn_01x02, J3 GRPB041VWVN-RC, J4 DM3BT-DSF-PEJS, J6 SM14B-SHLS-TF, Q1 DMP2110UVTQ-7, Q2 DMPH2040UVTQ-7, Q6 MMBT2907, Q7 DMPH2040UVTQ-7, Q8 DMN2050LQ-7, Q9 DMN2050LQ-7, U1 OSD3358-512M-BSM, U10 SN74LVC1G07DCK, U11 RCLAMP0504FB, U13 MAX2769, U14 TLVH431, U15 SKY65723-81, U16 BP2G+, U17 MAX8510EXK29+T, U18 MAX8510EXK29+T, U19 MAX8510EXK33+T, U2 MAX7310ATE, U20 TS5A21366DCUR, U21 MAX4211FETE, U23 ORION-B16, U24 D32G-016.368M, U28 LT1719IS6, U3 MIC842LYC5, U4 MIC842LYC5, U6 LTC3624, U8 TCAN330, U9 EMMC+RESET+5.1-COMPATIBLE-BA, Y1 24MHz, Y2 Crystal

Commit message: Updated Layout
Changes to BOM. Changes to footprint assignments.
Parts:
- C7: footprint oresat-passives:0603-C-NOSILK -> oresat-passives:0805-C-NOSILK
- L3: footprint oresat-passives:L_ECS_MPIP0420 -> oresat-passives:L_ECS-MPI4040
- moved C32 0.93 mm to (159.6, 102.2)
- moved C31 0.93 mm to (159.6, 105.4)
- moved C7 0.25 mm to (161.3, 64.8)
Routing:
- net /RF + RF Power/5V-FILT: track 11.1 -> 12.0 mm
- net Net-(C32-Pad1): track 4.75 -> 5.66 mm
