File: oresat-gps-card/oresat-gps-card.kicad_pcb (KiCad board)
At the start: 4 copper layers, 99.8 x 94.6 mm, 245 parts, among them J1 TFM-120-01-L-D-RA, J2 Conn_01x02, J3 GRPB041VWVN-RC, J4 DM3BT-DSF-PEJS, J6 SM14B-SHLS-TF, Q1 DMP2110UVTQ-7, Q2 DMPH2040UVTQ-7, Q6 MMBT2907, Q7 DMPH2040UVTQ-7, Q8 DMN2050LQ-7, Q9 DMN2050LQ-7, U1 OSD3358-1G-ISM, U10 SN74LVC1G07DCK, U11 RCLAMP0504FB, U13 MAX2769, U14 TLVH431, U15 SKY65723-81, U16 BP2G+, U17 MAX8510EXK29+T, U18 MAX8510EXK29+T, U19 MAX8510EXK33+T, U2 MAX7310ATE, U20 TS5A21366DCUR, U21 MAX4211FETE, U23 ORION-B16, U24 D32G-016.368M, U28 LT1719IS6, U3 MIC842LYC5, U4 MIC842LYC5, U6 LTC3624, U8 TCAN337GDCNR, U9 EMMC+RESET+5.1-COMPATIBLE-BA, Y1 24MHz, Y2 Crystal

Commit message: Fixed boot issue, updated date, updated version, ready for a final polish
Parts:
- U9: value EMMC+RESET+5.1-COMPATIBLE-BA -> E32GS22AXC-01011
Changed lines of the file:
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@@
 	(title_block
 		(title "OreSat GPS Card")
-		(date "2026-09-17")
+		(date "2026-10-04")
 		(rev "1.3")
 		(company "Portland State Aerospace Society")
@@
 			)
 		)
-		(property "Value" "EMMC+RESET+5.1-COMPATIBLE-BA"
+		(property "Value" "E32GS22AXC-01011"
 			(at -5.6 7.6 0)
 			(layer "F.Fab")
@@
 			)
 		)
-		(property "Datasheet" "https://www.micron.com/products/managed-nand/emmc/part-catalog/mtfc32gazaqhd-it?login"
+		(property "Datasheet" "https://mm.digikey.com/Volume0/opasdata/d220001/medias/docus/9015/E32GS22AXC-01011.pdf"
 			(at 0 0 0)
 			(layer "F.Fab")
@@
 			)
 		)
-		(property "Description" "FLASH - NAND Memory IC 256Gbit eMMC 200 MHz 153-VFBGA (11.5x13)"
+		(property "Description" "FLASH - NAND (TLC) Memory IC 256Gbit eMMC_5.1 200 MHz 153-FBGA (11.5x13)"
 			(at 0 0 0)
 			(layer "F.Fab")
@@
 			)
 		)
-		(property "DPN" "557-MTFC32GAZAQHD-IT-ND"
+		(property "DPN" "5625-E32GS22AXC-01011-ND"
 			(at 0 0 0)
 			(unlocked yes)
@@
 			)
 		)
-		(property "MFR" "Micron Technology Inc."
+		(property "MFR" "Kingston Technology"
 			(at 0 0 0)
 			(unlocked yes)
@@
 			)
 		)
-		(property "MPN" "MTFC32GAZAQHD-IT"
+		(property "MPN" "E32GS22AXC-01011"
 			(at 0 0 0)
 			(unlocked yes)
@@
 	)
 	(segment
+		(start 142.35625 84.075)
+		(end 141.98125 84.45)
+		(width 0.127)
+		(layer "F.Cu")
+		(net "/PMIC_SCL")
+	)
+	(segment
+		(start 142.35625 81.96875)
+		(end 143.8 80.525)
+		(width 0.2)
+		(layer "F.Cu")
+		(net "/PMIC_SCL")
+	)
+	(segment
+		(start 141.98125 84.45)
+		(end 141.245 84.45)
+		(width 0.127)
+		(layer "F.Cu")
+		(net "/PMIC_SCL")
+	)
+	(segment
+		(start 143.8 80.525)
+		(end 147.05 80.525)
+		(width 0.2)
+		(layer "F.Cu")
+		(net "/PMIC_SCL")
+	)
+	(segment
+		(start 147.05 80.525)
+		(end 152.625 74.95)
+		(width 0.2)
+		(layer "F.Cu")
+		(net "/PMIC_SCL")
+	)
+	(segment
+		(start 152.625 74.95)
+		(end 159.645 74.95)
+		(width 0.2)
+		(layer "F.Cu")
+		(net "/PMIC_SCL")
+	)
+	(segment
+		(start 142.35625 81.96875)
+		(end 142.35625 84.075)
+		(width 0.127)
+		(layer "F.Cu")
+		(net "/PMIC_SCL")
+	)
+	(segment
+		(start 159.645 74.95)
+		(end 160.295 74.3)
+		(width 0.2)
+		(layer "F.Cu")
+		(net "/PMIC_SCL")
+	)
+	(segment
+		(start 141.245 84.45)
+		(end 140.605 85.09)
+		(width 0.127)
+		(layer "F.Cu")
+		(net "/PMIC_SCL")
+	)
+	(segment
+		(start 140.605 85.09)
+		(end 140.605 86.36)
+		(width 0.4064)
+		(layer "F.Cu")
+		(net "/PMIC_SCL")
+	)
+	(segment
+		(start 142.66875 82.23125)
+		(end 142.66875 84.29625)
+		(width 0.127)
+		(layer "F.Cu")
+		(net "/PMIC_SDA")
+	)
+	(segment
+		(start 161.565 74.885)
+		(end 160.8 75.65)
+		(width 0.2)
+		(layer "F.Cu")
+		(net "/PMIC_SDA")
+	)
+	(segment
+		(start 161.565 74.3)
+		(end 161.565 74.885)
+		(width 0.2)
+		(layer "F.Cu")
+		(net "/PMIC_SDA")
+	)
+	(segment
+		(start 152.55 75.65)
+		(end 147.325 80.875)
+		(width 0.2)
+		(layer "F.Cu")
+		(net "/PMIC_SDA")
+	)
+	(segment
+		(start 142.66875 84.29625)
+		(end 141.875 85.09)
+		(width 0.127)
+		(layer "F.Cu")
+		(net "/PMIC_SDA")
+	)
+	(segment
+		(start 147.325 80.875)
+		(end 144.025 80.875)
+		(width 0.2)
+		(layer "F.Cu")
+		(net "/PMIC_SDA")
+	)
+	(segment
+		(start 144.025 80.875)
+		(end 142.66875 82.23125)
+		(width 0.2)
+		(layer "F.Cu")
+		(net "/PMIC_SDA")
+	)
+	(segment
+		(start 160.8 75.65)
+		(end 152.55 75.65)
+		(width 0.2)
+		(layer "F.Cu")
+		(net "/PMIC_SDA")
+	)
+	(segment
+		(start 141.875 85.09)
+		(end 141.875 86.36)
+		(width 0.4064)
+		(layer "F.Cu")
+		(net "/PMIC_SDA")
+	)
+	(segment
 		(start 131.91875 97.1375)
 		(end 131.0625 97.1375)
@@
 	)
 	(segment
-		(start 142.66875 82.23125)
-		(end 142.66875 84.29625)
-		(width 0.127)
-		(layer "F.Cu")
-		(net "/PMIC_SDA")
-	)
-	(segment
-		(start 161.565 74.885)
-		(end 160.8 75.65)
-		(width 0.2)
-		(layer "F.Cu")
-		(net "/PMIC_SDA")
-	)
-	(segment
-		(start 161.565 74.3)
-		(end 161.565 74.885)
-		(width 0.2)
-		(layer "F.Cu")
-		(net "/PMIC_SDA")
-	)
-	(segment
-		(start 152.55 75.65)
-		(end 147.325 80.875)
-		(width 0.2)
-		(layer "F.Cu")
-		(net "/PMIC_SDA")
-	)
-	(segment
-		(start 142.66875 84.29625)
-		(end 141.875 85.09)
-		(width 0.127)
-		(layer "F.Cu")
-		(net "/PMIC_SDA")
-	)
-	(segment
-		(start 147.325 80.875)
-		(end 144.025 80.875)
-		(width 0.2)
-		(layer "F.Cu")
-		(net "/PMIC_SDA")
-	)
-	(segment
-		(start 144.025 80.875)
-		(end 142.66875 82.23125)
-		(width 0.2)
-		(layer "F.Cu")
-		(net "/PMIC_SDA")
-	)
-	(segment
-		(start 160.8 75.65)
-		(end 152.55 75.65)
-		(width 0.2)
-		(layer "F.Cu")
-		(net "/PMIC_SDA")
-	)
-	(segment
-		(start 141.875 85.09)
-		(end 141.875 86.36)
-		(width 0.4064)
-		(layer "F.Cu")
-		(net "/PMIC_SDA")
-	)
-	(segment
-		(start 142.35625 84.075)
-		(end 141.98125 84.45)
-		(width 0.127)
-		(layer "F.Cu")
-		(net "/PMIC_SCL")
-	)
-	(segment
-		(start 142.35625 81.96875)
-		(end 143.8 80.525)
-		(width 0.2)
-		(layer "F.Cu")
-		(net "/PMIC_SCL")
-	)
-	(segment
-		(start 141.98125 84.45)
-		(end 141.245 84.45)
-		(width 0.127)
-		(layer "F.Cu")
-		(net "/PMIC_SCL")
-	)
-	(segment
-		(start 143.8 80.525)
-		(end 147.05 80.525)
-		(width 0.2)
-		(layer "F.Cu")
-		(net "/PMIC_SCL")
-	)
-	(segment
-		(start 147.05 80.525)
-		(end 152.625 74.95)
-		(width 0.2)
-		(layer "F.Cu")
-		(net "/PMIC_SCL")
-	)
-	(segment
-		(start 152.625 74.95)
-		(end 159.645 74.95)
-		(width 0.2)
-		(layer "F.Cu")
-		(net "/PMIC_SCL")
-	)
-	(segment
-		(start 142.35625 81.96875)
-		(end 142.35625 84.075)
-		(width 0.127)
-		(layer "F.Cu")
-		(net "/PMIC_SCL")
-	)
-	(segment
-		(start 159.645 74.95)
-		(end 160.295 74.3)
-		(width 0.2)
-		(layer "F.Cu")
-		(net "/PMIC_SCL")
-	)
-	(segment
-		(start 141.245 84.45)
-		(end 140.605 85.09)
-		(width 0.127)
-		(layer "F.Cu")
-		(net "/PMIC_SCL")
-	)
-	(segment
-		(start 140.605 85.09)
-		(end 140.605 86.36)
-		(width 0.4064)
-		(layer "F.Cu")
-		(net "/PMIC_SCL")
-	)
-	(segment
