File: oresat-gps-card/oresat-gps-card.kicad_sch (KiCad schematic)
At the start: 10 parts, among them J1 J-SAMTEC-TFM-120-01-L-D-RA, J3 GRPB041VWVN-RC, J6 SM14B-SHLS-TF

Commit message: Routine Push
Lots of footprint changes
Parts:
- R68: footprint Resistor_SMD:R_0603_1608Metric -> oresat-passives:0603-C-NOSILK
Changed lines of the file:
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@@
 			)
 		)
-		(property "Footprint" "Resistor_SMD:R_0603_1608Metric"
+		(property "Footprint" "oresat-passives:0603-C-NOSILK"
 			(at 208.534 209.296 90)
 			(hide yes)

Commit message: Routine Push
Parts:
- J1: DIS (none) -> DigiKey; DPN (none) -> SAM10145-ND; MFR (none) -> Samtec Inc.; MPN (none) -> TFM-120-01-L-D-RA
Connections:
- net ~{SD}: no longer names the net of J1.39
- net ~{SD}: no longer J1.40
- no-connect marks 22 -> 24
Changed lines of the file:
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@@
-	)
-	(junction
-		(at 152.4 135.89)
-		(diameter 0)
-		(color 0 0 0 0)
 	)
 	(junction
@@
 	)
 	(junction
+		(at 152.4 95.25)
+		(diameter 0)
+		(color 0 0 0 0)
+	)
+	(junction
 		(at 153.67 80.01)
 		(diameter 0)
@@
 	)
 	(no_connect
+		(at 149.86 138.43)
+	)
+	(no_connect
 		(at 149.86 92.71)
 	)
@@
 	)
 	(no_connect
+		(at 149.86 135.89)
+	)
+	(no_connect
 		(at 149.86 44.45)
 	)
@@
 	(wire
 		(pts
-			(xy 152.4 135.89) (xy 152.4 138.43)
-		)
-		(stroke
-			(width 0)
-			(type default)
-		)
-	)
-	(wire
-		(pts
 			(xy 203.2 200.66) (xy 256.54 200.66)
 		)
@@
 	(wire
 		(pts
+			(xy 156.21 95.25) (xy 152.4 95.25)
+		)
+		(stroke
+			(width 0)
+			(type default)
+		)
+	)
+	(wire
+		(pts
 			(xy 152.4 107.95) (xy 156.21 107.95)
 		)
@@
 	(wire
 		(pts
-			(xy 149.86 135.89) (xy 152.4 135.89)
-		)
-		(stroke
-			(width 0)
-			(type default)
-		)
-	)
-	(wire
-		(pts
 			(xy 232.41 247.65) (xy 256.54 247.65)
 		)
@@
 	(wire
 		(pts
-			(xy 149.86 138.43) (xy 152.4 138.43)
-		)
-		(stroke
-			(width 0)
-			(type default)
-		)
-	)
-	(wire
-		(pts
 			(xy 242.57 80.01) (xy 256.54 80.01)
 		)
@@
 	(wire
 		(pts
-			(xy 152.4 135.89) (xy 156.21 135.89)
-		)
-		(stroke
-			(width 0)
-			(type default)
-		)
-	)
-	(wire
-		(pts
 			(xy 153.67 80.01) (xy 224.79 80.01)
 		)
@@
 		(pts
 			(xy 341.63 158.75) (xy 347.98 158.75)
-		)
-		(stroke
-			(width 0)
-			(type default)
-		)
-	)
-	(wire
-		(pts
-			(xy 152.4 100.33) (xy 157.48 100.33)
 		)
 		(stroke
@@
 		)
 	)
-	(label "GND"
-		(at 156.21 107.95 180)
-		(effects
-			(font
-				(size 1.27 1.27)
-			)
-			(justify right bottom)
-		)
-	)
 	(label "C3-UART-RX"
 		(at 177.8 133.35 180)
@@
 		)
 	)
-	(label "VBUS"
-		(at 152.4 95.25 0)
-		(effects
-			(font
-				(size 1.27 1.27)
-			)
-			(justify left bottom)
-		)
-	)
 	(label "RF-IN"
 		(at 383.54 147.32 180)
@@
 			)
 			(justify right bottom)
-		)
-	)
-	(global_label "~{SD}"
-		(shape input)
-		(at 156.21 135.89 0)
-		(fields_autoplaced yes)
-		(effects
-			(font
-				(size 1.27 1.27)
-			)
-			(justify left)
-		)
-		(property "Intersheetrefs" "${INTERSHEET_REFS}"
-			(at 161.1026 135.8106 0)
-			(show_name no)
-			(do_not_autoplace no)
-			(effects
-				(font
-					(size 1.27 1.27)
-				)
-				(justify left)
-			)
 		)
 	)
@@
 	)
 	(symbol
+		(lib_id "oresat-power:VBUS")
+		(at 156.21 95.25 0)
+		(unit 1)
+		(body_style 1)
+		(exclude_from_sim no)
+		(in_bom yes)
+		(on_board yes)
+		(in_pos_files yes)
+		(dnp no)
+		(property "Reference" "#VBUS02"
+			(at 156.21 95.25 0)
+			(hide yes)
+			(show_name no)
+			(do_not_autoplace no)
+			(effects
+				(font
+					(size 1.27 1.27)
+				)
+			)
+		)
+		(property "Value" "VBUS"
+			(at 156.21 92.456 0)
+			(show_name no)
+			(do_not_autoplace no)
+			(effects
+				(font
+					(size 1.27 1.27)
+				)
+				(justify bottom)
+			)
+		)
+		(property "Footprint" ""
+			(at 156.21 95.25 0)
+			(hide yes)
+			(show_name no)
+			(do_not_autoplace no)
+			(effects
+				(font
+					(size 1.27 1.27)
+				)
+			)
+		)
+		(property "Datasheet" ""
+			(at 156.21 95.25 0)
+			(hide yes)
+			(show_name no)
+			(do_not_autoplace no)
+			(effects
+				(font
+					(size 1.27 1.27)
+				)
+			)
+		)
+		(property "Description" "Power symbol creates a global label with name \"VBUS\""
+			(at 156.21 95.25 0)
+			(hide yes)
+			(show_name no)
+			(do_not_autoplace no)
+			(effects
+				(font
+					(size 1.27 1.27)
+				)
+			)
+		)
+		(pin "1"
+		)
+		(instances
+			(project "oresat-gps-card"
+				(path "/65d12cdd-c326-4033-9053-c59fa4e0b25e"
+					(reference "#VBUS02")
+					(unit 1)
+				)
+			)
+		)
+	)
+	(symbol
+		(lib_id "power:GND")
+		(at 156.21 107.95 0)
+		(unit 1)
+		(body_style 1)
+		(exclude_from_sim no)
+		(in_bom yes)
+		(on_board yes)
+		(in_pos_files yes)
+		(dnp no)
+		(property "Reference" "#GND0103"
+			(at 156.21 114.3 0)
+			(hide yes)
+			(show_name no)
+			(do_not_autoplace no)
+			(effects
+				(font
+					(size 1.27 1.27)
+				)
+			)
+		)
+		(property "Value" "GND"
+			(at 156.21 111.76 0)
+			(show_name no)
+			(do_not_autoplace no)
+			(effects
+				(font
+					(size 1.27 1.27)
+				)
+			)
+		)
+		(property "Footprint" ""
+			(at 156.21 107.95 0)
+			(hide yes)
+			(show_name no)
+			(do_not_autoplace no)
+			(effects
+				(font
+					(size 1.27 1.27)
+				)
+			)
+		)
+		(property "Datasheet" ""
+			(at 156.21 107.95 0)
+			(hide yes)
+			(show_name no)
+			(do_not_autoplace no)
+			(effects
+				(font
+					(size 1.27 1.27)
+				)
+			)
+		)
+		(property "Description" "Power symbol creates a global label with name \"GND\" , ground"
+			(at 156.21 107.95 0)
+			(hide yes)
+			(show_name no)
+			(do_not_autoplace no)
+			(effects
+				(font
+					(size 1.27 1.27)
+				)
+			)
+		)
+		(pin "1"
+		)
+		(instances
+			(project "oresat-gps-card"
+				(path "/65d12cdd-c326-4033-9053-c59fa4e0b25e"
+					(reference "#GND0103")
+					(unit 1)
+				)
+			)
+		)
+	)
+	(symbol
 		(lib_id "oresat-pcbs:ORESAT-CARD-V1.3-1RF-POS2")
 		(at 96.52 201.93 0)
@@
 			)
 		)
-		(property "Datasheet" "https://suddendocs.samtec.com/catalog_english/tfm.pdf"
+		(property "Datasheet" "https://mm.digikey.com/Volume0/opasdata/d220001/medias/docus/6129/tfm-1xx-xx-xxx-d-xxx-x-xx-mkt.pdf"
 			(at 144.78 26.67 0)
 			(hide yes)
@@
 			)
 		)
-		(property "Description" ""
+		(property "Description" "Connector Header Through Hole, Right Angle 40 position 0.050\" (1.27mm)"
+			(at 144.78 87.63 0)
+			(hide yes)
+			(show_name no)
+			(do_not_autoplace no)
+			(effects
+				(font
+					(size 1.27 1.27)
+				)
+			)
+		)
+		(property "DIS" "DigiKey"
+			(at 144.78 87.63 0)
+			(hide yes)
+			(show_name no)
+			(do_not_autoplace no)
+			(effects
+				(font
+					(size 1.27 1.27)
+				)
+			)
+		)
+		(property "DPN" "SAM10145-ND"
+			(at 144.78 87.63 0)
+			(hide yes)
+			(show_name no)
+			(do_not_autoplace no)
+			(effects
+				(font
+					(size 1.27 1.27)
+				)
+			)
+		)
+		(property "MFR" "Samtec Inc."
+			(at 144.78 87.63 0)
+			(hide yes)
+			(show_name no)
+			(do_not_autoplace no)
+			(effects
+				(font
+					(size 1.27 1.27)
+				)
+			)
+		)
+		(property "MPN" "TFM-120-01-L-D-RA"
 			(at 144.78 87.63 0)
 			(hide yes)
@@
 					(unit 1)
 				)
-			)
-		)
-	)
-	(symbol
-		(lib_id "power:PWR_FLAG")
-		(at 157.48 100.33 270)
-		(unit 1)
-		(body_style 1)
-		(exclude_from_sim no)
-		(in_bom yes)
-		(on_board yes)
-		(in_pos_files yes)
-		(dnp no)
-		(fields_autoplaced yes)
-		(property "Reference" "#FLG02"
-			(at 159.385 100.33 0)
-			(hide yes)
-			(show_name no)
-			(do_not_autoplace no)
-			(effects
-				(font
-					(size 1.27 1.27)
-				)
-			)
-		)
-		(property "Value" "PWR_FLAG"
-			(at 161.29 100.33 90)
-			(show_name no)
-			(do_not_autoplace no)
-			(effects
-				(font
-					(size 1.27 1.27)
-				)
-				(justify left)
-			)
-		)
-		(property "Footprint" ""
-			(at 157.48 100.33 0)
-			(hide yes)
-			(show_name no)
-			(do_not_autoplace no)
-			(effects
-				(font
-					(size 1.27 1.27)
-				)
-			)
-		)
-		(property "Datasheet" ""
-			(at 157.48 100.33 0)
-			(hide yes)
-			(show_name no)
-			(do_not_autoplace no)
-			(effects
-				(font
-					(size 1.27 1.27)
-				)
-			)
-		)
-		(property "Description" ""
-			(at 157.48 100.33 0)
-			(hide yes)
-			(show_name no)
-			(do_not_autoplace no)
-			(effects
-				(font
-					(size 1.27 1.27)
-				)
-			)
-		)
-		(pin "1"
-		)
-		(instances
-			(project "oresat-gps-card"
-				(path "/65d12cdd-c326-4033-9053-c59fa4e0b25e"
-					(reference "#FLG02")
-					(unit 1)
-				)

Commit message: ERC and DRC cleaneup
Fixed symbols, fixed footprints, changed DRC rules to reduce errors,
updated footprints, mostly done.
Other:
- sheet OSD3358 SYSBOOT : SIP D ports: added BOOTCFG; removed SYSBOOT2
- sheet Power ports: added BOOTCFG; removed SYSBOOT2
- company: (none) -> Portland State Aerospace Society
- moved on the sheet: CM1, J1, J3, J6, R68, TP159

Commit message: Last of the GPS card cleanup
    Better plains in the RF section, lots of shortening and straitening, cleaned up all ERC and DRCs.
Parts:
- added TP16, TP6, TP7: (no value), oresat-misc:TestPoint_RF_Probe, symbol oresat-misc:Test-Point-RF-Probe-Stripline
Connections:
- net MAX2769/MAX-RF: now also TP7.1
- net RF + RF Power/STQ-RF: now also TP16.1
- net RF-IN renamed LNA-IN-RF
- net LNA-IN-RF: now also TP6.1
Other:
- sheet RF + RF Power ports: added LNA-IN-RF; removed RF-IN
- moved on the sheet: CM1

Commit message: Clean up Orion UART names
Other:
- sheet OSD3358 SYSBOOT : SIP D ports: added UART2_RX, UART2_TX; removed STQ_UART2_RX, STQ_UART2_TX
- sheet SkyTraq ports: added UART2_RX, UART2_TX; removed STQ_UART2_RX, STQ_UART2_TX
Changed lines of the file:
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@@
 			)
 		)
-		(pin "STQ_UART2_RX" input
+		(pin "UART2_RX" input
 			(at 248.92 153.67 0)
 			(effects
@@
 			)
 		)
-		(pin "STQ_UART2_TX" input
+		(pin "UART2_TX" input
 			(at 248.92 151.13 0)
 			(effects
@@
 			)
 		)
-		(pin "STQ_UART2_RX" input
+		(pin "UART2_RX" input
 			(at 266.7 153.67 180)
 			(effects
@@
 			)
 		)
-		(pin "STQ_UART2_TX" input
+		(pin "UART2_TX" input
 			(at 266.7 151.13 180)
 			(effects
