File: oresat-gps-card/oresat-gps-card.kicad_sch (KiCad schematic)
At the start: 13 parts, among them J1 J-SAMTEC-TFM-120-01-L-D-RA, J3 GRPB041VWVN-RC, J6 SM14B-SHLS-TF

Commit message: BOM Update
Parts:
- R68: DIS (none) -> DigiKey; DPN (none) -> RNCP0603FTD75R0CT-ND; MFR (none) -> Stackpole Electronics Inc; MPN (none) -> RNCP0603FTD75R0
Changed lines of the file:
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@@
 			)
 		)
-		(property "Datasheet" ""
+		(property "Datasheet" "https://www.seielect.com/catalog/SEI-RNCP.pdf"
 			(at 171.45 200.66 0)
 			(hide yes)
@@
 			)
 		)
-		(property "Description" "Resistor, US symbol"
+		(property "Description" "75 Ohms ±1% 0.125W, 1/8W Chip Resistor 0603 (1608 Metric) Anti-Sulfur Thin Film"
 			(at 171.45 200.66 0)
 			(hide yes)
 			(show_name no)
+			(do_not_autoplace no)
+			(effects
+				(font
+					(size 1.27 1.27)
+				)
+			)
+		)
+		(property "DIS" "DigiKey"
+			(at 171.45 200.66 90)
+			(hide yes)
+			(show_name no)
+			(do_not_autoplace no)
+			(effects
+				(font
+					(size 1.27 1.27)
+				)
+			)
+		)
+		(property "DPN" "RNCP0603FTD75R0CT-ND"
+			(at 171.45 200.66 90)
+			(hide yes)
+			(show_name no)
+			(do_not_autoplace no)
+			(effects
+				(font
+					(size 1.27 1.27)
+				)
+			)
+		)
+		(property "MFR" "Stackpole Electronics Inc"
+			(at 171.45 200.66 90)
+			(hide yes)
+			(show_name no)
+			(do_not_autoplace no)
+			(effects
+				(font
+					(size 1.27 1.27)
+				)
+			)
+		)
+		(property "MPN" "RNCP0603FTD75R0"
+			(at 171.45 200.66 90)
+			(hide yes)
+			(show_name no)

Commit message: Large BOM changes for v1.2, no changes to PCB
Parts:
- CM1: DIS (none) -> DigiKey; DPN (none) -> 343-2477330-1CT-ND; MFR (none) -> TE Connectivity Linx; MPN (none) -> 2477330-1
- FID1, FID2, FID3, PCB1: now left out of the parts list
- J1: DPN SAM10145-ND -> SAM14509CT-ND; MPN TFM-120-01-L-D-RA -> SFM-120-02-L-DH-TR
- R68: value 75 -> 100; DPN RNCP0603FTD75R0CT-ND -> RMCF0603FT100RCT-ND; MFR Stackpole Electronics Inc -> Stackpole Electronics; MPN RNCP0603FTD75R0 -> RMCF0603FT100R
- TP159: value 0.03x0.04 -> Test-Point; now left out of the parts list
Changed lines of the file:
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@@
 		(body_style 1)
 		(exclude_from_sim no)
-		(in_bom yes)
+		(in_bom no)
 		(on_board yes)
 		(in_pos_files yes)
@@
 		(body_style 1)
 		(exclude_from_sim no)
-		(in_bom yes)
+		(in_bom no)
 		(on_board yes)
 		(in_pos_files yes)
@@
 			)
 		)
-		(property "Datasheet" "https://mm.digikey.com/Volume0/opasdata/d220001/medias/docus/6129/tfm-1xx-xx-xxx-d-xxx-x-xx-mkt.pdf"
+		(property "Datasheet" "https://mm.digikey.com/Volume0/opasdata/d220001/medias/docus/6129/sfm-1xx-xx-x-xh-xr-mkt.pdf"
 			(at 107.95 19.05 0)
 			(hide yes)
@@
 			)
 		)
-		(property "Description" "Connector Header Through Hole, Right Angle 40 position 0.050\" (1.27mm)"
+		(property "Description" "40 Position Receptacle Connector 0.050\"\" (1.27mm) Surface Mount, Right Angle Gold"
 			(at 107.95 80.01 0)
 			(hide yes)
@@
 			)
 		)
-		(property "DPN" "SAM10145-ND"
+		(property "DPN" "SAM14509CT-ND"
 			(at 107.95 80.01 0)
 			(hide yes)
@@
 			)
 		)
-		(property "MPN" "TFM-120-01-L-D-RA"
+		(property "MPN" "SFM-120-02-L-DH-TR"
 			(at 107.95 80.01 0)
 			(hide yes)
@@
 		(body_style 1)
 		(exclude_from_sim no)
-		(in_bom yes)
+		(in_bom no)
 		(on_board yes)
 		(in_pos_files yes)
@@
 			)
 		)
-		(property "Value" "0.03x0.04"
+		(property "Value" "Test-Point"
 			(at 173.99 219.71 0)
 			(hide yes)
@@
 		)
 		(property "Footprint" "oresat-misc:TestPoint-0.75mm-th"
-			(at 173.99 219.71 0)
+			(at 181.61 219.71 0)
 			(hide yes)
 			(show_name no)
@@
 		)
 		(property "Datasheet" ""
-			(at 173.99 219.71 0)
-			(hide yes)
-			(show_name no)
-			(do_not_autoplace no)
-			(effects
-				(font
-					(size 1.27 1.27)
-				)
-			)
-		)
-		(property "Description" ""
+			(at 171.45 219.71 0)
+			(hide yes)
+			(show_name no)
+			(do_not_autoplace no)
+			(effects
+				(font
+					(size 1.27 1.27)
+				)
+			)
+		)
+		(property "Description" "1mm round SMT test point"
 			(at 171.45 219.71 0)
 			(hide yes)
@@
 		(body_style 1)
 		(exclude_from_sim no)
-		(in_bom yes)
+		(in_bom no)
 		(on_board yes)
 		(in_pos_files yes)
@@
 			)
 		)
-		(property "Datasheet" "https://tools.molex.com/pdm_docs/sd/733000020_sd.pdf"
+		(property "Datasheet" "https://www.te.com/commerce/DocumentDelivery/DDEController?Action=srchrtrv&DocNm=SMPM_Connectors_Product_Extension-en&DocType=Data+Sheet&DocLang=English&DocFormat=pdf&PartCntxt=2477330-1"
 			(at 361.95 130.81 0)
 			(hide yes)
@@
 			)
 		)
-		(property "Description" "SMPM Connector Plug, Male Pin 50Ohm Board Edge, Cutout; Surface Mount Solder"
+		(property "Description" "SMPM Connector Plug, Male Pin 50 Ohms Board Edge, Cutout; Surface Mount Solder"
+			(at 361.95 139.7 0)
+			(hide yes)
+			(show_name no)
+			(do_not_autoplace no)
+			(effects
+				(font
+					(size 1.27 1.27)
+				)
+			)
+		)
+		(property "DIS" "DigiKey"
+			(at 361.95 139.7 0)
+			(hide yes)
+			(show_name no)
+			(do_not_autoplace no)
+			(effects
+				(font
+					(size 1.27 1.27)
+				)
+			)
+		)
+		(property "DPN" "343-2477330-1CT-ND"
+			(at 361.95 139.7 0)
+			(hide yes)
+			(show_name no)
+			(do_not_autoplace no)
+			(effects
+				(font
+					(size 1.27 1.27)
+				)
+			)
+		)
+		(property "MFR" "TE Connectivity Linx"
+			(at 361.95 139.7 0)
+			(hide yes)
+			(show_name no)
+			(do_not_autoplace no)
+			(effects
+				(font
+					(size 1.27 1.27)
+				)
+			)
+		)
+		(property "MPN" "2477330-1"
 			(at 361.95 139.7 0)
 			(hide yes)
@@
 		(dnp no)
 		(property "Reference" "R68"
-			(at 171.45 203.2 90)
+			(at 173.482 196.596 90)
 			(show_name no)
 			(do_not_autoplace no)
@@
 			)
 		)
-		(property "Value" "75"
-			(at 175.26 203.2 90)
+		(property "Value" "100"
+			(at 173.482 198.628 90)
 			(show_name no)
 			(do_not_autoplace no)
@@
 			)
 		)
-		(property "Datasheet" "https://www.seielect.com/catalog/SEI-RNCP.pdf"
+		(property "Datasheet" "https://www.seielect.com/catalog/SEI-RMCF_RMCP.pdf"
 			(at 171.45 200.66 0)
 			(hide yes)
@@
 			)
 		)
-		(property "Description" "75 Ohms ±1% 0.125W, 1/8W Chip Resistor 0603 (1608 Metric) Anti-Sulfur Thin Film"
+		(property "Description" "100 Ohms ±1% 0.1W, 1/10W Chip Resistor 0603 (1608 Metric) Automotive AEC-Q200 Thick Film"
 			(at 171.45 200.66 0)
 			(hide yes)
@@
 			)
 		)
-		(property "DPN" "RNCP0603FTD75R0CT-ND"
+		(property "DPN" "RMCF0603FT100RCT-ND"
 			(at 171.45 200.66 90)
 			(hide yes)
@@
 			)
 		)
-		(property "MFR" "Stackpole Electronics Inc"
+		(property "MFR" "Stackpole Electronics"
 			(at 171.45 200.66 90)
 			(hide yes)
@@
 			)
 		)
-		(property "MPN" "RNCP0603FTD75R0"
+		(property "MPN" "RMCF0603FT100R"
 			(at 171.45 200.66 90)
 			(hide yes)
@@
 		(body_style 1)
 		(exclude_from_sim no)
-		(in_bom yes)
-		(on_board yes)
-		(in_pos_files yes)
+		(in_bom no)
+		(on_board yes)
+		(in_pos_files yes)

Commit message: Upped to v1.3.
Fixed backward EEPROM programming pin, fixed potential boot error with missing PMIC connections, fixed some power domain issues.
Parts:
- J1: value J-SAMTEC-TFM-120-01-L-D-RA -> TFM-120-01-L-D-RA; DPN SAM14509CT-ND -> SAM10145-ND; MFR Samtec Inc. -> Samtec; MPN SFM-120-02-L-DH-TR -> TFM-120-01-L-D-RA
Connections:
- net EEPROM_WP: now also J3.3 (Pin_3); no longer J3.2 (Pin_2)
- net GND: now also J3.4 (Pin_4); no longer J3.1 (Pin_1)
- net PMIC_SCL: now also J3.1 (Pin_1); no longer J3.4 (Pin_4)
- net PMIC_SDA: now also J3.2 (Pin_2); no longer J3.3 (Pin_3)
Other:
- sheet OSD3358 USB, XTAL, etc : SIP B ports: added none; removed nRESET
- moved on the sheet: J3
Changed lines of the file:
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@@
 	(title_block
 		(title "OreSat GPS Card")
-		(date "2026-07-06")
-		(rev "1.2")
+		(date "2026-09-17")
+		(rev "1.3")
 		(company "Portland State Aerospace Society")
 	)
@@
 	)
 	(junction
-		(at 212.09 200.66)
-		(diameter 0)
-		(color 0 0 0 0)
-	)
-	(junction
 		(at 115.57 92.71)
 		(diameter 0)
@@
 	(wire
 		(pts
-			(xy 212.09 200.66) (xy 219.71 200.66)
-		)
-		(stroke
-			(width 0)
-			(type default)
-		)
-	)
-	(wire
-		(pts
 			(xy 248.92 138.43) (xy 266.7 138.43)
 		)
@@
 	(symbol
 		(lib_id "Connector_Generic:Conn_01x04")
-		(at 190.5 240.03 180)
+		(at 190.5 237.49 0)
+		(mirror y)
 		(unit 1)
 		(body_style 1)
@@
 		(in_pos_files yes)
 		(dnp no)
-		(fields_autoplaced yes)
 		(property "Reference" "J3"
-			(at 190.5 228.6 0)
+			(at 191.516 228.6 0)
 			(show_name no)
 			(do_not_autoplace no)
@@
 					(size 1.27 1.27)
 				)
+				(justify left)
 			)
 		)
 		(property "Value" "GRPB041VWVN-RC"
-			(at 190.5 231.14 0)
+			(at 199.39 231.14 0)
 			(show_name no)
 			(do_not_autoplace no)
@@
 					(size 1.27 1.27)
 				)
+				(justify left)
 			)
 		)
 		(property "Footprint" "Connector_PinHeader_1.27mm:PinHeader_1x04_P1.27mm_Vertical"
-			(at 190.5 240.03 0)
+			(at 190.5 237.49 0)
 			(hide yes)
 			(show_name no)
@@
 		)
 		(property "Datasheet" "https://s3.amazonaws.com/catalogspreads-pdf/PAGE94-95%20.050%20MALE%20HDR%20ST%20RA%20SMT.pdf"
-			(at 190.5 240.03 0)
+			(at 190.5 237.49 0)
 			(hide yes)
 			(show_name no)
@@
 		)
 		(property "Description" "Connector Header Through Hole 4 position 0.050\" (1.27mm)"
-			(at 190.5 240.03 0)
+			(at 190.5 237.49 0)
 			(hide yes)
 			(show_name no)
@@
 		)
 		(property "DPN" "S9014E-04-ND"
-			(at 190.5 240.03 0)
+			(at 190.5 237.49 0)
 			(hide yes)
 			(show_name no)
@@
 		)
 		(property "MFR" "Sullins Connector Solutions"
-			(at 190.5 240.03 0)
+			(at 190.5 237.49 0)
 			(hide yes)
 			(show_name no)
@@
 		)
 		(property "MPN" "GRPB041VWVN-RC"
-			(at 190.5 240.03 0)
+			(at 190.5 237.49 0)
 			(hide yes)
 			(show_name no)
@@
 		)
 		(property "DIS" "DigiKey"
-			(at 190.5 240.03 0)
+			(at 190.5 237.49 0)
 			(hide yes)
 			(show_name no)
@@
 			)
 		)
-		(property "Value" "J-SAMTEC-TFM-120-01-L-D-RA"
+		(property "Value" "TFM-120-01-L-D-RA"
 			(at 107.95 26.67 0)
 			(show_name no)
@@
 			)
 		)
-		(property "Datasheet" "https://mm.digikey.com/Volume0/opasdata/d220001/medias/docus/6129/sfm-1xx-xx-x-xh-xr-mkt.pdf"
+		(property "Datasheet" "https://suddendocs.samtec.com/catalog_english/tfm.pdf"
 			(at 107.95 19.05 0)
 			(hide yes)
@@
 			)
 		)
-		(property "Description" "40 Position Receptacle Connector 0.050\"\" (1.27mm) Surface Mount, Right Angle Gold"
+		(property "Description" "Connector Header Through Hole, Right Angle 40 position 0.050\" (1.27mm)"
 			(at 107.95 80.01 0)
 			(hide yes)
@@
 			)
 		)
-		(property "DPN" "SAM14509CT-ND"
+		(property "DPN" "SAM10145-ND"
 			(at 107.95 80.01 0)
 			(hide yes)
@@
 			)
 		)
-		(property "MFR" "Samtec Inc."
+		(property "MFR" "Samtec"
 			(at 107.95 80.01 0)
 			(hide yes)
@@
 			)
 		)
-		(property "MPN" "SFM-120-02-L-DH-TR"
+		(property "MPN" "TFM-120-01-L-D-RA"
 			(at 107.95 80.01 0)
 			(hide yes)
@@
 			)
 		)
-		(pin "GPS-EN" input
+		(pin "GPS-EN" output
 			(at 248.92 167.64 0)
 			(effects
@@
 			)
 		)
-		(pin "MAX_~{SHDN}" input
+		(pin "MAX_~{SHDN}" output
 			(at 248.92 125.73 0)
 			(effects
@@
 			)
 		)
-		(pin "MAX_SPI1_CS0" input
+		(pin "MAX_SPI1_CS0" output
 			(at 248.92 135.89 0)
 			(effects
@@
 			)
 		)
-		(pin "MAX_SPI1_D0" input
+		(pin "MAX_SPI1_D0" output
 			(at 248.92 133.35 0)
 			(effects
@@
 			)
 		)
-		(pin "MAX_SPI1_SCLK" input
+		(pin "MAX_SPI1_SCLK" output
 			(at 248.92 138.43 0)
 			(effects
@@
 			)
 		)
-		(pin "UART2_TX" input
+		(pin "UART2_TX" output
 			(at 248.92 151.13 0)
 			(effects
@@
 			)
 		)
-		(pin "nRESET" input
-			(at 219.71 200.66 180)
-			(effects
-				(font
-					(size 1.27 1.27)
-				)
-				(justify left)
-			)
-		)
 		(pin "USB_CLI_P" input
 			(at 219.71 190.5 180)
@@
 			)
 		)
-		(pin "Q1" input
+		(pin "Q1" output
 			(at 266.7 105.41 180)
 			(effects
@@
 			)
 		)
-		(pin "Q0" input
+		(pin "Q0" output
 			(at 266.7 102.87 180)
 			(effects
@@
 			)
 		)
-		(pin "I1" input
+		(pin "I1" output
 			(at 266.7 111.76 180)
 			(effects
@@
 			)
 		)
-		(pin "I0" input
+		(pin "I0" output
 			(at 266.7 109.22 180)
 			(effects
@@
 			)
 		)
-		(pin "MAX-CLKOUT" input
+		(pin "MAX-CLKOUT" output
 			(at 266.7 97.79 180)
 			(effects
@@
 			)
 		)
-		(pin "MAX-LD" input
+		(pin "MAX-LD" output
 			(at 266.7 128.27 180)
 			(effects
@@
 			)
 		)
-		(pin "STQ-RF" input
+		(pin "STQ-RF" output
 			(at 311.15 143.51 180)
 			(effects
@@
 			)
 		)
-		(pin "MAX-RF" input
+		(pin "MAX-RF" output
 			(at 311.15 132.08 180)
 			(effects
@@
 			)
 		)
-		(pin "CAN2_H" input
+		(pin "CAN2_H" bidirectional
 			(at 219.71 107.95 180)
 			(effects
@@
 			)
 		)
-		(pin "CAN2_L" input
+		(pin "CAN2_L" bidirectional
 			(at 219.71 110.49 180)
 			(effects
@@
 			)
 		)
-		(pin "STQ-1PPS" input
+		(pin "STQ-1PPS" output
 			(at 266.7 160.02 180)
 			(effects
@@
 			)
 		)
-		(pin "UART2_RX" input
+		(pin "UART2_RX" output
 			(at 266.7 153.67 180)
 			(effects
