File: oresat-gps-card/oresat-gps-card-sch-osd3358-sd-emmc.kicad_sch (KiCad schematic)
At the start: 21 parts, among them J4 DM3BT-DSF-PEJS, U1 OSD3358-512M-BSM, U8 TCAN330, U9 EMMC+RESET+5.1-COMPATIBLE-BA

Commit message: Routine Push
Lots of footprint changes
Parts:
- added D10, D11, D14: BLUE, LED_SMD:LED_0603_1608Metric, symbol Device:LED
- added R49, R50, R61: 10k, oresat-passives:0603-C-NOSILK, symbol Device:R_US
- C16, C25: footprint Capacitor_SMD:C_0603_1608Metric -> oresat-passives:0805-C-NOSILK
- C17, C18, C19, C20, C21, C22, C23, C24: footprint Capacitor_SMD:C_0603_1608Metric -> oresat-passives:0603-C-NOSILK
- R45: footprint Resistor_SMD:R_0603_1608Metric -> oresat-passives:0603-C-NOSILK
Connections:
- net GND: now also D10.1 (K), D11.1 (K), D14.1 (K)
- net at U1.P13 (GPMC_A5): now also R61.1
- net at U1.R14 (GPMC_A7): now also R49.1
- net at U1.T14 (GPMC_A6): now also R50.1
- new net: D10.2 (A), R49.2
- new net: D11.2 (A), R50.2
- new net: D14.2 (A), R61.2
- no-connect marks 50 -> 47

Commit message: Routine Push
Parts:
- renumbered D14 to D6, D11 to D7, D10 to D8, D7 to D9
Changed lines of the file:
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@@
 		(in_pos_files yes)
 		(dnp no)
-		(property "Reference" "D11"
+		(property "Reference" "D7"
 			(at 265.43 103.378 0)
 			(show_name no)
@@
 			(project "oresat-gps-card"
 				(path "/65d12cdd-c326-4033-9053-c59fa4e0b25e/f3d147ad-4cea-4d77-ae60-95882b03454e"
-					(reference "D11")
+					(reference "D7")
 					(unit 1)
 				)
@@
 		(in_pos_files yes)
 		(dnp no)
-		(property "Reference" "D10"
+		(property "Reference" "D8"
 			(at 265.43 109.728 0)
 			(show_name no)
@@
 			(project "oresat-gps-card"
 				(path "/65d12cdd-c326-4033-9053-c59fa4e0b25e/f3d147ad-4cea-4d77-ae60-95882b03454e"
-					(reference "D10")
+					(reference "D8")
 					(unit 1)
 				)
@@
 		(in_pos_files yes)
 		(dnp no)
-		(property "Reference" "D14"
+		(property "Reference" "D6"
 			(at 265.43 97.028 0)
 			(show_name no)
@@
 			(project "oresat-gps-card"
 				(path "/65d12cdd-c326-4033-9053-c59fa4e0b25e/f3d147ad-4cea-4d77-ae60-95882b03454e"
-					(reference "D14")
+					(reference "D6")
 					(unit 1)
 				)
@@
 		(in_pos_files yes)
 		(dnp no)
-		(property "Reference" "D7"
+		(property "Reference" "D9"
 			(at 265.43 116.078 0)
 			(show_name no)
@@
 			(project "oresat-gps-card"
 				(path "/65d12cdd-c326-4033-9053-c59fa4e0b25e/f3d147ad-4cea-4d77-ae60-95882b03454e"
-					(reference "D7")
+					(reference "D9")
 					(unit 1)
 				)

Commit message: Routine Push
Parts:
- C19, C20, C21, C22, C23, C24: DIS (none) -> DigiKey; DPN (none) -> 490-GRT188R71E105KE13DCT-ND; MFR (none) -> Murata Electronics; MPN (none) -> GRT188R71E105KE13D
- D6, D7, D8, D9: DIS (none) -> DigiKey; DPN (none) -> 732-4966-1-ND; MFR (none) -> Wurth; MPN (none) -> 150060BS75000
- J4: DIS (none) -> DigiKey; DPN (none) -> HR1942CT-ND; MFR (none) -> Hirose; MPN (none) -> DM3BT-DSF-PEJS
- R45, R49, R50, R61: DIS (none) -> DigiKey; DPN (none) -> RMCF0603FT10K0CT-ND; MFR (none) -> Stackpole Electronics; MPN (none) -> RMCF0603FT10K0
- U1: DIS (none) -> DigiKey; MFR (none) -> Octavo Systems LLC

Commit message: ERC and DRC cleaneup
Fixed symbols, fixed footprints, changed DRC rules to reduce errors,
updated footprints, mostly done.
Other:
- company: (none) -> Portland State Aerospace Society
Changed lines of the file:
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@@
 	(title_block
 		(title "OreSat GPS Card")
-		(date "2026-06-28")
+		(date "2026-07-06")
 		(rev "1.2")
+		(company "Portland State Aerospace Society")
 	)
 	(text "CAN1 RX --> B11 --> UART1_TXD\nCAN1 TX --> A11 --> UART1_RXD"
@@
 		)
 		(pin "E9"
-		)
-		(pin "E9"

Commit message: Last of the GPS card cleanup
    Better plains in the RF section, lots of shortening and straitening, cleaned up all ERC and DRCs.
Other:
- note added: "HH"
- note added: "LL"
- note added: "ZH"
- note added: "ZL"
- note added: "Z[L|0|CLK]"
- note removed: "KEEP OUT ZONE FOR UNCONNECTED EMMC PINS"
- moved on the sheet: TP26, TP27

Commit message: BOM Update
Parts:
- C16, C25: DIS (none) -> DigiKey; DPN (none) -> 490-GRT21BC71E106KE13KCT-ND; MFR (none) -> Murata Electronics; MPN (none) -> GRT21BC71E106KE13K
- C17, C18: DIS (none) -> DigiKey; DPN (none) -> 399-6856-1-ND; MFR (none) -> KEMET; MPN (none) -> C0603C104K5RACAUTO
- R69, R70, R71: DIS (none) -> DigiKey; DPN (none) -> RAVF164DJT10K0CT-ND; MFR (none) -> Stackpole Electronics Inc; MPN (none) -> RAVF164DJT10K0

Commit message: Large BOM changes for v1.2, no changes to PCB
Parts:
- R69, R70, R71: DPN RAVF164DJT10K0CT-ND -> U7103CT-ND; MFR Stackpole Electronics Inc -> Panasonic Electronic Components; MPN RAVF164DJT10K0 -> EXB-A10P103J
- TP26, TP27: value 0.03x0.04 -> Test-Point; now left out of the parts list
- U1: DPN (none) -> 1676-OSD3358-1G-ISM-ND; MFR Octavo Systems LLC -> Octavo Systems; MPN OSD3358-512M-BSM -> OSD3358-1G-ISM
- U8: DIS (none) -> DigiKey; DPN (none) -> 296-48971-1-ND; MFR (none) -> Texas Instruments; MPN (none) -> TCAN337GDCNR
- U9: DIS (none) -> DigiKey; DPN (none) -> 557-MTFC32GAZAQHD-IT-ND; MFR (none) -> Micron Technology Inc.; MPN (none) -> MTFC32GAZAQHD-IT
Changed lines of the file:
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@@
 		(body_style 1)
 		(exclude_from_sim no)
-		(in_bom yes)
+		(in_bom no)
 		(on_board yes)
 		(in_pos_files yes)
@@
 			)
 		)
-		(property "Value" "0.03x0.04"
+		(property "Value" "Test-Point"
 			(at 157.48 101.6 0)
 			(hide yes)
@@
 		)
 		(property "Footprint" "oresat-misc:TestPoint-0.75mm-th"
-			(at 157.48 101.6 0)
+			(at 157.48 93.98 0)
 			(hide yes)
 			(show_name no)
@@
 		)
 		(property "Datasheet" ""
-			(at 157.48 101.6 0)
+			(at 157.48 104.14 0)
 			(hide yes)
 			(show_name no)
@@
 			)
 		)
-		(property "Description" ""
+		(property "Description" "1mm round SMT test point"
 			(at 157.48 104.14 0)
 			(hide yes)
@@
 			)
 		)
-		(property "Datasheet" ""
+		(property "Datasheet" "https://www.micron.com/products/managed-nand/emmc/part-catalog/mtfc32gazaqhd-it?login"
 			(at 330.2 175.26 0)
 			(hide yes)
@@
 			)
 		)
-		(property "Description" ""
+		(property "Description" "FLASH - NAND Memory IC 256Gbit eMMC 200 MHz 153-VFBGA (11.5x13)"
+			(at 330.2 175.26 0)
+			(hide yes)
+			(show_name no)
+			(do_not_autoplace no)
+			(effects
+				(font
+					(size 1.27 1.27)
+				)
+			)
+		)
+		(property "DIS" "DigiKey"
+			(at 330.2 175.26 0)
+			(hide yes)
+			(show_name no)
+			(do_not_autoplace no)
+			(effects
+				(font
+					(size 1.27 1.27)
+				)
+			)
+		)
+		(property "DPN" "557-MTFC32GAZAQHD-IT-ND"
+			(at 330.2 175.26 0)
+			(hide yes)
+			(show_name no)
+			(do_not_autoplace no)
+			(effects
+				(font
+					(size 1.27 1.27)
+				)
+			)
+		)
+		(property "MFR" "Micron Technology Inc."
+			(at 330.2 175.26 0)
+			(hide yes)
+			(show_name no)
+			(do_not_autoplace no)
+			(effects
+				(font
+					(size 1.27 1.27)
+				)
+			)
+		)
+		(property "MPN" "MTFC32GAZAQHD-IT"
 			(at 330.2 175.26 0)
 			(hide yes)
@@
 			)
 		)
-		(property "Datasheet" "http://www.ti.com/lit/ds/symlink/tcan337.pdf"
+		(property "Datasheet" "https://www.ti.com/lit/ds/symlink/tcan337.pdf"
 			(at 160.02 48.26 0)
 			(hide yes)
@@
 			)
 		)
-		(property "Description" ""
+		(property "Description" "1/1 Transceiver CANbus SOT-23-8"
+			(at 160.02 48.26 0)
+			(hide yes)
+			(show_name no)
+			(do_not_autoplace no)
+			(effects
+				(font
+					(size 1.27 1.27)
+				)
+			)
+		)
+		(property "DIS" "DigiKey"
+			(at 160.02 48.26 0)
+			(hide yes)
+			(show_name no)
+			(do_not_autoplace no)
+			(effects
+				(font
+					(size 1.27 1.27)
+				)
+			)
+		)
+		(property "DPN" "296-48971-1-ND"
+			(at 160.02 48.26 0)
+			(hide yes)
+			(show_name no)
+			(do_not_autoplace no)
+			(effects
+				(font
+					(size 1.27 1.27)
+				)
+			)
+		)
+		(property "MFR" "Texas Instruments"
+			(at 160.02 48.26 0)
+			(hide yes)
+			(show_name no)
+			(do_not_autoplace no)
+			(effects
+				(font
+					(size 1.27 1.27)
+				)
+			)
+		)
+		(property "MPN" "TCAN337GDCNR"
 			(at 160.02 48.26 0)
 			(hide yes)
@@
 			)
 		)
-		(property "Description" "OSD335x Embedded Module 1GHz 512MB"
+		(property "Description" "Embedded Module ARM® Cortex®-A8, AM3358 1GHz 1GB"
 			(at 193.04 53.34 0)
 			(hide yes)
@@
 			)
 		)
-		(property "MPN" "OSD3358-512M-BSM"
+		(property "MPN" "OSD3358-1G-ISM"
 			(at 193.04 58.42 0)
 			(hide yes)
@@
 			)
 		)
-		(property "MFR" "Octavo Systems LLC"
+		(property "MFR" "Octavo Systems"
+			(at 193.04 157.48 0)
+			(hide yes)
+			(show_name no)
+			(do_not_autoplace no)
+			(effects
+				(font
+					(size 1.27 1.27)
+				)
+			)
+		)
+		(property "DPN" "1676-OSD3358-1G-ISM-ND"
 			(at 193.04 157.48 0)
 			(hide yes)
@@
 		(body_style 1)
 		(exclude_from_sim no)
-		(in_bom yes)
+		(in_bom no)
 		(on_board yes)
 		(in_pos_files yes)
@@
 			)
 		)
-		(property "Value" "0.03x0.04"
+		(property "Value" "Test-Point"
 			(at 157.48 104.14 0)
 			(hide yes)
@@
 		)
 		(property "Footprint" "oresat-misc:TestPoint-0.75mm-th"
-			(at 157.48 104.14 0)
+			(at 157.48 111.76 0)
 			(hide yes)
 			(show_name no)
@@
 		)
 		(property "Datasheet" ""
-			(at 157.48 104.14 0)
+			(at 157.48 101.6 0)
 			(hide yes)
 			(show_name no)
@@
 			)
 		)
-		(property "Description" ""
+		(property "Description" "1mm round SMT test point"
 			(at 157.48 101.6 0)
 			(hide yes)
@@
 			)
 		)
-		(property "Datasheet" "https://www.seielect.com/catalog/SEI-RAVF.pdf"
+		(property "Datasheet" "https://industrial.panasonic.com/ww/products/pt/resistor-network-array/models/EXBA10P103J"
 			(at 86.36 99.06 0)
 			(hide yes)
@@
 			)
 		)
-		(property "Description" "10k Ohm ±5% 100mW Power Per Element Isolated 4 Resistor Network/Array ±200ppm/°C 1206 (3216 Metric), Convex, Long Side Terminals"
+		(property "Description" "10k Ohm ±5% 62.5mW Power Per Element Bussed 8 Resistor Network/Array ±200ppm/°C 2512 (6432 Metric), Concave, Long Side Terminals"
 			(at 86.36 99.06 0)
 			(hide yes)
@@
 			)
 		)
-		(property "DPN" "RAVF164DJT10K0CT-ND"
+		(property "DPN" "U7103CT-ND"
 			(at 86.36 99.06 90)
 			(hide yes)
@@
 			)
 		)
-		(property "MFR" "Stackpole Electronics Inc"
+		(property "MFR" "Panasonic Electronic Components"
 			(at 86.36 99.06 90)
 			(hide yes)
@@
 			)
 		)
-		(property "MPN" "RAVF164DJT10K0"
+		(property "MPN" "EXB-A10P103J"
 			(at 86.36 99.06 90)
 			(hide yes)
@@
 			)
 		)
-		(property "Datasheet" "https://www.seielect.com/catalog/SEI-RAVF.pdf"
+		(property "Datasheet" "https://industrial.panasonic.com/ww/products/pt/resistor-network-array/models/EXBA10P103J"
 			(at 261.62 139.7 0)
 			(hide yes)
@@
 			)
 		)
-		(property "Description" "10k Ohm ±5% 100mW Power Per Element Isolated 4 Resistor Network/Array ±200ppm/°C 1206 (3216 Metric), Convex, Long Side Terminals"
+		(property "Description" "10k Ohm ±5% 62.5mW Power Per Element Bussed 8 Resistor Network/Array ±200ppm/°C 2512 (6432 Metric), Concave, Long Side Terminals"
 			(at 261.62 139.7 0)
 			(hide yes)
@@
 			)
 		)
-		(property "DPN" "RAVF164DJT10K0CT-ND"
+		(property "DPN" "U7103CT-ND"
 			(at 261.62 139.7 90)
 			(hide yes)
@@
 			)
 		)
-		(property "MFR" "Stackpole Electronics Inc"
+		(property "MFR" "Panasonic Electronic Components"
 			(at 261.62 139.7 90)
 			(hide yes)
@@
 			)
 		)
-		(property "MPN" "RAVF164DJT10K0"
+		(property "MPN" "EXB-A10P103J"
 			(at 261.62 139.7 90)
 			(hide yes)
@@
 			)
 		)
-		(property "Datasheet" "https://www.seielect.com/catalog/SEI-RAVF.pdf"
+		(property "Datasheet" "https://industrial.panasonic.com/ww/products/pt/resistor-network-array/models/EXBA10P103J"
 			(at 281.94 139.7 0)
 			(hide yes)
@@
 			)
 		)
-		(property "Description" "10k Ohm ±5% 100mW Power Per Element Isolated 4 Resistor Network/Array ±200ppm/°C 1206 (3216 Metric), Convex, Long Side Terminals"
+		(property "Description" "10k Ohm ±5% 62.5mW Power Per Element Bussed 8 Resistor Network/Array ±200ppm/°C 2512 (6432 Metric), Concave, Long Side Terminals"
 			(at 281.94 139.7 0)
 			(hide yes)
@@
 			)
 		)
-		(property "DPN" "RAVF164DJT10K0CT-ND"
+		(property "DPN" "U7103CT-ND"
 			(at 281.94 139.7 90)
 			(hide yes)
@@
 			)
 		)
-		(property "MFR" "Stackpole Electronics Inc"
+		(property "MFR" "Panasonic Electronic Components"
 			(at 281.94 139.7 90)
 			(hide yes)
@@
 			)
 		)
-		(property "MPN" "RAVF164DJT10K0"
+		(property "MPN" "EXB-A10P103J"
 			(at 281.94 139.7 90)
 			(hide yes)
