File: oresat-gps-card/oresat-gps-card-sch-osd3358-power.kicad_sch (KiCad schematic)
At the start: 17 parts, among them Q6 MMBT2907, U1 OSD3358-512M-BSM, U10 SN74LVC1G07DCK, U14 TLVH431

Commit message: Routine Push
Parts:
- C34, C35, C36: DIS (none) -> DigiKey; DPN (none) -> 490-12409-1-ND; MFR (none) -> Murata Electronics; MPN (none) -> GRT31CC81C226KE01L
- D4: DIS (none) -> DigiKey; DPN (none) -> 732-4971-1-ND; MFR (none) -> Wurth; MPN (none) -> 150060GS75000
- R48, R53, R54, R57: DIS (none) -> DigiKey; DPN (none) -> RMCF0603FT10K0CT-ND; MFR (none) -> Stackpole Electronics; MPN (none) -> RMCF0603FT10K0
- U1: DIS (none) -> DigiKey; MFR (none) -> Octavo Systems LLC
- U10: DIS (none) -> DigiKey; DPN (none) -> 296-8486-1-ND; MFR (none) -> Texas Instruments; MPN (none) -> SN74LVC1G07DCKR
- U14: DIS (none) -> DigiKey; DPN (none) -> 296-17972-1-ND; MFR (none) -> Texas Instruments; MPN (none) -> TLVH431AQDBZR

Commit message: ERC and DRC cleaneup
Fixed symbols, fixed footprints, changed DRC rules to reduce errors,
updated footprints, mostly done.
Parts:
- Q6: symbol Device:Q_PNP_BEC -> Transistor_BJT:Q_PNP_BEC
Other:
- company: (none) -> Portland State Aerospace Society
Changed lines of the file:
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@@
 	(title_block
 		(title "OreSat GPS Card")
-		(date "2026-06-28")
+		(date "2026-07-06")
 		(rev "1.2")
+		(company "Portland State Aerospace Society")
 	)
 	(text "Power from Debug \nconnector\n(USB client)"
@@
 	)
 	(symbol
-		(lib_name "GND_6")
 		(lib_id "power:GND")
 		(at 193.04 87.63 0)
@@
 	)
 	(symbol
-		(lib_name "GND_10")
 		(lib_id "power:GND")
 		(at 208.28 200.66 0)
@@
 	)
 	(symbol
-		(lib_name "GND_7")
 		(lib_id "power:GND")
 		(at 185.42 63.5 0)
@@
 	)
 	(symbol
-		(lib_name "GND_8")
 		(lib_id "power:GND")
 		(at 86.36 220.98 0)
@@
 	)
 	(symbol
-		(lib_name "GND_9")
 		(lib_id "power:GND")
 		(at 76.2 81.28 0)
@@
 	)
 	(symbol
-		(lib_name "GND_2")
 		(lib_id "power:GND")
 		(at 73.66 218.44 0)
@@
 	)
 	(symbol
-		(lib_name "GND_3")
 		(lib_id "power:GND")
 		(at 355.6 114.3 0)
@@
 	)
 	(symbol
-		(lib_id "Device:Q_PNP_BEC")
+		(lib_id "Transistor_BJT:Q_PNP_BEC")
 		(at 195.58 132.08 0)
 		(mirror y)
@@
 			)
 		)
-		(property "Description" ""
+		(property "Description" "PNP transistor, base/emitter/collector"
+			(at 195.58 132.08 0)
+			(hide yes)
+			(show_name no)
+			(do_not_autoplace no)
+			(effects
+				(font
+					(size 1.27 1.27)
+				)
+			)
+		)
+		(property "Sim.Device" "PNP"
+			(at 195.58 132.08 0)
+			(hide yes)
+			(show_name no)
+			(do_not_autoplace no)
+			(effects
+				(font
+					(size 1.27 1.27)
+				)
+			)
+		)
+		(property "Sim.Pins" "1=B 2=E 3=C"
 			(at 195.58 132.08 0)
 			(hide yes)
@@
 	)
 	(symbol
-		(lib_name "GND_4")
 		(lib_id "power:GND")
 		(at 195.58 208.28 0)
@@
 	)
 	(symbol
-		(lib_name "GND_5")
 		(lib_id "power:GND")
 		(at 76.2 63.5 0)
@@
 	)
 	(symbol
-		(lib_name "GND_1")
 		(lib_id "power:GND")
 		(at 289.56 114.3 0)

Commit message: Last of the GPS card cleanup
    Better plains in the RF section, lots of shortening and straitening, cleaned up all ERC and DRCs.
Connections:
- net 1.1V: no longer names the net of C36.1, U1.K6 (SYS_VOUT@1), U1.K7 (SYS_VOUT@2), U1.L6 (SYS_VOUT@3), U1.L7 (SYS_VOUT@4)
Other:
- note added: "1206"
- moved on the sheet: D4, R54

Commit message: BOM Update
Parts:
- C33, C78: DIS (none) -> DigiKey; DPN (none) -> 399-6856-1-ND; MFR (none) -> KEMET; MPN (none) -> C0603C104K5RACAUTO
- R55: DIS (none) -> DigiKey; DPN (none) -> RMCF0603FT499RCT-ND; MFR (none) -> Stackpole Electronics Inc; MPN (none) -> RMCF0603FT499R
- R56: DIS (none) -> DigiKey; DPN (none) -> RMCF0603FT40K2CT-ND; MFR (none) -> Stackpole Electronics Inc; MPN (none) -> RMCF0603FT40K2
Changed lines of the file:
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@@
 			)
 		)
-		(property "Datasheet" ""
+		(property "Datasheet" "https://search.kemet.com/download/specsheet/C0603C104K5RACAUTO"
 			(at 208.28 195.58 0)
 			(hide yes)
@@
 			)
 		)
-		(property "Description" "Unpolarized capacitor"
+		(property "Description" "0.1 µF ±10% 50V Ceramic Capacitor X7R 0603 (1608 Metric)"
+			(at 208.28 195.58 0)
+			(hide yes)
+			(show_name no)
+			(do_not_autoplace no)
+			(effects
+				(font
+					(size 1.27 1.27)
+				)
+			)
+		)
+		(property "DIS" "DigiKey"
+			(at 208.28 195.58 0)
+			(hide yes)
+			(show_name no)
+			(do_not_autoplace no)
+			(effects
+				(font
+					(size 1.27 1.27)
+				)
+			)
+		)
+		(property "DPN" "399-6856-1-ND"
+			(at 208.28 195.58 0)
+			(hide yes)
+			(show_name no)
+			(do_not_autoplace no)
+			(effects
+				(font
+					(size 1.27 1.27)
+				)
+			)
+		)
+		(property "MFR" "KEMET"
+			(at 208.28 195.58 0)
+			(hide yes)
+			(show_name no)
+			(do_not_autoplace no)
+			(effects
+				(font
+					(size 1.27 1.27)
+				)
+			)
+		)
+		(property "MPN" "C0603C104K5RACAUTO"
 			(at 208.28 195.58 0)
 			(hide yes)
@@
 			)
 		)
-		(property "Datasheet" ""
+		(property "Datasheet" "https://www.seielect.com/catalog/SEI-RMCF_RMCP.pdf"
 			(at 208.28 140.97 0)
 			(hide yes)
@@
 			)
 		)
-		(property "Description" "Resistor, US symbol"
+		(property "Description" "499 Ohms ±1% 0.1W, 1/10W Chip Resistor 0603 (1608 Metric) Automotive AEC-Q200 Thick Film"
 			(at 208.28 140.97 0)
 			(hide yes)
@@
 			)
 		)
+		(property "DIS" "DigiKey"
+			(at 208.28 140.97 90)
+			(hide yes)
+			(show_name no)
+			(do_not_autoplace no)
+			(effects
+				(font
+					(size 1.27 1.27)
+				)
+			)
+		)
+		(property "DPN" "RMCF0603FT499RCT-ND"
+			(at 208.28 140.97 90)
+			(hide yes)
+			(show_name no)
+			(do_not_autoplace no)
+			(effects
+				(font
+					(size 1.27 1.27)
+				)
+			)
+		)
+		(property "MFR" "Stackpole Electronics Inc"
+			(at 208.28 140.97 90)
+			(hide yes)
+			(show_name no)
+			(do_not_autoplace no)
+			(effects
+				(font
+					(size 1.27 1.27)
+				)
+			)
+		)
+		(property "MPN" "RMCF0603FT499R"
+			(at 208.28 140.97 90)
+			(hide yes)
+			(show_name no)
+			(do_not_autoplace no)
+			(effects
+				(font
+					(size 1.27 1.27)
+				)
+			)
+		)
 		(pin "1"
 		)
@@
 			)
 		)
-		(property "Datasheet" ""
+		(property "Datasheet" "https://www.seielect.com/catalog/SEI-RMCF_RMCP.pdf"
 			(at 218.44 115.57 0)
 			(hide yes)
@@
 			)
 		)
-		(property "Description" "Resistor, US symbol"
+		(property "Description" "40.2 kOhms ±1% 0.1W, 1/10W Chip Resistor 0603 (1608 Metric) Automotive AEC-Q200 Thick Film"
 			(at 218.44 115.57 0)
 			(hide yes)
@@
 			)
 		)
+		(property "DIS" "DigiKey"
+			(at 218.44 115.57 90)
+			(hide yes)
+			(show_name no)
+			(do_not_autoplace no)
+			(effects
+				(font
+					(size 1.27 1.27)
+				)
+			)
+		)
+		(property "DPN" "RMCF0603FT40K2CT-ND"
+			(at 218.44 115.57 90)
+			(hide yes)
+			(show_name no)
+			(do_not_autoplace no)
+			(effects
+				(font
+					(size 1.27 1.27)
+				)
+			)
+		)
+		(property "MFR" "Stackpole Electronics Inc"
+			(at 218.44 115.57 90)
+			(hide yes)
+			(show_name no)
+			(do_not_autoplace no)
+			(effects
+				(font
+					(size 1.27 1.27)
+				)
+			)
+		)
+		(property "MPN" "RMCF0603FT40K2"
+			(at 218.44 115.57 90)
+			(hide yes)
+			(show_name no)
+			(do_not_autoplace no)
+			(effects
+				(font
+					(size 1.27 1.27)
+				)
+			)
+		)
 		(pin "1"
 		)
@@
 			)
 		)
-		(property "Datasheet" ""
+		(property "Datasheet" "https://search.kemet.com/download/specsheet/C0603C104K5RACAUTO"
+			(at 218.44 220.98 0)
+			(hide yes)
+			(show_name no)
+			(do_not_autoplace no)
+			(effects
+				(font
+					(size 1.27 1.27)
+				)
+			)
+		)
+		(property "Description" "0.1 µF ±10% 50V Ceramic Capacitor X7R 0603 (1608 Metric)"
+			(at 218.44 220.98 0)
+			(hide yes)
+			(show_name no)
+			(do_not_autoplace no)
+			(effects
+				(font
+					(size 1.27 1.27)
+				)
+			)
+		)
+		(property "DIS" "DigiKey"
+			(at 218.44 220.98 0)
+			(hide yes)
+			(show_name no)
+			(do_not_autoplace no)
+			(effects
+				(font
+					(size 1.27 1.27)
+				)
+			)
+		)
+		(property "DPN" "399-6856-1-ND"
+			(at 218.44 220.98 0)
+			(hide yes)
+			(show_name no)
+			(do_not_autoplace no)
+			(effects
+				(font
+					(size 1.27 1.27)
+				)
+			)
+		)
+		(property "MFR" "KEMET"
 			(at 218.44 220.98 0)
 			(hide yes)
@@
 			)
 		)
-		(property "Description" "Unpolarized capacitor"
+		(property "MPN" "C0603C104K5RACAUTO"
 			(at 218.44 220.98 0)
 			(hide yes)

Commit message: Large BOM changes for v1.2, no changes to PCB
Parts:
- Q6: DIS (none) -> DigiKey; DPN (none) -> 1727-5176-1-ND; MFR (none) -> Nexperia; MPN (none) -> PMBT2907,215
- TP158: value 0.03x0.04 -> Test-Point; now left out of the parts list
- U1: DPN (none) -> 1676-OSD3358-1G-ISM-ND; MFR Octavo Systems LLC -> Octavo Systems; MPN OSD3358-512M-BSM -> OSD3358-1G-ISM
Changed lines of the file:
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@@
 		(body_style 1)
 		(exclude_from_sim no)
-		(in_bom yes)
+		(in_bom no)
 		(on_board yes)
 		(in_pos_files yes)
@@
 			)
 		)
-		(property "Value" "0.03x0.04"
+		(property "Value" "Test-Point"
 			(at 73.66 215.9 0)
 			(hide yes)
@@
 		)
 		(property "Footprint" "oresat-misc:TestPoint-0.75mm-th"
-			(at 73.66 215.9 0)
+			(at 73.66 223.52 0)
 			(hide yes)
 			(show_name no)
@@
 		)
 		(property "Datasheet" ""
-			(at 73.66 215.9 0)
-			(hide yes)
-			(show_name no)
-			(do_not_autoplace no)
-			(effects
-				(font
-					(size 1.27 1.27)
-				)
-			)
-		)
-		(property "Description" ""
+			(at 73.66 213.36 0)
+			(hide yes)
+			(show_name no)
+			(do_not_autoplace no)
+			(effects
+				(font
+					(size 1.27 1.27)
+				)
+			)
+		)
+		(property "Description" "1mm round SMT test point"
 			(at 73.66 213.36 0)
 			(hide yes)
@@
 			)
 		)
-		(property "Description" "OSD335x Embedded Module 1GHz 512MB"
+		(property "Description" "Embedded Module ARM® Cortex®-A8, AM3358 1GHz 1GB"
 			(at 322.58 76.2 0)
 			(hide yes)
@@
 			)
 		)
-		(property "MPN" "OSD3358-512M-BSM"
+		(property "MPN" "OSD3358-1G-ISM"
 			(at 322.58 81.28 0)
 			(hide yes)
@@
 			)
 		)
-		(property "MFR" "Octavo Systems LLC"
+		(property "MFR" "Octavo Systems"
+			(at 322.58 180.34 0)
+			(hide yes)
+			(show_name no)
+			(do_not_autoplace no)
+			(effects
+				(font
+					(size 1.27 1.27)
+				)
+			)
+		)
+		(property "DPN" "1676-OSD3358-1G-ISM-ND"
 			(at 322.58 180.34 0)
 			(hide yes)
@@
 			)
 		)
-		(property "Description" "OSD335x Embedded Module 1GHz 512MB"
+		(property "Description" "Embedded Module ARM® Cortex®-A8, AM3358 1GHz 1GB"
 			(at 134.62 27.94 0)
 			(hide yes)
@@
 			)
 		)
-		(property "MPN" "OSD3358-512M-BSM"
+		(property "MPN" "OSD3358-1G-ISM"
 			(at 134.62 33.02 0)
 			(hide yes)
@@
 			)
 		)
-		(property "MFR" "Octavo Systems LLC"
+		(property "MFR" "Octavo Systems"
+			(at 134.62 132.08 0)
+			(hide yes)
+			(show_name no)
+			(do_not_autoplace no)
+			(effects
+				(font
+					(size 1.27 1.27)
+				)
+			)
+		)
+		(property "DPN" "1676-OSD3358-1G-ISM-ND"
 			(at 134.62 132.08 0)
 			(hide yes)
@@
 			)
 		)
-		(property "Datasheet" ""
+		(property "Datasheet" "https://assets.nexperia.com/documents/data-sheet/PMBT2907.pdf"
 			(at 195.58 132.08 0)
 			(hide yes)
@@
 			)
 		)
-		(property "Description" "PNP transistor, base/emitter/collector"
+		(property "Description" "Bipolar (BJT) Transistor PNP 40 V 600 mA 200MHz 250 mW Surface Mount TO-236AB"
 			(at 195.58 132.08 0)
 			(hide yes)
@@
 		)
 		(property "Sim.Pins" "1=B 2=E 3=C"
+			(at 195.58 132.08 0)
+			(hide yes)
+			(show_name no)
+			(do_not_autoplace no)
+			(effects
+				(font
+					(size 1.27 1.27)
+				)
+			)
+		)
+		(property "DIS" "DigiKey"
+			(at 195.58 132.08 0)
+			(hide yes)
+			(show_name no)
+			(do_not_autoplace no)
+			(effects
+				(font
+					(size 1.27 1.27)
+				)
+			)
+		)
+		(property "DPN" "1727-5176-1-ND"
+			(at 195.58 132.08 0)
+			(hide yes)
+			(show_name no)
+			(do_not_autoplace no)
+			(effects
+				(font
+					(size 1.27 1.27)
+				)
+			)
+		)
+		(property "MFR" "Nexperia"
+			(at 195.58 132.08 0)
+			(hide yes)
+			(show_name no)
+			(do_not_autoplace no)
+			(effects
+				(font
+					(size 1.27 1.27)
+				)
+			)
+		)
+		(property "MPN" "PMBT2907,215"
 			(at 195.58 132.08 0)
 			(hide yes)
@@
 			)
 		)
-		(property "Description" "OSD335x Embedded Module 1GHz 512MB"
+		(property "Description" "Embedded Module ARM® Cortex®-A8, AM3358 1GHz 1GB"
 			(at 322.58 -27.94 0)
 			(hide yes)
@@
 			)
 		)
-		(property "MPN" "OSD3358-512M-BSM"
+		(property "MPN" "OSD3358-1G-ISM"
 			(at 322.58 -22.86 0)
 			(hide yes)
@@
 			)
 		)
-		(property "MFR" "Octavo Systems LLC"
+		(property "MFR" "Octavo Systems"
 			(at 322.58 76.2 0)
 			(hide yes)
+			(show_name no)
+			(do_not_autoplace no)
+			(effects
+				(font
+					(size 1.27 1.27)
+				)
+			)
+		)
+		(property "DPN" "1676-OSD3358-1G-ISM-ND"
+			(at 322.58 76.2 0)
+			(hide yes)

Commit message: Upped to v1.3.
Fixed backward EEPROM programming pin, fixed potential boot error with missing PMIC connections, fixed some power domain issues.
Parts:
- added D3: GRN, LED_SMD:LED_0603_1608Metric, symbol Device:LED
- added R33: 10k, oresat-passives:0603-C-NOSILK, symbol Device:R_US
- U1: value OSD3358-512M-BSM -> OSD3358-1G-ISM
Connections:
- net GND: now also D3.1 (K)
- net at U1.D4 (EXTINTN): now also U1.E4 (PMIC_NINT)
- net at C36.1, U1.K6 (SYS_VOUT@1), U1.K7 (SYS_VOUT@2)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: now also R33.2
- net at U1.L4 (PMIC_NWAKEUP): now also U1.M4 (EXT_WAKEUP)
- net at U1.N10 (PMIC_POWER_EN): now also U1.N11 (PMIC_PWR_EN)
- net at U1.N4 (PMIC_LDO_PGOOD): now also U1.N5 (RTC_PWRONRSTN)
- new net: D3.2 (A), R33.1
- no-connect marks 20 -> 12
Other:
- note added: ""5V""
- note added: "I2C0 has internal 4.7K pullups"
- moved on the sheet: D4, R54
